File: Electrical/PCB v1/L1/l1 v1/l1 v1.kicad_pcb (KiCad board)
At the start: 2 copper layers, 8.2 x 5 mm, 133 parts, among them J1 Conn_01x01_Socket, J2 Conn_01x01_Socket, P1 USB_C_Plug_USB2.0

Commit message: errr new resources parts list
Parts:
- removed P1: USB_C_Plug_USB2.0, Connector_USB:USB_C_Plug_JAE_DX07P024AJ1
- added LED_1: R_Photo, photoresistor:XDCR_ALS-PT19-315C_L177_TR8, F.Cu at (102.5, 66.2)
- added LED_10: R_Photo, photoresistor:XDCR_ALS-PT19-315C_L177_TR8, F.Cu at (106.9, 66.2)
- added LED_11: R_Photo, photoresistor:XDCR_ALS-PT19-315C_L177_TR8, F.Cu at (106.9, 68.5)
- added LED_12: R_Photo, photoresistor:XDCR_ALS-PT19-315C_L177_TR8, F.Cu at (106.9, 70.9)
- added LED_13: R_Photo, photoresistor:XDCR_ALS-PT19-315C_L177_TR8, F.Cu at (106.9, 73.2)
- added LED_14: R_Photo, photoresistor:XDCR_ALS-PT19-315C_L177_TR8, F.Cu at (106.9, 75.6)
- added LED_15: R_Photo, photoresistor:XDCR_ALS-PT19-315C_L177_TR8, F.Cu at (106.9, 78.0)
- added LED_16: R_Photo, photoresistor:XDCR_ALS-PT19-315C_L177_TR8, F.Cu at (106.9, 80.3)
- added LED_17: R_Photo, photoresistor:XDCR_ALS-PT19-315C_L177_TR8, F.Cu at (106.9, 82.7)
- added LED_18: R_Photo, photoresistor:XDCR_ALS-PT19-315C_L177_TR8, F.Cu at (106.9, 85.0)
- added LED_19: R_Photo, photoresistor:XDCR_ALS-PT19-315C_L177_TR8, F.Cu at (111.2, 66.2)
- added LED_2: R_Photo, photoresistor:XDCR_ALS-PT19-315C_L177_TR8, F.Cu at (102.5, 68.5)
- added LED_20: R_Photo, photoresistor:XDCR_ALS-PT19-315C_L177_TR8, F.Cu at (111.2, 68.5)
- added LED_21: R_Photo, photoresistor:XDCR_ALS-PT19-315C_L177_TR8, F.Cu at (111.2, 70.9)
- added LED_22: R_Photo, photoresistor:XDCR_ALS-PT19-315C_L177_TR8, F.Cu at (111.2, 73.2)
- added LED_23: R_Photo, photoresistor:XDCR_ALS-PT19-315C_L177_TR8, F.Cu at (111.2, 75.6)
- added LED_24: R_Photo, photoresistor:XDCR_ALS-PT19-315C_L177_TR8, F.Cu at (111.2, 78.0)
- added LED_25: R_Photo, photoresistor:XDCR_ALS-PT19-315C_L177_TR8, F.Cu at (111.2, 80.3)
- added LED_26: R_Photo, photoresistor:XDCR_ALS-PT19-315C_L177_TR8, F.Cu at (111.2, 82.7)
- added LED_27: R_Photo, photoresistor:XDCR_ALS-PT19-315C_L177_TR8, F.Cu at (111.2, 85.0)
- added LED_28: R_Photo, photoresistor:XDCR_ALS-PT19-315C_L177_TR8, F.Cu at (115.6, 66.2)
- added LED_29: R_Photo, photoresistor:XDCR_ALS-PT19-315C_L177_TR8, F.Cu at (115.6, 68.5)
- added LED_3: R_Photo, photoresistor:XDCR_ALS-PT19-315C_L177_TR8, F.Cu at (102.5, 70.9)
- added LED_30: R_Photo, photoresistor:XDCR_ALS-PT19-315C_L177_TR8, F.Cu at (115.6, 70.9)
- added LED_31: R_Photo, photoresistor:XDCR_ALS-PT19-315C_L177_TR8, F.Cu at (115.6, 73.2)
- added LED_32: R_Photo, photoresistor:XDCR_ALS-PT19-315C_L177_TR8, F.Cu at (115.6, 75.6)
- added LED_4: R_Photo, photoresistor:XDCR_ALS-PT19-315C_L177_TR8, F.Cu at (102.5, 73.2)
- added LED_5: R_Photo, photoresistor:XDCR_ALS-PT19-315C_L177_TR8, F.Cu at (102.5, 75.6)
- added LED_6: R_Photo, photoresistor:XDCR_ALS-PT19-315C_L177_TR8, F.Cu at (102.5, 78.0)
- added LED_7: R_Photo, photoresistor:XDCR_ALS-PT19-315C_L177_TR8, F.Cu at (102.5, 80.3)
- added LED_8: R_Photo, photoresistor:XDCR_ALS-PT19-315C_L177_TR8, F.Cu at (102.5, 82.7)
- added LED_9: R_Photo, photoresistor:XDCR_ALS-PT19-315C_L177_TR8, F.Cu at (102.5, 85.0)
- moved LED1 0.95 mm to (72.0, 63.8), turned to 180 degrees
Other:
- board outline removed

Commit message: mounting holes!
Parts:
- added H1: MountingHole, MountingHole:MountingHole_3.2mm_M3, F.Cu at (93.8, 175.3)
- added H10: MountingHole, MountingHole:MountingHole_3.2mm_M3, F.Cu at (124.7, 78.0)
- added H11: MountingHole, MountingHole:MountingHole_3.2mm_M3, F.Cu at (117.3, 34.5)
- added H12: MountingHole, MountingHole:MountingHole_3.2mm_M3, F.Cu at (109.9, 78.0)
- added H13: MountingHole, MountingHole:MountingHole_3.2mm_M3, F.Cu at (96.2, 64.2)
- added H14: MountingHole, MountingHole:MountingHole_3.2mm_M3, F.Cu at (73.0, 87.4)
- added H15: MountingHole, MountingHole:MountingHole_3.2mm_M3, F.Cu at (86.8, 101.1)
- added H16: MountingHole, MountingHole:MountingHole_3.2mm_M3, F.Cu at (43.3, 108.5)
- added H17: MountingHole, MountingHole:MountingHole_3.2mm_M3, F.Cu at (86.8, 115.9)
- added H18: MountingHole, MountingHole:MountingHole_3.2mm_M3, F.Cu at (73.0, 129.6)
- added H19: MountingHole, MountingHole:MountingHole_3.2mm_M3, F.Cu at (96.2, 152.7)
- added H2: MountingHole, MountingHole:MountingHole_3.2mm_M3, F.Cu at (140.8, 175.3)
- added H20: MountingHole, MountingHole:MountingHole_3.2mm_M3, F.Cu at (109.9, 139.0)
- added H21: MountingHole, MountingHole:MountingHole_3.2mm_M3, F.Cu at (124.7, 139.0)
- added H3: MountingHole, MountingHole:MountingHole_3.2mm_M3, F.Cu at (138.4, 152.8)
- added H4: MountingHole, MountingHole:MountingHole_3.2mm_M3, F.Cu at (161.5, 129.7)
- added H5: MountingHole, MountingHole:MountingHole_3.2mm_M3, F.Cu at (147.8, 115.9)
- added H6: MountingHole, MountingHole:MountingHole_3.2mm_M3, F.Cu at (191.3, 108.5)
- added H7: MountingHole, MountingHole:MountingHole_3.2mm_M3, F.Cu at (147.8, 101.1)
- added H8: MountingHole, MountingHole:MountingHole_3.2mm_M3, F.Cu at (161.5, 87.4)
- added H9: MountingHole, MountingHole:MountingHole_3.2mm_M3, F.Cu at (138.4, 64.2)
- added LED1 (x31): WHITE 3528, LED_SMD:LED_0201_0603Metric, F.Cu at (0.00, 0.00)
- LED1, LED10, LED11, LED12, LED13, LED14, LED15, LED16, LED17, LED18, LED19, LED2, LED20, LED21, LED22, LED23, LED24, LED25, LED26, LED27, LED28, LED29, LED3, LED30, LED31, LED32, LED4, LED5, LED6, LED7, LED8, LED9: footprint SM0603UYC:LED_SM0603UYC -> LED_SMD:LED_0201_0603Metric
- moved C1 256.2 mm to (-114.3, 26.7)
- moved C10 256.2 mm to (-114.3, 49.3)
- moved C11 256.2 mm to (-114.3, 51.8)
- moved C2 256.2 mm to (-114.3, 29.2)
- moved C3 256.2 mm to (-114.3, 31.7)
- moved C4 256.2 mm to (-114.3, 34.2)
- moved C5 256.2 mm to (-114.3, 36.8)
- moved C6 256.2 mm to (-114.3, 39.3)
- moved C7 256.2 mm to (-114.3, 41.8)
- moved C8 256.2 mm to (-114.3, 44.3)
- moved C9 256.2 mm to (-114.3, 46.8)
- moved L10 256.2 mm to (-109.5, 54.5)
- moved L11 256.2 mm to (-109.5, 57.2)
- moved L12 256.2 mm to (-109.5, 60.0)
- moved L13 256.2 mm to (-109.5, 62.7)
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
Commit message: new version with the thingy wutht the light ringt
i need the photoresistors to be in yikai to do
Parts:
- removed C10, C11, C12, C13, C14, C15, C16, C17, C18, C19, C2, C20, C21, C22, C23, C24, C25, C26, C27, C28, C29, C3, C30, C31, C32, C4, C5, C6, C7, C8, C9: 1uF, Capacitor_SMD:C_0603_1608Metric
- removed the LED1 at (0.00, 0.00) (x32)
- removed LED10, LED11, LED12, LED13, LED14, LED15, LED16, LED17, LED18, LED19, LED2, LED20, LED21, LED22, LED23, LED24, LED25, LED26, LED27, LED28, LED29, LED3, LED30, LED31, LED32, LED4, LED5, LED6, LED7, LED8, LED9: WHITE 3528, LED_SMD:LED_0201_0603Metric
- removed R1, R10, R11, R12, R13, R14, R15, R16, R17, R18, R19, R2, R20, R21, R22, R23, R24, R25, R26, R27, R28, R29, R3, R30, R31, R32, R4, R5, R6, R7, R8, R9: 0R39, Resistor_SMD:R_0603_1608Metric
- added C33: 1uF, Capacitor_SMD:C_0603_1608Metric, F.Cu at (97.0, 105.8)
- added C34: 1uF, Capacitor_SMD:C_0603_1608Metric, F.Cu at (97.4, 109.7)
- added C35: 1uF, Capacitor_SMD:C_0603_1608Metric, F.Cu at (98.6, 113.5)
- added C36: 1uF, Capacitor_SMD:C_0603_1608Metric, F.Cu at (100.4, 116.9)
- added C37: 1uF, Capacitor_SMD:C_0603_1608Metric, F.Cu at (102.9, 119.9)
- added C38: 1uF, Capacitor_SMD:C_0603_1608Metric, F.Cu at (106.0, 122.4)
- added C39: 1uF, Capacitor_SMD:C_0603_1608Metric, F.Cu at (109.5, 124.2)
- added C40: 1uF, Capacitor_SMD:C_0603_1608Metric, F.Cu at (113.2, 125.3)
- added C41: 1uF, Capacitor_SMD:C_0603_1608Metric, F.Cu at (117.1, 125.7)
- added C42: 1uF, Capacitor_SMD:C_0603_1608Metric, F.Cu at (121.0, 125.2)
- added C43: 1uF, Capacitor_SMD:C_0603_1608Metric, F.Cu at (124.8, 124.1)
- added C44: 1uF, Capacitor_SMD:C_0603_1608Metric, F.Cu at (128.2, 122.2)
- added C45: 1uF, Capacitor_SMD:C_0603_1608Metric, F.Cu at (131.2, 119.7)
- added C46: 1uF, Capacitor_SMD:C_0603_1608Metric, F.Cu at (133.7, 116.6)
- added C47: 1uF, Capacitor_SMD:C_0603_1608Metric, F.Cu at (135.5, 113.2)
- added C48: 1uF, Capacitor_SMD:C_0603_1608Metric, F.Cu at (136.6, 109.4)
- added C49: 1uF, Capacitor_SMD:C_0603_1608Metric, F.Cu at (137.0, 105.5)
- added C50: 1uF, Capacitor_SMD:C_0603_1608Metric, F.Cu at (136.5, 101.6)
- added C51: 1uF, Capacitor_SMD:C_0603_1608Metric, F.Cu at (135.4, 97.8)
- added C52: 1uF, Capacitor_SMD:C_0603_1608Metric, F.Cu at (133.5, 94.4)
- added C53: 1uF, Capacitor_SMD:C_0603_1608Metric, F.Cu at (131.0, 91.4)
- added C54: 1uF, Capacitor_SMD:C_0603_1608Metric, F.Cu at (127.9, 88.9)
- added C55: 1uF, Capacitor_SMD:C_0603_1608Metric, F.Cu at (124.5, 87.1)
- added C56: 1uF, Capacitor_SMD:C_0603_1608Metric, F.Cu at (120.7, 86.0)
- added C57: 1uF, Capacitor_SMD:C_0603_1608Metric, F.Cu at (116.8, 85.7)
- added C58: 1uF, Capacitor_SMD:C_0603_1608Metric, F.Cu at (112.9, 86.1)
- added C59: 1uF, Capacitor_SMD:C_0603_1608Metric, F.Cu at (109.2, 87.2)
- added C60: 1uF, Capacitor_SMD:C_0603_1608Metric, F.Cu at (105.7, 89.1)
- added C61: 1uF, Capacitor_SMD:C_0603_1608Metric, F.Cu at (102.7, 91.6)
- added C62: 1uF, Capacitor_SMD:C_0603_1608Metric, F.Cu at (100.2, 94.7)
- added C63: 1uF, Capacitor_SMD:C_0603_1608Metric, F.Cu at (98.4, 98.2)
- added LED1: WHITE 3528, LED_SMD:LED_0201_0603Metric, F.Cu at (116.6, 162.5)
- added LED33: WHITE 3528, LED_SMD:LED_0201_0603Metric, F.Cu at (127.3, 161.4)
- added LED34: WHITE 3528, LED_SMD:LED_0201_0603Metric, F.Cu at (137.6, 158.3)
- added LED35: WHITE 3528, LED_SMD:LED_0201_0603Metric, F.Cu at (147.1, 153.2)
- added LED36: WHITE 3528, LED_SMD:LED_0201_0603Metric, F.Cu at (155.5, 146.4)
- added LED37: WHITE 3528, LED_SMD:LED_0201_0603Metric, F.Cu at (162.3, 138.0)
- added LED38: WHITE 3528, LED_SMD:LED_0201_0603Metric, F.Cu at (167.4, 128.5)
- added LED39: WHITE 3528, LED_SMD:LED_0201_0603Metric, F.Cu at (170.5, 118.2)
- added LED40: WHITE 3528, LED_SMD:LED_0201_0603Metric, F.Cu at (171.6, 107.5)
- added LED41: WHITE 3528, LED_SMD:LED_0201_0603Metric, F.Cu at (170.5, 96.8)
- added LED42: WHITE 3528, LED_SMD:LED_0201_0603Metric, F.Cu at (167.4, 86.4)
- added LED43: WHITE 3528, LED_SMD:LED_0201_0603Metric, F.Cu at (162.3, 76.9)
- added LED44: WHITE 3528, LED_SMD:LED_0201_0603Metric, F.Cu at (155.5, 68.6)
- added LED45: WHITE 3528, LED_SMD:LED_0201_0603Metric, F.Cu at (147.1, 61.7)
- added LED46: WHITE 3528, LED_SMD:LED_0201_0603Metric, F.Cu at (137.6, 56.7)
- added LED47: WHITE 3528, LED_SMD:LED_0201_0603Metric, F.Cu at (127.3, 53.5)
- added LED48: WHITE 3528, LED_SMD:LED_0201_0603Metric, F.Cu at (116.6, 52.5)
- added LED49: WHITE 3528, LED_SMD:LED_0201_0603Metric, F.Cu at (105.8, 53.5)
- added LED50: WHITE 3528, LED_SMD:LED_0201_0603Metric, F.Cu at (95.5, 56.7)
- added LED51: WHITE 3528, LED_SMD:LED_0201_0603Metric, F.Cu at (86.0, 61.7)
- added LED52: WHITE 3528, LED_SMD:LED_0201_0603Metric, F.Cu at (77.7, 68.6)
- added LED53: WHITE 3528, LED_SMD:LED_0201_0603Metric, F.Cu at (70.8, 76.9)
- added LED54: WHITE 3528, LED_SMD:LED_0201_0603Metric, F.Cu at (65.8, 86.4)
- added LED55: WHITE 3528, LED_SMD:LED_0201_0603Metric, F.Cu at (62.6, 96.8)
- added LED56: WHITE 3528, LED_SMD:LED_0201_0603Metric, F.Cu at (61.6, 107.5)
- added LED57: WHITE 3528, LED_SMD:LED_0201_0603Metric, F.Cu at (62.6, 118.2)
- added LED58: WHITE 3528, LED_SMD:LED_0201_0603Metric, F.Cu at (65.8, 128.5)
- added LED59: WHITE 3528, LED_SMD:LED_0201_0603Metric, F.Cu at (70.8, 138.0)
- added LED60: WHITE 3528, LED_SMD:LED_0201_0603Metric, F.Cu at (77.7, 146.4)
- added LED61: WHITE 3528, LED_SMD:LED_0201_0603Metric, F.Cu at (86.0, 153.2)
- added LED62: WHITE 3528, LED_SMD:LED_0201_0603Metric, F.Cu at (95.5, 158.3)
- added LED63: WHITE 3528, LED_SMD:LED_0201_0603Metric, F.Cu at (105.8, 161.4)
- moved C1 224.6 mm to (97.3, 101.9)
- moved L1 183.8 mm to (65.0, 96.0), turned to -90 degrees
- moved L10 117.5 mm to (-23.0, 133.9)
- moved L11 117.5 mm to (-23.0, 136.7)
- moved L12 117.5 mm to (-23.0, 139.4)
- moved L13 117.5 mm to (-23.0, 142.2)
- moved L14 117.5 mm to (-23.0, 144.9)
- moved L15 117.5 mm to (-23.0, 147.7)
- moved L16 117.5 mm to (-23.0, 150.4)
- moved L17 117.5 mm to (-23.0, 153.2)
- moved L18 117.5 mm to (-23.0, 155.9)
- moved L2 117.5 mm to (-27.5, 136.7)
- moved L3 117.5 mm to (-27.5, 139.4)
- moved L4 117.5 mm to (-27.5, 142.2)
- moved L5 117.5 mm to (-27.5, 144.9)
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
Commit message: edge cuts xt 30 adn the essp 32 to be added
Parts:
- removed the C1 at (97.3, 101.9)
- removed C33, C34, C35, C36, C37, C38, C39, C40, C41, C42, C43, C44, C45, C46, C47, C48, C49, C50, C51, C52, C53, C54, C55, C56, C57, C58, C59, C60, C61, C62, C63: 1uF, Capacitor_SMD:C_0603_1608Metric
- removed J1: Conn_01x01_Socket, Connector_Wire:SolderWirePad_1x01_SMD_1x2mm
- removed J2: Conn_01x01_Socket, Connector_Wire:SolderWire-0.5sqmm_1x01_D0.9mm_OD2.1mm
- removed the L1 at (65.0, 96.0)
- removed the LED1 at (116.6, 162.5)
- removed LED33, LED34, LED35, LED36, LED37, LED38, LED39, LED40, LED41, LED42, LED43, LED44, LED45, LED46, LED47, LED48, LED49, LED50, LED51, LED52, LED53, LED54, LED55, LED56, LED57, LED58, LED59, LED60, LED61, LED62, LED63: WHITE 3528, LED_SMD:LED_0201_0603Metric
- removed LED_1, LED_10, LED_11, LED_12, LED_13, LED_14, LED_15, LED_16, LED_17, LED_18, LED_19, LED_2, LED_20, LED_21, LED_22, LED_23, LED_24, LED_25, LED_26, LED_27, LED_28, LED_29, LED_3, LED_30, LED_31, LED_32, LED_4, LED_5, LED_6, LED_7, LED_8, LED_9: R_Photo, photoresistor:XDCR_ALS-PT19-315C_L177_TR8
- removed TP1, TP2: TestPoint, TestPoint:TestPoint_2Pads_Pitch2.54mm_Drill0.8mm
- added C1: 1uF, Capacitor_SMD:C_0603_1608Metric, F.Cu at (107.0, 164.5)
- added C1: 1uF, Capacitor_SMD:C_0603_1608Metric, F.Cu at (166.6, 76.9)
- added C1: 1uF, Capacitor_SMD:C_0603_1608Metric, F.Cu at (62.4, 119.1)
- added C1: 1uF, Capacitor_SMD:C_0603_1608Metric, F.Cu at (129.4, 164.7)
- added C1: 1uF, Capacitor_SMD:C_0603_1608Metric, F.Cu at (97.2, 55.3)
- added C1: 1uF, Capacitor_SMD:C_0603_1608Metric, F.Cu at (118.2, 165.7)
- added C1: 1uF, Capacitor_SMD:C_0603_1608Metric, F.Cu at (171.8, 86.9)
- added C1: 1uF, Capacitor_SMD:C_0603_1608Metric, F.Cu at (70.8, 139.8)
- added C1: 1uF, Capacitor_SMD:C_0603_1608Metric, F.Cu at (77.8, 148.6)
- added C1: 1uF, Capacitor_SMD:C_0603_1608Metric, F.Cu at (140.2, 161.5)
- added C1: 1uF, Capacitor_SMD:C_0603_1608Metric, F.Cu at (96.3, 161.1)
- added C1: 1uF, Capacitor_SMD:C_0603_1608Metric, F.Cu at (175.0, 97.7)
- added C1: 1uF, Capacitor_SMD:C_0603_1608Metric, F.Cu at (119.2, 51.1)
- added C1: 1uF, Capacitor_SMD:C_0603_1608Metric, F.Cu at (62.6, 96.8)
- added C1: 1uF, Capacitor_SMD:C_0603_1608Metric, F.Cu at (86.5, 155.8)
- added C1: 1uF, Capacitor_SMD:C_0603_1608Metric, F.Cu at (171.4, 130.7)
- added C1: 1uF, Capacitor_SMD:C_0603_1608Metric, F.Cu at (176.0, 108.9)
- added C1: 1uF, Capacitor_SMD:C_0603_1608Metric, F.Cu at (174.8, 120.0)
- added C1: 1uF, Capacitor_SMD:C_0603_1608Metric, F.Cu at (71.3, 76.2)
- added C1: 1uF, Capacitor_SMD:C_0603_1608Metric, F.Cu at (65.9, 86.0)
- added C1: 1uF, Capacitor_SMD:C_0603_1608Metric, F.Cu at (78.5, 67.5)
- added C1: 1uF, Capacitor_SMD:C_0603_1608Metric, F.Cu at (87.2, 60.5)
- added C1: 1uF, Capacitor_SMD:C_0603_1608Metric, F.Cu at (65.6, 129.9)
- added C1: 1uF, Capacitor_SMD:C_0603_1608Metric, F.Cu at (158.0, 148.6)
- added C1: 1uF, Capacitor_SMD:C_0603_1608Metric, F.Cu at (130.3, 52.3)
- added C1: 1uF, Capacitor_SMD:C_0603_1608Metric, F.Cu at (141.0, 55.6)
- added C1: 1uF, Capacitor_SMD:C_0603_1608Metric, F.Cu at (166.1, 140.6)
- added C1: 1uF, Capacitor_SMD:C_0603_1608Metric, F.Cu at (159.5, 68.2)
- added C1: 1uF, Capacitor_SMD:C_0603_1608Metric, F.Cu at (108.0, 52.1)
- added C1: 1uF, Capacitor_SMD:C_0603_1608Metric, F.Cu at (150.9, 61.0)
- added C1: 1uF, Capacitor_SMD:C_0603_1608Metric, F.Cu at (149.9, 156.0)
- added C1: 1uF, Capacitor_SMD:C_0603_1608Metric, F.Cu at (61.4, 107.9)
- added C10: 1uF, Capacitor_SMD:C_0603_1608Metric, F.Cu at (-128.6, 62.6)
- added C11: 1uF, Capacitor_SMD:C_0603_1608Metric, F.Cu at (-124.6, 42.6)
- added C12: 1uF, Capacitor_SMD:C_0603_1608Metric, F.Cu at (-124.6, 45.1)
- added C13: 1uF, Capacitor_SMD:C_0603_1608Metric, F.Cu at (-124.6, 47.6)
- added C14: 1uF, Capacitor_SMD:C_0603_1608Metric, F.Cu at (-124.6, 50.1)
- added C15: 1uF, Capacitor_SMD:C_0603_1608Metric, F.Cu at (-124.6, 52.6)
- added C16: 1uF, Capacitor_SMD:C_0603_1608Metric, F.Cu at (-124.6, 55.1)
- added C17: 1uF, Capacitor_SMD:C_0603_1608Metric, F.Cu at (-124.6, 57.6)
- added C18: 1uF, Capacitor_SMD:C_0603_1608Metric, F.Cu at (-124.6, 60.1)
- added C19: 1uF, Capacitor_SMD:C_0603_1608Metric, F.Cu at (-124.6, 62.6)
- added C2: 1uF, Capacitor_SMD:C_0603_1608Metric, F.Cu at (-128.6, 42.6)
- added C20: 1uF, Capacitor_SMD:C_0603_1608Metric, F.Cu at (-120.6, 42.6)
- added C21: 1uF, Capacitor_SMD:C_0603_1608Metric, F.Cu at (-120.6, 45.1)
- added C22: 1uF, Capacitor_SMD:C_0603_1608Metric, F.Cu at (-120.6, 47.6)
- added C23: 1uF, Capacitor_SMD:C_0603_1608Metric, F.Cu at (-120.6, 50.1)
- added C24: 1uF, Capacitor_SMD:C_0603_1608Metric, F.Cu at (-120.6, 52.6)
- added C25: 1uF, Capacitor_SMD:C_0603_1608Metric, F.Cu at (-120.6, 55.1)
- added C26: 1uF, Capacitor_SMD:C_0603_1608Metric, F.Cu at (-120.6, 57.6)
- added C27: 1uF, Capacitor_SMD:C_0603_1608Metric, F.Cu at (-120.6, 60.1)
- added C28: 1uF, Capacitor_SMD:C_0603_1608Metric, F.Cu at (-120.6, 62.6)
- added C29: 1uF, Capacitor_SMD:C_0603_1608Metric, F.Cu at (-116.6, 42.6)
- added C3: 1uF, Capacitor_SMD:C_0603_1608Metric, F.Cu at (-128.6, 45.1)
- added C30: 1uF, Capacitor_SMD:C_0603_1608Metric, F.Cu at (-116.6, 45.1)
- added C31: 1uF, Capacitor_SMD:C_0603_1608Metric, F.Cu at (-116.6, 47.6)
- added C32: 1uF, Capacitor_SMD:C_0603_1608Metric, F.Cu at (-116.6, 50.1)
- added C4: 1uF, Capacitor_SMD:C_0603_1608Metric, F.Cu at (-128.6, 47.6)
- added C5: 1uF, Capacitor_SMD:C_0603_1608Metric, F.Cu at (-128.6, 50.1)
- added C6: 1uF, Capacitor_SMD:C_0603_1608Metric, F.Cu at (-128.6, 52.6)
- added C7: 1uF, Capacitor_SMD:C_0603_1608Metric, F.Cu at (-128.6, 55.1)
- added C8: 1uF, Capacitor_SMD:C_0603_1608Metric, F.Cu at (-128.6, 57.6)
- added C9: 1uF, Capacitor_SMD:C_0603_1608Metric, F.Cu at (-128.6, 60.1)
- added L1: 10µH, Inductor_SMD:L_0805_2012Metric, F.Cu at (111.9, 166.9)
- added L1: 10µH, Inductor_SMD:L_0805_2012Metric, F.Cu at (63.7, 91.3)
- added L1: 10µH, Inductor_SMD:L_0805_2012Metric, F.Cu at (74.8, 71.6)
- added L1: 10µH, Inductor_SMD:L_0805_2012Metric, F.Cu at (90.4, 159.9)
- added L1: 10µH, Inductor_SMD:L_0805_2012Metric, F.Cu at (103.2, 53.5)
- added L1: 10µH, Inductor_SMD:L_0805_2012Metric, F.Cu at (136.8, 54.2)
- added L1: 10µH, Inductor_SMD:L_0805_2012Metric, F.Cu at (125.7, 51.8)
- added L1: 10µH, Inductor_SMD:L_0805_2012Metric, F.Cu at (61.2, 102.4)
- added L1: 10µH, Inductor_SMD:L_0805_2012Metric, F.Cu at (145.0, 161.1)
- added L1: 10µH, Inductor_SMD:L_0805_2012Metric, F.Cu at (83.0, 63.7)
- added L1: 10µH, Inductor_SMD:L_0805_2012Metric, F.Cu at (156.6, 65.3)
- added L1: 10µH, Inductor_SMD:L_0805_2012Metric, F.Cu at (67.1, 135.6)
- added L1: 10µH, Inductor_SMD:L_0805_2012Metric, F.Cu at (68.3, 80.9)
- added L1: 10µH, Inductor_SMD:L_0805_2012Metric, F.Cu at (123.3, 167.2)
- added L1: 10µH, Inductor_SMD:L_0805_2012Metric, F.Cu at (164.4, 73.5)
- added L1: 10µH, Inductor_SMD:L_0805_2012Metric, F.Cu at (114.4, 51.5)
- added L1: 10µH, Inductor_SMD:L_0805_2012Metric, F.Cu at (81.1, 153.4)
- added L1: 10µH, Inductor_SMD:L_0805_2012Metric, F.Cu at (169.4, 137.8)
- added L1: 10µH, Inductor_SMD:L_0805_2012Metric, F.Cu at (162.0, 146.5)
- added L1: 10µH, Inductor_SMD:L_0805_2012Metric, F.Cu at (154.4, 154.7)
- added L1: 10µH, Inductor_SMD:L_0805_2012Metric, F.Cu at (174.7, 93.7)
- added L1: 10µH, Inductor_SMD:L_0805_2012Metric, F.Cu at (92.6, 57.6)
- added L1: 10µH, Inductor_SMD:L_0805_2012Metric, F.Cu at (61.0, 113.8)
- added L1: 10µH, Inductor_SMD:L_0805_2012Metric, F.Cu at (73.2, 145.2)
- added L1: 10µH, Inductor_SMD:L_0805_2012Metric, F.Cu at (134.5, 165.2)
- added L1: 10µH, Inductor_SMD:L_0805_2012Metric, F.Cu at (173.9, 127.4)
- added L1: 10µH, Inductor_SMD:L_0805_2012Metric, F.Cu at (63.0, 125.0)
- added L1: 10µH, Inductor_SMD:L_0805_2012Metric, F.Cu at (176.6, 104.9)
- added L1: 10µH, Inductor_SMD:L_0805_2012Metric, F.Cu at (147.2, 58.8)
- added L1: 10µH, Inductor_SMD:L_0805_2012Metric, F.Cu at (170.5, 83.1)
- added L1: 10µH, Inductor_SMD:L_0805_2012Metric, F.Cu at (100.8, 164.5)
- added L1: 10µH, Inductor_SMD:L_0805_2012Metric, F.Cu at (176.4, 116.3)
- added LED1: WHITE 3528, LED_SMD:LED_0201_0603Metric, F.Cu at (140.2, 59.2)
- added LED1: WHITE 3528, LED_SMD:LED_0201_0603Metric, F.Cu at (162.7, 139.0)
- added LED1: WHITE 3528, LED_SMD:LED_0201_0603Metric, F.Cu at (147.4, 153.2)
- added LED1: WHITE 3528, LED_SMD:LED_0201_0603Metric, F.Cu at (74.7, 77.7)
- added LED1: WHITE 3528, LED_SMD:LED_0201_0603Metric, F.Cu at (81.5, 69.7)
- added LED1: WHITE 3528, LED_SMD:LED_0201_0603Metric, F.Cu at (157.3, 71.2)
- added LED1: WHITE 3528, LED_SMD:LED_0201_0603Metric, F.Cu at (149.3, 64.4)
- added LED1: WHITE 3528, LED_SMD:LED_0201_0603Metric, F.Cu at (73.5, 137.3)
- added LED1: WHITE 3528, LED_SMD:LED_0201_0603Metric, F.Cu at (130.2, 56.0)
- added LED1: WHITE 3528, LED_SMD:LED_0201_0603Metric, F.Cu at (119.7, 54.8)
- added LED1: WHITE 3528, LED_SMD:LED_0201_0603Metric, F.Cu at (171.1, 119.9)
- added LED1: WHITE 3528, LED_SMD:LED_0201_0603Metric, F.Cu at (128.1, 161.2)
- added LED1: WHITE 3528, LED_SMD:LED_0201_0603Metric, F.Cu at (66.3, 96.9)
- added LED1: WHITE 3528, LED_SMD:LED_0201_0603Metric, F.Cu at (163.8, 79.4)
- added LED1: WHITE 3528, LED_SMD:LED_0201_0603Metric, F.Cu at (68.8, 128.0)
- added LED1: WHITE 3528, LED_SMD:LED_0201_0603Metric, F.Cu at (155.0, 146.4)
- added LED1: WHITE 3528, LED_SMD:LED_0201_0603Metric, F.Cu at (167.8, 129.9)
- added LED1: WHITE 3528, LED_SMD:LED_0201_0603Metric, F.Cu at (99.1, 58.5)
- added LED1: WHITE 3528, LED_SMD:LED_0201_0603Metric, F.Cu at (88.0, 152.4)
- added LED1: WHITE 3528, LED_SMD:LED_0201_0603Metric, F.Cu at (69.5, 86.9)
- added LED1: WHITE 3528, LED_SMD:LED_0201_0603Metric, F.Cu at (117.7, 162.0)
- added LED1: WHITE 3528, LED_SMD:LED_0201_0603Metric, F.Cu at (65.9, 117.8)
- added LED1: WHITE 3528, LED_SMD:LED_0201_0603Metric, F.Cu at (97.2, 157.5)
- added LED1: WHITE 3528, LED_SMD:LED_0201_0603Metric, F.Cu at (138.3, 158.3)
- added LED1: WHITE 3528, LED_SMD:LED_0201_0603Metric, F.Cu at (65.1, 107.4)
- added LED1: WHITE 3528, LED_SMD:LED_0201_0603Metric, F.Cu at (80.0, 145.6)
- added LED1: WHITE 3528, LED_SMD:LED_0201_0603Metric, F.Cu at (109.2, 55.6)
- added LED1: WHITE 3528, LED_SMD:LED_0201_0603Metric, F.Cu at (171.5, 98.9)
- added LED1: WHITE 3528, LED_SMD:LED_0201_0603Metric, F.Cu at (89.7, 63.2)
- added LED1: WHITE 3528, LED_SMD:LED_0201_0603Metric, F.Cu at (168.6, 88.8)
- added LED1: WHITE 3528, LED_SMD:LED_0201_0603Metric, F.Cu at (107.2, 160.8)
- added LED1: WHITE 3528, LED_SMD:LED_0201_0603Metric, F.Cu at (172.3, 109.4)
- added LED10: WHITE 3528, LED_SMD:LED_0201_0603Metric, F.Cu at (-126.5, 86.8)
- added LED11: WHITE 3528, LED_SMD:LED_0201_0603Metric, F.Cu at (-126.5, 88.5)
- added LED12: WHITE 3528, LED_SMD:LED_0201_0603Metric, F.Cu at (-126.5, 90.3)
- added LED13: WHITE 3528, LED_SMD:LED_0201_0603Metric, F.Cu at (-126.5, 92.0)
- added LED14: WHITE 3528, LED_SMD:LED_0201_0603Metric, F.Cu at (-126.5, 93.8)
- added LED15: WHITE 3528, LED_SMD:LED_0201_0603Metric, F.Cu at (-126.5, 95.5)
- added LED16: WHITE 3528, LED_SMD:LED_0201_0603Metric, F.Cu at (-126.5, 97.3)
- added LED17: WHITE 3528, LED_SMD:LED_0201_0603Metric, F.Cu at (-126.5, 99.0)
- added LED18: WHITE 3528, LED_SMD:LED_0201_0603Metric, F.Cu at (-123.8, 86.8)
- added LED19: WHITE 3528, LED_SMD:LED_0201_0603Metric, F.Cu at (-123.8, 88.5)
- added LED2: WHITE 3528, LED_SMD:LED_0201_0603Metric, F.Cu at (-129.1, 86.8)
- added LED20: WHITE 3528, LED_SMD:LED_0201_0603Metric, F.Cu at (-123.8, 90.3)
- added LED21: WHITE 3528, LED_SMD:LED_0201_0603Metric, F.Cu at (-123.8, 92.0)
- added LED22: WHITE 3528, LED_SMD:LED_0201_0603Metric, F.Cu at (-123.8, 93.8)
- added LED23: WHITE 3528, LED_SMD:LED_0201_0603Metric, F.Cu at (-123.8, 95.5)
- added LED24: WHITE 3528, LED_SMD:LED_0201_0603Metric, F.Cu at (-123.8, 97.3)
- added LED25: WHITE 3528, LED_SMD:LED_0201_0603Metric, F.Cu at (-123.8, 99.0)
- added LED26: WHITE 3528, LED_SMD:LED_0201_0603Metric, F.Cu at (-121.1, 86.8)
- added LED27: WHITE 3528, LED_SMD:LED_0201_0603Metric, F.Cu at (-121.1, 88.5)
- added LED28: WHITE 3528, LED_SMD:LED_0201_0603Metric, F.Cu at (-121.1, 90.3)
- added LED29: WHITE 3528, LED_SMD:LED_0201_0603Metric, F.Cu at (-121.1, 92.0)
- added LED3: WHITE 3528, LED_SMD:LED_0201_0603Metric, F.Cu at (-129.1, 88.5)
- added LED30: WHITE 3528, LED_SMD:LED_0201_0603Metric, F.Cu at (-121.1, 93.8)
- added LED31: WHITE 3528, LED_SMD:LED_0201_0603Metric, F.Cu at (-121.1, 95.5)
- added LED32: WHITE 3528, LED_SMD:LED_0201_0603Metric, F.Cu at (-121.1, 97.3)
- added LED4: WHITE 3528, LED_SMD:LED_0201_0603Metric, F.Cu at (-129.1, 90.3)
- added LED5: WHITE 3528, LED_SMD:LED_0201_0603Metric, F.Cu at (-129.1, 92.0)
- added LED6: WHITE 3528, LED_SMD:LED_0201_0603Metric, F.Cu at (-129.1, 93.8)
- added LED7: WHITE 3528, LED_SMD:LED_0201_0603Metric, F.Cu at (-129.1, 95.5)
- added LED8: WHITE 3528, LED_SMD:LED_0201_0603Metric, F.Cu at (-129.1, 97.3)
- added LED9: WHITE 3528, LED_SMD:LED_0201_0603Metric, F.Cu at (-129.1, 99.0)
- added R1: 0R39, Resistor_SMD:R_0603_1608Metric, F.Cu at (148.0, 63.5)
- added R1: 0R39, Resistor_SMD:R_0603_1608Metric, F.Cu at (74.4, 138.7)
- added R1: 0R39, Resistor_SMD:R_0603_1608Metric, F.Cu at (108.8, 161.1)
- added R1: 0R39, Resistor_SMD:R_0603_1608Metric, F.Cu at (168.0, 87.3)
- added R1: 0R39, Resistor_SMD:R_0603_1608Metric, F.Cu at (88.4, 64.1)
- added R1: 0R39, Resistor_SMD:R_0603_1608Metric, F.Cu at (97.6, 59.1)
- added R1: 0R39, Resistor_SMD:R_0603_1608Metric, F.Cu at (128.6, 55.7)
- added R1: 0R39, Resistor_SMD:R_0603_1608Metric, F.Cu at (66.2, 119.4)
- added R1: 0R39, Resistor_SMD:R_0603_1608Metric, F.Cu at (80.3, 70.9)
- added R1: 0R39, Resistor_SMD:R_0603_1608Metric, F.Cu at (119.3, 162.0)
- added R1: 0R39, Resistor_SMD:R_0603_1608Metric, F.Cu at (139.8, 157.7)
- added R1: 0R39, Resistor_SMD:R_0603_1608Metric, F.Cu at (162.9, 78.1)
- added R1: 0R39, Resistor_SMD:R_0603_1608Metric, F.Cu at (118.1, 54.8)
- added R1: 0R39, Resistor_SMD:R_0603_1608Metric, F.Cu at (81.2, 146.7)
- added R1: 0R39, Resistor_SMD:R_0603_1608Metric, F.Cu at (68.9, 88.4)
- added R1: 0R39, Resistor_SMD:R_0603_1608Metric, F.Cu at (66.0, 98.5)
- added R1: 0R39, Resistor_SMD:R_0603_1608Metric, F.Cu at (65.1, 109.0)
- added R1: 0R39, Resistor_SMD:R_0603_1608Metric, F.Cu at (171.4, 118.3)
- added R1: 0R39, Resistor_SMD:R_0603_1608Metric, F.Cu at (98.7, 158.2)
- added R1: 0R39, Resistor_SMD:R_0603_1608Metric, F.Cu at (172.3, 107.8)
- added R1: 0R39, Resistor_SMD:R_0603_1608Metric, F.Cu at (107.6, 55.9)
- added R1: 0R39, Resistor_SMD:R_0603_1608Metric, F.Cu at (138.7, 58.6)
- added R1: 0R39, Resistor_SMD:R_0603_1608Metric, F.Cu at (89.4, 153.3)
- added R1: 0R39, Resistor_SMD:R_0603_1608Metric, F.Cu at (168.5, 128.4)
- added R1: 0R39, Resistor_SMD:R_0603_1608Metric, F.Cu at (156.2, 70.0)
- added R1: 0R39, Resistor_SMD:R_0603_1608Metric, F.Cu at (148.7, 152.3)
- added R1: 0R39, Resistor_SMD:R_0603_1608Metric, F.Cu at (171.2, 97.3)
- added R1: 0R39, Resistor_SMD:R_0603_1608Metric, F.Cu at (73.8, 79.1)
- added R1: 0R39, Resistor_SMD:R_0603_1608Metric, F.Cu at (69.4, 129.5)
- added R1: 0R39, Resistor_SMD:R_0603_1608Metric, F.Cu at (163.6, 137.7)
- added R1: 0R39, Resistor_SMD:R_0603_1608Metric, F.Cu at (156.1, 145.3)
- added R1: 0R39, Resistor_SMD:R_0603_1608Metric, F.Cu at (129.7, 160.9)
- added R10: 0R39, Resistor_SMD:R_0603_1608Metric, F.Cu at (-112.6, 50.1)
- added R11: 0R39, Resistor_SMD:R_0603_1608Metric, F.Cu at (-112.6, 52.6)
- added R12: 0R39, Resistor_SMD:R_0603_1608Metric, F.Cu at (-112.6, 55.1)
- added R13: 0R39, Resistor_SMD:R_0603_1608Metric, F.Cu at (-112.6, 57.6)
- added R14: 0R39, Resistor_SMD:R_0603_1608Metric, F.Cu at (-112.6, 60.1)
- added R15: 0R39, Resistor_SMD:R_0603_1608Metric, F.Cu at (-112.6, 62.6)
- added R16: 0R39, Resistor_SMD:R_0603_1608Metric, F.Cu at (-108.5, 42.6)
- added R17: 0R39, Resistor_SMD:R_0603_1608Metric, F.Cu at (-108.5, 45.1)
- added R18: 0R39, Resistor_SMD:R_0603_1608Metric, F.Cu at (-108.5, 47.6)
- added R19: 0R39, Resistor_SMD:R_0603_1608Metric, F.Cu at (-108.5, 50.1)
- added R2: 0R39, Resistor_SMD:R_0603_1608Metric, F.Cu at (-116.6, 52.6)
- added R20: 0R39, Resistor_SMD:R_0603_1608Metric, F.Cu at (-108.5, 52.6)
- added R21: 0R39, Resistor_SMD:R_0603_1608Metric, F.Cu at (-108.5, 55.1)
- added R22: 0R39, Resistor_SMD:R_0603_1608Metric, F.Cu at (-108.5, 57.6)
- added R23: 0R39, Resistor_SMD:R_0603_1608Metric, F.Cu at (-108.5, 60.1)
- added R24: 0R39, Resistor_SMD:R_0603_1608Metric, F.Cu at (-108.5, 62.6)
- added R25: 0R39, Resistor_SMD:R_0603_1608Metric, F.Cu at (-104.5, 42.6)
- added R26: 0R39, Resistor_SMD:R_0603_1608Metric, F.Cu at (-104.5, 45.1)
- added R27: 0R39, Resistor_SMD:R_0603_1608Metric, F.Cu at (-104.5, 47.6)
- added R28: 0R39, Resistor_SMD:R_0603_1608Metric, F.Cu at (-104.5, 50.1)
- added R29: 0R39, Resistor_SMD:R_0603_1608Metric, F.Cu at (-104.5, 52.6)
- added R3: 0R39, Resistor_SMD:R_0603_1608Metric, F.Cu at (-116.6, 55.1)
- added R30: 0R39, Resistor_SMD:R_0603_1608Metric, F.Cu at (-104.5, 55.1)
- added R31: 0R39, Resistor_SMD:R_0603_1608Metric, F.Cu at (-104.5, 57.6)
- added R32: 0R39, Resistor_SMD:R_0603_1608Metric, F.Cu at (-104.5, 60.1)
- added R4: 0R39, Resistor_SMD:R_0603_1608Metric, F.Cu at (-116.6, 57.6)
- added R5: 0R39, Resistor_SMD:R_0603_1608Metric, F.Cu at (-116.6, 60.1)
- added R6: 0R39, Resistor_SMD:R_0603_1608Metric, F.Cu at (-116.6, 62.6)
- added R7: 0R39, Resistor_SMD:R_0603_1608Metric, F.Cu at (-112.6, 42.6)
- added R8: 0R39, Resistor_SMD:R_0603_1608Metric, F.Cu at (-112.6, 45.1)
- added R9: 0R39, Resistor_SMD:R_0603_1608Metric, F.Cu at (-112.6, 47.6)
- moved H21 222.2 mm to (-61.6, 17.9)
- moved H19 218.2 mm to (-61.6, 1.97)
- moved H20 214.7 mm to (-61.6, 9.92)
- moved H12 194.9 mm to (-69.6, 1.97)
- moved H18 191.1 mm to (-61.6, -5.98)
- moved H17 180.4 mm to (-69.6, 25.8)
- moved H15 177.1 mm to (-69.6, 17.9)
- moved H14 162.3 mm to (-69.6, 9.92)
- moved H13 149.4 mm to (-49.1, 99.0)
- moved H9 149.4 mm to (-6.91, 99.0)
- moved L18 132.2 mm to (-119.2, 65.3)
- moved L26 130.3 mm to (-114.7, 65.3)
- moved L27 130.3 mm to (-114.7, 68.0)
- moved L2 123.5 mm to (-128.3, 65.3)
- moved L3 123.5 mm to (-128.3, 68.0)
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Routing:
- net Net-(LED1-A): track 0.00 -> 262.6 mm
- net Net-(L1-Pad2): track 0.00 -> 176.1 mm
- net GNDPWR: track 0.00 -> 145.4 mm
- net /LED: track 0.00 -> 88.6 mm
Other:
- board outline added: 177.9 x 169.6 mm
- board text added: "2 Chairs Just Better"
- board text added: "两张椅子 比你好"
