File: Electrical/PCB v1/L1/l1 v1/l1 v1.kicad_pcb (KiCad board)
At the start: 2 copper layers, 177.9 x 169.6 mm, 273 parts

Commit message: wired pcb minus esp 32 wiring
to be checked by haoyuan/haojun not done 100%
Parts:
- removed C10, C11, C12, C13, C14, C15, C16, C17, C18, C19, C2, C20, C21, C22, C23, C24, C25, C26, C27, C28, C29, C3, C30, C31, C32, C4, C5, C6, C7, C8, C9: 1uF, Capacitor_SMD:C_0603_1608Metric
- removed L10, L11, L12, L13, L14, L15, L16, L17, L18, L19, L2, L20, L21, L22, L23, L24, L25, L26, L27, L28, L29, L3, L30, L31, L32, L4, L5, L6, L7, L8, L9: 10µH, Inductor_SMD:L_0805_2012Metric
- removed LED10, LED11, LED12, LED13, LED14, LED15, LED16, LED17, LED18, LED19, LED2, LED20, LED21, LED22, LED23, LED24, LED25, LED26, LED27, LED28, LED29, LED3, LED30, LED31, LED32, LED4, LED5, LED6, LED7, LED8, LED9: WHITE 3528, LED_SMD:LED_0201_0603Metric
- removed R10, R11, R12, R13, R14, R15, R16, R17, R18, R19, R2, R20, R21, R22, R23, R24, R25, R26, R27, R28, R29, R3, R30, R31, R32, R4, R5, R6, R7, R8, R9: 0R39, Resistor_SMD:R_0603_1608Metric
- added J1: Conn_01x01_Socket, Connector_Wire:SolderWirePad_1x01_SMD_1x2mm, F.Cu at (57.5, 97.7)
- added J2: Conn_01x01_Socket, Connector_Wire:SolderWire-0.5sqmm_1x01_D0.9mm_OD2.1mm, F.Cu at (95.0, 91.9)
- added LED_1: R_Photo, photoresistor:XDCR_ALS-PT19-315C_L177_TR8, F.Cu at (83.3, 71.8)
- added LED_10: R_Photo, photoresistor:XDCR_ALS-PT19-315C_L177_TR8, F.Cu at (90.5, 149.4)
- added LED_11: R_Photo, photoresistor:XDCR_ALS-PT19-315C_L177_TR8, F.Cu at (99.3, 154.0)
- added LED_12: R_Photo, photoresistor:XDCR_ALS-PT19-315C_L177_TR8, F.Cu at (108.4, 157.0)
- added LED_13: R_Photo, photoresistor:XDCR_ALS-PT19-315C_L177_TR8, F.Cu at (118.0, 158.3)
- added LED_14: R_Photo, photoresistor:XDCR_ALS-PT19-315C_L177_TR8, F.Cu at (127.7, 157.6)
- added LED_15: R_Photo, photoresistor:XDCR_ALS-PT19-315C_L177_TR8, F.Cu at (137.0, 154.5)
- added LED_16: R_Photo, photoresistor:XDCR_ALS-PT19-315C_L177_TR8, F.Cu at (145.4, 149.6)
- added LED_17: R_Photo, photoresistor:XDCR_ALS-PT19-315C_L177_TR8, F.Cu at (152.5, 143.1)
- added LED_18: R_Photo, photoresistor:XDCR_ALS-PT19-315C_L177_TR8, F.Cu at (159.6, 136.1)
- added LED_19: R_Photo, photoresistor:XDCR_ALS-PT19-315C_L177_TR8, F.Cu at (164.2, 127.4)
- added LED_2: R_Photo, photoresistor:XDCR_ALS-PT19-315C_L177_TR8, F.Cu at (77.3, 79.9)
- added LED_20: R_Photo, photoresistor:XDCR_ALS-PT19-315C_L177_TR8, F.Cu at (167.2, 118.4)
- added LED_21: R_Photo, photoresistor:XDCR_ALS-PT19-315C_L177_TR8, F.Cu at (167.9, 108.9)
- added LED_22: R_Photo, photoresistor:XDCR_ALS-PT19-315C_L177_TR8, F.Cu at (167.1, 99.3)
- added LED_23: R_Photo, photoresistor:XDCR_ALS-PT19-315C_L177_TR8, F.Cu at (164.0, 89.8)
- added LED_24: R_Photo, photoresistor:XDCR_ALS-PT19-315C_L177_TR8, F.Cu at (159.1, 80.2)
- added LED_25: R_Photo, photoresistor:XDCR_ALS-PT19-315C_L177_TR8, F.Cu at (153.7, 74.1)
- added LED_26: R_Photo, photoresistor:XDCR_ALS-PT19-315C_L177_TR8, F.Cu at (128.7, 61.6)
- added LED_27: R_Photo, photoresistor:XDCR_ALS-PT19-315C_L177_TR8, F.Cu at (119.6, 59.9)
- added LED_28: R_Photo, photoresistor:XDCR_ALS-PT19-315C_L177_TR8, F.Cu at (146.1, 68.1)
- added LED_29: R_Photo, photoresistor:XDCR_ALS-PT19-315C_L177_TR8, F.Cu at (137.8, 64.2)
- added LED_3: R_Photo, photoresistor:XDCR_ALS-PT19-315C_L177_TR8, F.Cu at (72.8, 88.9)
- added LED_30: R_Photo, photoresistor:XDCR_ALS-PT19-315C_L177_TR8, F.Cu at (109.9, 59.5)
- added LED_31: R_Photo, photoresistor:XDCR_ALS-PT19-315C_L177_TR8, F.Cu at (101.0, 62.6)
- added LED_32: R_Photo, photoresistor:XDCR_ALS-PT19-315C_L177_TR8, F.Cu at (91.4, 67.0)
- added LED_4: R_Photo, photoresistor:XDCR_ALS-PT19-315C_L177_TR8, F.Cu at (69.6, 98.5)
- added LED_5: R_Photo, photoresistor:XDCR_ALS-PT19-315C_L177_TR8, F.Cu at (68.6, 109.0)
- added LED_6: R_Photo, photoresistor:XDCR_ALS-PT19-315C_L177_TR8, F.Cu at (68.9, 118.1)
- added LED_7: R_Photo, photoresistor:XDCR_ALS-PT19-315C_L177_TR8, F.Cu at (72.0, 126.8)
- added LED_8: R_Photo, photoresistor:XDCR_ALS-PT19-315C_L177_TR8, F.Cu at (76.4, 136.4)
- added LED_9: R_Photo, photoresistor:XDCR_ALS-PT19-315C_L177_TR8, F.Cu at (82.7, 143.3)
- added SW1: SW_SPDT, Button_Switch_SMD:Nidec_Copal_CAS-120A, F.Cu at (102.8, 92.3)
- added TP1: TestPoint, TestPoint:TestPoint_2Pads_Pitch2.54mm_Drill0.8mm, F.Cu at (88.9, 87.8)
- added TP2: TestPoint, TestPoint:TestPoint_2Pads_Pitch2.54mm_Drill0.8mm, F.Cu at (87.0, 91.5)
- added U1: ESP32-WROOM-32D-N4, esp32 thinfy:MODULE_ESP32-WROOM-32D-N4, B.Cu at (117.6, 103.0)
- added U2: CD74HC4067SM, mux thingy:SOP65P780X200-24N, F.Cu at (77.8, 107.9)
- added U3: CD74HC4067SM, mux thingy:SOP65P780X200-24N, F.Cu at (155.4, 108.4)
- moved H12 243.1 mm to (155.8, 93.0)
- moved H14 207.1 mm to (126.8, 75.9)
- moved H15 186.6 mm to (107.8, 75.9)
- moved H13 184.2 mm to (132.7, 69.9)
- moved H20 181.9 mm to (84.7, 118.0)
- moved H17 177.0 mm to (101.8, 69.9)
- moved H21 175.9 mm to (78.7, 124.0)
- moved H19 175.5 mm to (84.7, 99.0)
- moved H18 171.8 mm to (78.7, 93.1)
- moved H9 158.0 mm to (149.9, 118.0)
- moved H10 19.0 mm to (149.9, 99.0)
Routing:
- net Net-(LED_1-Pad1): track 0.00 -> 299.4 mm
- net Net-(LED_17-Pad1): track 0.00 -> 179.2 mm
- net /LED: track 88.6 -> 241.1 mm
- net Net-(U2-I15): track 0.00 -> 116.3 mm, vias 0 -> 1
- net Net-(U2-I14): track 0.00 -> 90.0 mm, vias 0 -> 1
- net Net-(U3-I15): track 0.00 -> 82.7 mm
- net Net-(U2-I12): track 0.00 -> 81.4 mm, vias 0 -> 1
- net Net-(U2-I13): track 0.00 -> 81.2 mm, vias 0 -> 1
- net Net-(U3-I14): track 0.00 -> 73.1 mm
- net Net-(U2-I11): track 0.00 -> 68.5 mm, vias 0 -> 1
- net Net-(U3-I13): track 0.00 -> 68.3 mm
- net Net-(U3-I12): track 0.00 -> 68.2 mm, vias 0 -> 2
- net Net-(U3-I10): track 0.00 -> 65.4 mm
- net Net-(U3-I11): track 0.00 -> 64.3 mm
- net Net-(U3-I9): track 0.00 -> 63.7 mm
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Other:
- board text added: "2 Chairs"
- board text added: "Just Better."
- board text removed: "2 Chairs Just Better"

Commit message: gnd filled
Routing:
- net Net-(U1-IO21): track 0.00 -> 125.3 mm
- net Net-(U1-IO27): track 0.00 -> 110.8 mm, vias 0 -> 2
- net Net-(U1-IO33): track 0.00 -> 107.8 mm, vias 0 -> 2
- net Net-(U1-IO0): track 0.00 -> 55.0 mm
- net Net-(U1-IO22): track 0.00 -> 47.0 mm, vias 0 -> 1
- net Net-(U1-GND-Pad1): track 58.3 -> 100.9 mm
- net Net-(U1-RXD0): track 0.00 -> 31.8 mm
- added copper zone on B.Cu, net GND
- added copper zone on F.Cu, net GND

Commit message: wires half done to br finiished @chenyikaithegoat to wire esp32 and i do the wiring finish
Parts:
- moved J1 41.0 mm to (98.3, 101.2)
- moved LED_1 0.84 mm to (83.8, 72.5)
- turned U2 to -90 degrees
- turned U3 to -90 degrees
Connections:
- net /LED renamed pwr for photoresistors
- LED_17 pad 1: Net-(LED_17-Pad1) -> Net-(LED_1-Pad1)
- LED_18 pad 1: Net-(LED_17-Pad1) -> Net-(LED_1-Pad1)
- LED_19 pad 1: Net-(LED_17-Pad1) -> Net-(LED_1-Pad1)
- LED_20 pad 1: Net-(LED_17-Pad1) -> Net-(LED_1-Pad1)
- LED_21 pad 1: Net-(LED_17-Pad1) -> Net-(LED_1-Pad1)
- LED_22 pad 1: Net-(LED_17-Pad1) -> Net-(LED_1-Pad1)
- LED_23 pad 1: Net-(LED_17-Pad1) -> Net-(LED_1-Pad1)
- LED_24 pad 1: Net-(LED_17-Pad1) -> Net-(LED_1-Pad1)
- LED_25 pad 1: Net-(LED_17-Pad1) -> Net-(LED_1-Pad1)
- LED_26 pad 1: Net-(LED_17-Pad1) -> Net-(LED_1-Pad1)
- LED_27 pad 1: Net-(LED_17-Pad1) -> Net-(LED_1-Pad1)
- LED_28 pad 1: Net-(LED_17-Pad1) -> Net-(LED_1-Pad1)
- LED_29 pad 1: Net-(LED_17-Pad1) -> Net-(LED_1-Pad1)
- LED_30 pad 1: Net-(LED_17-Pad1) -> Net-(LED_1-Pad1)
- LED_31 pad 1: Net-(LED_17-Pad1) -> Net-(LED_1-Pad1)
- LED_32 pad 1: Net-(LED_17-Pad1) -> Net-(LED_1-Pad1)
- U1 pad 2: unconnected-(U1-3V3-Pad2) -> 3V3
- U3 pad 15: Net-(U1-IO23) -> unconnected-(U3-~{E}-Pad15)
Routing:
- net Net-(LED_1-Pad1): track 299.4 -> 573.1 mm
- net Net-(LED_17-Pad1): track 179.2 -> 0.00 mm
- net Net-(U1-IO21): track 125.3 -> 0.00 mm
- net Net-(U1-IO27): track 110.8 -> 0.00 mm, vias 2 -> 0
- net Net-(U1-IO33): track 107.8 -> 0.00 mm, vias 2 -> 0
- net pwr for photoresistors: track 241.1 -> 137.7 mm, vias 0 -> 1
- net Net-(U1-GND-Pad1): track 100.9 -> 0.00 mm
- net Net-(U3-I14): track 73.1 -> 0.00 mm
- net Net-(U3-I13): track 68.3 -> 0.00 mm
- net Net-(U3-I12): track 68.2 -> 0.00 mm, vias 2 -> 0
- net Net-(U3-I10): track 65.4 -> 0.00 mm
- net Net-(U3-I9): track 63.7 -> 0.00 mm
- net Net-(U3-I15): track 82.7 -> 19.7 mm
- net Net-(U1-IO0): track 55.0 -> 0.00 mm
- net Net-(U1-IO22): track 47.0 -> 0.00 mm, vias 1 -> 0
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- removed copper zone on B.Cu, net GND
- removed copper zone on F.Cu, net GND
