File: Electrical/PCB v1/L1/l1 v1/l1 v1.kicad_sch (KiCad schematic)
At the start: 189 parts, among them J1 Conn_01x01_Socket, J2 Conn_01x01_Socket, SW1 SW_SPDT, U1 ESP32-WROOM-32D-N4, U2 CD74HC4067SM, U3 CD74HC4067SM

Commit message: wires half done to br finiished @chenyikaithegoat to wire esp32 and i do the wiring finish
Connections:
- net at LED_1.1, LED_10.1, LED_11.1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: now also LED_17.1, LED_18.1, LED_19.1, LED_20.1, LED_21.1, LED_22.1, LED_23.1, LED_24.1, LED_25.1, LED_26.1, LED_27.1, LED_28.1, LED_29.1, LED_30.1, LED_31.1, LED_32.1
- net LED renamed pwr for photoresistors
Changed lines of the file:
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@@
+	)
+	(junction
+		(at 280.67 146.05)
+		(diameter 0)
+		(color 0 0 0 0)
 	)
 	(junction
@@
 	)
 	(junction
+		(at 210.82 143.51)
+		(diameter 0)
+		(color 0 0 0 0)
+	)
+	(junction
 		(at 184.15 72.39)
 		(diameter 0)
@@
 	(junction
 		(at 215.9 100.33)
+		(diameter 0)
+		(color 0 0 0 0)
+	)
+	(junction
+		(at 72.39 60.96)
 		(diameter 0)
 		(color 0 0 0 0)
@@
 	(wire
 		(pts
-			(xy 190.5 127) (xy 229.87 127)
-		)
-		(stroke
-			(width 0)
-			(type default)
-		)
-	)
-	(wire
-		(pts
 			(xy 160.02 100.33) (xy 167.64 100.33)
 		)
@@
 	(wire
 		(pts
+			(xy 72.39 60.96) (xy 62.23 60.96)
+		)
+		(stroke
+			(width 0)
+			(type default)
+		)
+	)
+	(wire
+		(pts
 			(xy 113.03 100.33) (xy 120.65 100.33)
 		)
@@
 	(wire
 		(pts
-			(xy 260.35 138.43) (xy 229.87 138.43)
-		)
-		(stroke
-			(width 0)
-			(type default)
-		)
-	)
-	(wire
-		(pts
 			(xy 311.15 100.33) (xy 318.77 100.33)
 		)
@@
 	(wire
 		(pts
+			(xy 210.82 143.51) (xy 210.82 121.92)
+		)
+		(stroke
+			(width 0)
+			(type default)
+		)
+	)
+	(wire
+		(pts
 			(xy 161.29 69.85) (xy 166.37 69.85)
 		)
@@
 	(wire
 		(pts
+			(xy 314.96 146.05) (xy 280.67 146.05)
+		)
+		(stroke
+			(width 0)
+			(type default)
+		)
+	)
+	(wire
+		(pts
 			(xy 74.93 55.88) (xy 80.01 55.88)
 		)
@@
 	(wire
 		(pts
+			(xy 62.23 60.96) (xy 62.23 62.23)
+		)
+		(stroke
+			(width 0)
+			(type default)
+		)
+	)
+	(wire
+		(pts
 			(xy 210.82 168.91) (xy 210.82 171.45)
 		)
@@
 	(wire
 		(pts
+			(xy 210.82 121.92) (xy 314.96 121.92)
+		)
+		(stroke
+			(width 0)
+			(type default)
+		)
+	)
+	(wire
+		(pts
 			(xy 210.82 179.07) (xy 210.82 181.61)
 		)
@@
 	(wire
 		(pts
-			(xy 72.39 62.23) (xy 72.39 59.69)
+			(xy 72.39 62.23) (xy 72.39 60.96)
 		)
 		(stroke
@@
 	(wire
 		(pts
+			(xy 72.39 60.96) (xy 72.39 59.69)
+		)
+		(stroke
+			(width 0)
+			(type default)
+		)
+	)
+	(wire
+		(pts
 			(xy 246.38 175.26) (xy 246.38 180.34)
 		)
@@
 	(wire
 		(pts
+			(xy 314.96 121.92) (xy 314.96 146.05)
+		)
+		(stroke
+			(width 0)
+			(type default)
+		)
+	)
+	(wire
+		(pts
 			(xy 190.5 135.89) (xy 190.5 127)
 		)
@@
 		(pts
 			(xy 247.65 168.91) (xy 247.65 175.26)
-		)
-		(stroke
-			(width 0)
-			(type default)
-		)
-	)
-	(wire
-		(pts
-			(xy 229.87 138.43) (xy 229.87 127)
 		)
 		(stroke
@@
 			)
 			(justify left bottom)
+		)
+	)
+	(global_label "3v3"
+		(shape input)
+		(at 260.35 138.43 90)
+		(fields_autoplaced yes)
+		(effects
+			(font
+				(size 1.27 1.27)
+			)
+			(justify left)
+		)
+		(property "Intersheetrefs" "${INTERSHEET_REFS}"
+			(at 260.35 132.0582 90)
+			(effects
+				(font
+					(size 1.27 1.27)
+				)
+				(justify left)
+				(hide yes)
+			)
+		)
+	)
+	(global_label "pwr for photoresistors"
+		(shape input)
+		(at 62.23 62.23 180)
+		(fields_autoplaced yes)
+		(effects
+			(font
+				(size 1.27 1.27)
+			)
+			(justify right)
+		)
+		(property "Intersheetrefs" "${INTERSHEET_REFS}"
+			(at 37.8365 62.23 0)
+			(effects
+				(font
+					(size 1.27 1.27)
+				)
+				(justify right)
+				(hide yes)
+			)
 		)
 	)
@@
 		)
 	)
+	(global_label "3v3"
+		(shape input)
+		(at 190.5 127 90)
+		(fields_autoplaced yes)
+		(effects
+			(font
+				(size 1.27 1.27)
+			)
+			(justify left)
+		)
+		(property "Intersheetrefs" "${INTERSHEET_REFS}"
+			(at 190.5 120.6282 90)
+			(effects
+				(font
+					(size 1.27 1.27)
+				)
+				(justify left)
+				(hide yes)
+			)
+		)
+	)
 	(global_label "3V3"
 		(shape input)
@@
 				(hide yes)
 			)
-		)
-	)
-	(global_label "3v3"
-		(shape input)
-		(at 229.87 127 90)
-		(fields_autoplaced yes)
-		(effects
-			(font
-				(size 1.27 1.27)
-			)
-			(justify left)
-		)
-		(property "Intersheetrefs" "${INTERSHEET_REFS}"
-			(at 229.87 120.6282 90)
-			(effects
-				(font
-					(size 1.27 1.27)
-				)
-				(justify left)
-				(hide yes)
-			)
