File: Electrical/PCB V2 ( 26 Nov)/L1/l1 v2/l1v2/l1v2.kicad_pcb (KiCad board)
At the start: 2 copper layers, 177.9 x 169.6 mm, 194 parts, among them J1 Conn_01x01_Socket, J2 Conn_01x01_Socket, J3 Conn_01x02, SW1 SW_SPDT, U1 102010428, U2 CD74HC4067SM, U3 CD74HC4067SM, U4 XT30UPB-M

Commit message: Update PCB V2 ( 26 Nov) before renaming
Routing:
- net GND: track 7.98 -> 4.26 mm
