File: Electrical/PCB V2 ( 26 Nov)/L1/l1 v2/l1v2/l1v2-backups/l1v2-2025-01-06_150755/l1v2.kicad_pcb (KiCad board)
At the start: 2 copper layers, 177.9 x 169.6 mm, 194 parts, among them J1 Conn_01x01_Socket, J2 Conn_01x01_Socket, J3 Conn_01x02, SW1 SW_SPDT, U1 102010428, U2 CD74HC4067SM, U3 CD74HC4067SM, U4 XT30UPB-M

Commit message: finished layer 1?
Parts:
- removed J3: Conn_01x02, Connector_PinHeader_1.00mm:PinHeader_1x02_P1.00mm_Horizontal
Connections:
- U1 pad 1: /Mux Com (1-16) -> unconnected-(U1-P26/A0/D0-Pad1)
- U1 pad 10: /S2 -> unconnected-(U1-D9/MISO/P4-Pad10)
- U1 pad 11: /S3 -> unconnected-(U1-D10/MOSI/P3-Pad11)
- U1 pad 2: /Mux Com (17-32) -> unconnected-(U1-P27/A1/D1-Pad2)
- U1 pad 5: /SDA -> unconnected-(U1-P6/SDA/D4-Pad5)
- U1 pad 6: /SCL -> unconnected-(U1-P7/SCL/D5-Pad6)
- U1 pad 8: /S0 -> unconnected-(U1-D7/CSB/P1/RX-Pad8)
- U1 pad 9: /S1 -> unconnected-(U1-D8/SCK/P2-Pad9)
- U2 pad 10: /S0 -> /Mux 1 
- U2 pad 11: /S1 -> /Mux 2
- U2 pad 13: /S3 -> /Mux 4
- U2 pad 14: /S2 -> /Mux 3
- U2 pad 15: /Mux Com (1-16) -> unconnected-(U2-~{E}-Pad15)
- U3 pad 1: /Mux Com (17-32) -> unconnected-(U3-COM-Pad1)
- U3 pad 10: /S0 -> /Mux 8
- U3 pad 11: /S1 -> /Mux 7
- U3 pad 13: /S3 -> /Mux 5
- U3 pad 14: /S2 -> /Mux 6
Routing:
- net /S3: track 114.4 -> 0.00 mm, vias 3 -> 0
- net /S2: track 111.4 -> 0.00 mm, vias 3 -> 0
- net /Mux Com (1-16): track 102.3 -> 0.00 mm, vias 1 -> 0
- net /S1: track 93.8 -> 0.00 mm, vias 1 -> 0
- net /S0: track 87.3 -> 0.00 mm, vias 1 -> 0
- net /Mux Com (17-32): track 76.2 -> 0.00 mm, vias 1 -> 0
- net /SCL: track 9.44 -> 0.00 mm
- net /SDA: track 8.00 -> 0.00 mm
- net unconnected-(U1-P28/A2/D2-Pad3): track 1.50 -> 0.00 mm
- net unconnected-(U1-P0//TX/D6-Pad7): track 1.34 -> 0.00 mm
Other:
- board text removed: "2-Chairs"
- board text removed: "Layer 1"
