File: Electrical/PCB V2 ( 26 Nov)/L1/l1 v2/l1v2/l1v2-backups/l1v2-2025-01-06_150755/l1v2.kicad_sch (KiCad schematic)
At the start: 194 parts, among them J1 Conn_01x01_Socket, J2 Conn_01x01_Socket, J3 Conn_01x02, SW1 SW_SPDT, U1 102010428, U2 CD74HC4067SM, U3 CD74HC4067SM, U4 XT30UPB-M

Commit message: finished layer 1?
Parts:
- removed J3: Conn_01x02, Connector_PinHeader_1.00mm:PinHeader_1x02_P1.00mm_Horizontal, symbol Connector_Generic:Conn_01x02
Connections:
- net Mux Com (1-16): no longer names the net of U2.15 (~{E})
- net Mux Com (1-16): no longer U1.1 (P26/A0/D0)
- net Mux Com (17-32): no longer names the net of U3.1 (COM)
- net Mux Com (17-32): no longer U1.2 (P27/A1/D1)
- removed net S0: U1.8 (D7/CSB/P1/RX), U2.10 (S0), U3.10 (S0)
- removed net S1: U1.9 (D8/SCK/P2), U2.11 (S1), U3.11 (S1)
- removed net S2: U1.10 (D9/MISO/P4), U2.14 (S2), U3.14 (S2)
- removed net S3: U1.11 (D10/MOSI/P3), U2.13 (S3), U3.13 (S3)
- net SCL: no longer names the net of U1.6 (P7/SCL/D5)
- net SDA: no longer names the net of U1.5 (P6/SDA/D4)
- new net Mux 1 : U2.10 (S0)
- new net Mux 2: U2.11 (S1)
- new net Mux 3: U2.14 (S2)
- new net Mux 4: U2.13 (S3)
- new net Mux 5: U3.13 (S3)
- new net Mux 6: U3.14 (S2)
- new net Mux 7: U3.11 (S1)
- new net Mux 8: U3.10 (S0)
- no-connect marks 9 -> 11
Changed lines of the file:
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@@
 	)
 	(no_connect
-		(at 177.8 170.18)
+		(at 251.46 213.36)
 	)
 	(no_connect
-		(at 198.12 218.44)
+		(at 177.8 170.18)
 	)
 	(no_connect
@@
 	)
 	(no_connect
+		(at 247.65 179.07)
+	)
+	(no_connect
 		(at 251.46 203.2)
 	)
@@
 	)
 	(no_connect
-		(at 198.12 226.06)
+		(at 251.46 218.44)
 	)
 	(no_connect
-		(at 198.12 215.9)
+		(at 209.55 180.34)
+	)
+	(no_connect
+		(at 251.46 215.9)
 	)
 	(wire
@@
 	(wire
 		(pts
+			(xy 209.55 165.1) (xy 213.36 165.1)
+		)
+		(stroke
+			(width 0)
+			(type default)
+		)
+	)
+	(wire
+		(pts
 			(xy 176.53 152.4) (xy 176.53 149.86)
 		)
@@
 	(wire
 		(pts
+			(xy 209.55 167.64) (xy 215.9 167.64)
+		)
+		(stroke
+			(width 0)
+			(type default)
+		)
+	)
+	(wire
+		(pts
 			(xy 176.53 170.18) (xy 176.53 167.64)
 		)
@@
 	(wire
 		(pts
-			(xy 209.55 167.64) (xy 217.17 167.64)
-		)
-		(stroke
-			(width 0)
-			(type default)
-		)
-	)
-	(wire
-		(pts
 			(xy 113.03 100.33) (xy 120.65 100.33)
 		)
@@
 	(wire
 		(pts
-			(xy 120.65 69.85) (xy 125.73 69.85)
+			(xy 209.55 170.18) (xy 218.44 170.18)
 		)
 		(stroke
@@
 	(wire
 		(pts
-			(xy 209.55 162.56) (xy 212.09 162.56)
+			(xy 120.65 69.85) (xy 125.73 69.85)
 		)
 		(stroke
@@
 	(wire
 		(pts
-			(xy 209.55 165.1) (xy 214.63 165.1)
-		)
-		(stroke
-			(width 0)
-			(type default)
-		)
-	)
-	(wire
-		(pts
 			(xy 72.39 62.23) (xy 80.01 62.23)
 		)
@@
 	(wire
 		(pts
-			(xy 209.55 170.18) (xy 219.71 170.18)
-		)
-		(stroke
-			(width 0)
-			(type default)
-		)
-	)
-	(wire
-		(pts
 			(xy 128.27 100.33) (xy 135.89 100.33)
 		)
@@
 	(wire
 		(pts
+			(xy 210.82 162.56) (xy 209.55 162.56)
+		)
+		(stroke
+			(width 0)
+			(type default)
+		)
+	)
+	(wire
+		(pts
 			(xy 72.39 60.96) (xy 72.39 59.69)
 		)
@@
 		)
 	)
-	(label "S3"
-		(at 212.09 162.56 90)
+	(label "Mux 8"
+		(at 218.44 170.18 90)
 		(fields_autoplaced yes)
 		(effects
@@
 		)
 	)
-	(label "Mux Com (17-32)"
-		(at 209.55 180.34 0)
+	(label "Mux 6"
+		(at 213.36 165.1 90)
 		(fields_autoplaced yes)
 		(effects
@@
 		)
 	)
-	(label "S0"
-		(at 219.71 170.18 90)
-		(fields_autoplaced yes)
-		(effects
-			(font
-				(size 1.27 1.27)
-			)
-			(justify left bottom)
-		)
-	)
-	(label "Mux Com (1-16)"
-		(at 198.12 210.82 180)
-		(fields_autoplaced yes)
-		(effects
-			(font
-				(size 1.27 1.27)
-			)
-			(justify right bottom)
-		)
-	)
 	(label "LED"
 		(at 91.44 53.34 0)
@@
 		)
 	)
-	(label "S2"
+	(label "Mux 3"
 		(at 245.11 166.37 90)
 		(fields_autoplaced yes)
@@
 		)
 	)
-	(label "S1"
-		(at 217.17 167.64 90)
-		(fields_autoplaced yes)
-		(effects
-			(font
-				(size 1.27 1.27)
-			)
-			(justify left bottom)
-		)
-	)
-	(label "S0"
+	(label "Mux 1 "
 		(at 240.03 161.29 90)
 		(fields_autoplaced yes)
@@
 		)
 	)
-	(label "SDA"
-		(at 162.56 218.44 0)
-		(fields_autoplaced yes)
-		(effects
-			(font
-				(size 1.27 1.27)
-			)
-			(justify left bottom)
-		)
-	)
-	(label "S3"
-		(at 251.46 213.36 0)
-		(fields_autoplaced yes)
-		(effects
-			(font
-				(size 1.27 1.27)
-			)
-			(justify left bottom)
-		)
-	)
-	(label "S1"
-		(at 251.46 218.44 0)
-		(fields_autoplaced yes)
-		(effects
-			(font
-				(size 1.27 1.27)
-			)
-			(justify left bottom)
-		)
-	)
-	(label "S3"
+	(label "Mux 4"
 		(at 247.65 168.91 90)
 		(fields_autoplaced yes)
@@
 		)
 	)
-	(label "S0"
-		(at 251.46 220.98 0)
-		(fields_autoplaced yes)
-		(effects
-			(font
-				(size 1.27 1.27)
-			)
-			(justify left bottom)
-		)
-	)
-	(label "S2"
-		(at 251.46 215.9 0)
-		(fields_autoplaced yes)
-		(effects
-			(font
-				(size 1.27 1.27)
-			)
-			(justify left bottom)
-		)
-	)
-	(label "SCL"
-		(at 162.56 220.98 0)
-		(fields_autoplaced yes)
-		(effects
-			(font
-				(size 1.27 1.27)
-			)
-			(justify left bottom)
-		)
-	)
 	(label "LED"
 		(at 109.22 57.15 0)
@@
 		)
 	)
-	(label "SCL"
-		(at 198.12 223.52 180)
+	(label "Mux 7"
+		(at 215.9 167.64 90)
 		(fields_autoplaced yes)
 		(effects
@@
 				(size 1.27 1.27)
 			)
-			(justify right bottom)
+			(justify left bottom)
 		)
 	)
-	(label "S1"
+	(label "Mux 2"
 		(at 242.57 163.83 90)
 		(fields_autoplaced yes)
@@
 		)
 	)
-	(label "Mux Com (17-32)"
-		(at 198.12 213.36 180)
-		(fields_autoplaced yes)
-		(effects
-			(font
-				(size 1.27 1.27)
-			)
-			(justify right bottom)
-		)
-	)
-	(label "S2"
-		(at 214.63 165.1 90)
+	(label "Mux 5"
+		(at 210.82 162.56 90)
 		(fields_autoplaced yes)
 		(effects
@@
 		)
 	)
-	(label "SDA"
-		(at 198.12 220.98 180)
-		(fields_autoplaced yes)
-		(effects
-			(font
-				(size 1.27 1.27)
-			)
-			(justify right bottom)
-		)
-	)
-	(label "Mux Com (1-16)"
-		(at 247.65 179.07 180)
-		(fields_autoplaced yes)
-		(effects
-			(font
-				(size 1.27 1.27)
-			)
-			(justify right bottom)
-		)
-	)
 	(global_label "GND"
 		(shape input)
@@
 					(unit 1)
 				)
-			)
-		)
-	)
-	(symbol
-		(lib_id "Connector_Generic:Conn_01x02")
-		(at 157.48 220.98 180)
-		(unit 1)
-		(exclude_from_sim no)
-		(in_bom yes)
-		(on_board yes)
-		(dnp no)
-		(fields_autoplaced yes)
-		(property "Reference" "J3"
-			(at 157.48 212.09 0)
-			(effects
-				(font
-					(size 1.27 1.27)
-				)
-			)
-		)
-		(property "Value" "Conn_01x02"
-			(at 157.48 214.63 0)
-			(effects
-				(font
-					(size 1.27 1.27)
-				)
-			)
-		)
-		(property "Footprint" "Connector_PinHeader_1.00mm:PinHeader_1x02_P1.00mm_Horizontal"
-			(at 157.48 220.98 0)
-			(effects
-				(font
-					(size 1.27 1.27)
-				)
-				(hide yes)
-			)
-		)
-		(property "Datasheet" "~"
-			(at 157.48 220.98 0)
-			(effects
-				(font
-					(size 1.27 1.27)
-				)
-				(hide yes)
-			)
-		)
-		(property "Description" "Generic connector, single row, 01x02, script generated (kicad-library-utils/schlib/autogen/connector/)"
-			(at 157.48 220.98 0)
-			(effects
-				(font
-					(size 1.27 1.27)
-				)
-				(hide yes)
-			)
-		)
-		(pin "1"
-		)
-		(pin "2"
-		)
-		(instances
-			(project ""
-				(path "/9e8a7821-ee65-4356-a785-1f444d794ef4"
-					(reference "J3")
-					(unit 1)
-				)
