File: Electrical/PCB V2 ( 26 Nov)/L2/Layer_2/Layer_2.kicad_pcb (KiCad board)
At the start: 2 copper layers, 0 parts

Commit message: hehe
Parts:
- added L298N1: ~, l298n:TO127P2020X500X2100-15, F.Cu at (244.9, 52.7)
- added L298N2: ~, l298n:TO127P2020X500X2100-15, F.Cu at (246.1, 125.1)
- added SW1: SW_Push, flipswitch:SW_100SP1T1B4M2QE, F.Cu at (247.8, 98.3)
- added U1: LM2596ADJ, Motor Controller:LM2596ADJ, F.Cu at (249.0, 83.8)
- added U2: LM2596ADJ, Motor Controller:LM2596ADJ, F.Cu at (260.8, 83.8)
- added U3: XT30UPB-M, xt30:XT30UPB-M, F.Cu at (237.5, 78.2)
- added U4: XT30UPB-M, xt30:XT30UPB-M, F.Cu at (237.5, 84.6)
- added U5: ESP32-S3-DEVKITM-1-N8, ESP32 DEV KIT:MODULE_ESP32-S3-DEVKITM-1-N8, F.Cu at (218.4, 111.9)
- added U6: XT30UPB-M, xt30:XT30UPB-M, F.Cu at (237.5, 90.9)
- added U7: XT30UPB-M, xt30:XT30UPB-M, F.Cu at (237.5, 97.2)
- added U8: XT30UPB-M, xt30:XT30UPB-M, F.Cu at (237.5, 103.6)
- added U9: XT30UPB-M, xt30:XT30UPB-M, F.Cu at (237.5, 109.9)

Commit message: xt30 added
Parts:
- added H1: MountingHole, MountingHole:MountingHole_3.2mm_M3_DIN965_Pad, F.Cu at (80.5, 29.0)
- added H10: MountingHole, MountingHole:MountingHole_3.2mm_M3_DIN965_Pad, F.Cu at (184.5, 133.0)
- added H11: MountingHole, MountingHole:MountingHole_3.2mm_M3_DIN965_Pad, F.Cu at (184.5, 83.0)
- added H12: MountingHole, MountingHole:MountingHole_3.2mm_M3_DIN965_Pad, F.Cu at (130.5, 29.0)
- added H2: MountingHole, MountingHole:MountingHole_3.2mm_M3_DIN965_Pad, F.Cu at (26.5, 83.0)
- added H3: MountingHole, MountingHole:MountingHole_3.2mm_M3_DIN965_Pad, F.Cu at (26.5, 133.0)
- added H4: MountingHole, MountingHole:MountingHole_3.2mm_M3_DIN965_Pad, F.Cu at (82.0, 169.8)
- added H5: MountingHole, MountingHole:MountingHole_3.2mm_M3_DIN965_Pad, F.Cu at (102.0, 149.4)
- added H6: MountingHole, MountingHole:MountingHole_3.2mm_M3_DIN965_Pad, F.Cu at (102.0, 173.0)
- added H7: MountingHole, MountingHole:MountingHole_3.2mm_M3_DIN965_Pad, F.Cu at (109.0, 149.4)
- added H8: MountingHole, MountingHole:MountingHole_3.2mm_M3_DIN965_Pad, F.Cu at (109.0, 173.0)
- added H9: MountingHole, MountingHole:MountingHole_3.2mm_M3_DIN965_Pad, F.Cu at (129.0, 169.7)
- added U10, U11, U12: XT30UPB-M, xt30:XT30UPB-M, F.Cu at (107.6, 66.1)
- moved L298N2 226.3 mm to (21.4, 98.0)
- moved U7 181.8 mm to (55.9, 105.9), turned to 95 degrees
- moved U1 179.1 mm to (71.4, 106.5)
- moved U4 139.2 mm to (108.1, 135.7)
- moved U3 130.5 mm to (107.6, 66.1)
- moved U9 130.0 mm to (107.5, 112.7)
- moved U8 129.2 mm to (108.8, 92.1)
- moved U2 123.1 mm to (139.8, 106.6)
- moved L298N1 83.7 mm to (188.5, 114.6)
- moved U6 78.1 mm to (160.6, 104.2), turned to 90 degrees

Commit message: concern
Parts:
- removed L298N1, L298N2: ~, l298n:TO127P2020X500X2100-15
- removed U10, U12, U8: XT30UPB-M, xt30:XT30UPB-M
- moved U5 112.2 mm to (106.8, 99.4)
- moved U4 88.2 mm to (112.8, 47.6)
- moved U6 87.8 mm to (84.6, 60.2), turned to 0 degrees
- moved SW1 87.7 mm to (171.5, 55.2), turned to 40 degrees
- moved U7 39.7 mm to (71.7, 69.5), turned to 0 degrees
- moved U9 34.0 mm to (79.6, 93.3)
- moved U11 33.6 mm to (78.9, 83.7)
- moved U3 31.1 mm to (80.1, 51.5)
Connections:
- net /Out3 renamed /O7
- net /Out4 renamed /O8
- net Net-(L298N1-Out1) renamed /O5
- net Net-(L298N1-Out2) renamed /O6
- U11 pad P$1: /5v -> Net-(U11-+)
- U11 pad P$2: GND -> Net-(U11--)
Routing:
- net /3v3: track 0.00 -> 278.4 mm
- net GND: track 0.00 -> 234.5 mm, vias 0 -> 2
- net /12v: track 0.00 -> 191.9 mm
- net /5v: track 0.00 -> 80.7 mm, vias 0 -> 2
- added copper zone on B.Cu, net GND
- added copper zone on F.Cu, net GND
Other:
- board outline added: 178 x 178 mm

Commit message: motor driver for motor 1 done
Parts:
- removed H1, H10, H11, H12, H2, H3, H4, H5, H6, H7, H8, H9: MountingHole, MountingHole:MountingHole_3.2mm_M3_DIN965_Pad
- removed SW1: SW_Push, flipswitch:SW_100SP1T1B4M2QE
- removed U1, U2: LM2596ADJ, Motor Controller:LM2596ADJ
- removed U11, U3, U4, U6, U7, U9: XT30UPB-M, xt30:XT30UPB-M
- removed U5: ESP32-S3-DEVKITM-1-N8, ESP32 DEV KIT:MODULE_ESP32-S3-DEVKITM-1-N8
Routing:
- net /3v3: track 278.4 -> 0.00 mm
- net GND: track 234.5 -> 0.00 mm, vias 2 -> 0
- net /12v: track 191.9 -> 0.00 mm
- net /5v: track 80.7 -> 0.00 mm, vias 2 -> 0
- removed copper zone on B.Cu, net GND
- removed copper zone on F.Cu, net GND
Other:
- board size 178 x 178 mm -> 178 x 169.6 mm

Commit message: 4 motor drivers
Parts:
- added A1: TEENSY_4.0, Sen Robo:Teensy 4.0, F.Cu at (262.8, 152.9)
- added C1: 470u, Sen Robo:CP_Radial_D8.0mm_P3.50mm, F.Cu at (268.0, 70.1)
- added C2: 470u, Sen Robo:CP_Radial_D8.0mm_P3.50mm, F.Cu at (268.0, 79.7)
- added C3: 470u, Sen Robo:CP_Radial_D8.0mm_P3.50mm, F.Cu at (310.0, 66.6)
- added C4: 470u, Sen Robo:CP_Radial_D8.0mm_P3.50mm, F.Cu at (310.0, 76.2)
- added C5: 470u, Sen Robo:CP_Radial_D8.0mm_P3.50mm, F.Cu at (319.5, 66.6)
- added C6: 470u, Sen Robo:CP_Radial_D8.0mm_P3.50mm, F.Cu at (319.5, 76.2)
- added C7: 470u, Sen Robo:CP_Radial_D8.0mm_P3.50mm, F.Cu at (329.1, 66.6)
- added C8: 470u, Sen Robo:CP_Radial_D8.0mm_P3.50mm, F.Cu at (329.1, 76.2)
- added H1: MountingHole, MountingHole:MountingHole_3.2mm_M3_DIN965_Pad, F.Cu at (80.5, 29.0)
- added H10: MountingHole, MountingHole:MountingHole_3.2mm_M3_DIN965_Pad, F.Cu at (109.0, 173.0)
- added H11: MountingHole, MountingHole:MountingHole_3.2mm_M3_DIN965_Pad, F.Cu at (102.0, 149.4)
- added H12: MountingHole, MountingHole:MountingHole_3.2mm_M3_DIN965_Pad, F.Cu at (80.5, 87.0)
- added H13: MountingHole, MountingHole:MountingHole_3.2mm_M3_DIN965_Pad, F.Cu at (184.5, 83.0)
- added H14: MountingHole, MountingHole:MountingHole_3.2mm_M3_DIN965_Pad, F.Cu at (130.5, 87.0)
- added H15: MountingHole, MountingHole:MountingHole_3.2mm_M3_DIN965_Pad, F.Cu at (129.0, 169.8)
- added H16: MountingHole, MountingHole:MountingHole_3.2mm_M3_DIN965_Pad, F.Cu at (109.0, 149.4)
- added H17: MountingHole, MountingHole:MountingHole_3.2mm_M3_DIN965_Pad, F.Cu at (82.4, 138.0)
- added H18: MountingHole, MountingHole:MountingHole_3.2mm_M3_DIN965_Pad, F.Cu at (82.4, 78.0)
- added H19: MountingHole, MountingHole:MountingHole_3.2mm_M3_DIN965_Pad, F.Cu at (26.5, 133.0)
- added H2: MountingHole, MountingHole:MountingHole_3.2mm_M3_DIN965_Pad, F.Cu at (184.5, 133.0)
- added H20: MountingHole, MountingHole:MountingHole_3.2mm_M3_DIN965_Pad, F.Cu at (26.5, 83.0)
- added H3: MountingHole, MountingHole:MountingHole_3.2mm_M3_DIN965_Pad, F.Cu at (130.5, 129.0)
- added H4: MountingHole, MountingHole:MountingHole_3.2mm_M3_DIN965_Pad, F.Cu at (102.0, 173.0)
- added H5: MountingHole, MountingHole:MountingHole_3.2mm_M3_DIN965_Pad, F.Cu at (82.0, 169.8)
- added H6: MountingHole, MountingHole:MountingHole_3.2mm_M3_DIN965_Pad, F.Cu at (80.5, 129.0)
- added H7: MountingHole, MountingHole:MountingHole_3.2mm_M3_DIN965_Pad, F.Cu at (130.5, 29.0)
- added H8: MountingHole, MountingHole:MountingHole_3.2mm_M3_DIN965_Pad, F.Cu at (128.6, 78.0)
- added H9: MountingHole, MountingHole:MountingHole_3.2mm_M3_DIN965_Pad, F.Cu at (128.6, 138.0)
- added J1: Conn_01x02, Connector_PinHeader_1.00mm:PinHeader_1x02_P1.00mm_Horizontal, F.Cu at (308.5, 121.2)
- added J2: Conn_01x02, Connector_PinHeader_1.00mm:PinHeader_1x02_P1.00mm_Horizontal, F.Cu at (315.9, 152.5)
- added Q1: AON6354, Sen Robo:8-DFN (5x6), F.Cu at (253.9, 84.3)
- added Q2: AON6354, Sen Robo:8-DFN (5x6), F.Cu at (306.0, 85.2)
- added Q3: AON6354, Sen Robo:8-DFN (5x6), F.Cu at (312.9, 85.2)
- added Q4: AON6354, Sen Robo:8-DFN (5x6), F.Cu at (319.8, 85.2)
- added R1: 1K, Sen Robo:res0603, F.Cu at (252.1, 97.2)
- added R10: 3K3, Sen Robo:res0603, F.Cu at (368.3, 106.2)
- added R11: 10K, Sen Robo:res0603, F.Cu at (368.3, 109.1)
- added R12: 1K, Sen Robo:res0603, F.Cu at (368.3, 112.0)
- added R13: 1K, Sen Robo:res0603, F.Cu at (368.3, 114.9)
- added R14: 1K, Sen Robo:res0603, F.Cu at (368.3, 117.8)
- added R15: 1K, Sen Robo:res0603, F.Cu at (368.3, 120.7)
- added R16: 1K, Sen Robo:res0603, F.Cu at (368.3, 123.6)
- added R17: 3K3, Sen Robo:res0603, F.Cu at (368.3, 126.5)
- added R18: 3K3, Sen Robo:res0603, F.Cu at (368.3, 129.4)
- added R19: 10K, Sen Robo:res0603, F.Cu at (373.0, 106.2)
- added R2: 1K, Sen Robo:res0603, F.Cu at (252.1, 100.1)
- added R20: 1K, Sen Robo:res0603, F.Cu at (373.0, 109.1)
- added R21: 1K, Sen Robo:res0603, F.Cu at (373.0, 112.0)
- added R22: 1K, Sen Robo:res0603, F.Cu at (373.0, 114.9)
- added R23: 1K, Sen Robo:res0603, F.Cu at (373.0, 117.8)
- added R24: 1K, Sen Robo:res0603, F.Cu at (373.0, 120.7)
- added R25: 3K3, Sen Robo:res0603, F.Cu at (373.0, 123.6)
- added R26: 3K3, Sen Robo:res0603, F.Cu at (373.0, 126.5)
- added R27: 10K, Sen Robo:res0603, F.Cu at (373.0, 129.4)
- added R28: 1K, Sen Robo:res0603, F.Cu at (377.7, 106.2)
- added R29: 1K, Sen Robo:res0603, F.Cu at (377.7, 109.1)
- added R3: 1K, Sen Robo:res0603, F.Cu at (252.1, 103.0)
- added R30: 1K, Sen Robo:res0603, F.Cu at (377.7, 112.0)
- added R31: 1K, Sen Robo:res0603, F.Cu at (377.7, 114.9)
- added R32: 1K, Sen Robo:res0603, F.Cu at (377.7, 117.8)
- added R33: 1K, Sen Robo:res0603, F.Cu at (316.8, 156.5)
- added R4: 1K, Sen Robo:res0603, F.Cu at (259.7, 107.1)
- added R5: 1K, Sen Robo:res0603, F.Cu at (252.1, 108.8)
- added R6: 10K, Sen Robo:res0603, F.Cu at (252.1, 111.7)
- added R7: 3K3, Sen Robo:res0603, F.Cu at (252.1, 114.6)
- added R8: 3K3, Sen Robo:res0603, F.Cu at (252.1, 117.5)
- added R9: 3K3, Sen Robo:res0603, F.Cu at (363.6, 129.4)
- added SW1: SW_Push, flipswitch:SW_100SP1T1B4M2QE, F.Cu at (311.7, 112.6)
- added SW2: SW_Nidec_CAS-120A1, Button_Switch_SMD:Nidec_Copal_CAS-120A, F.Cu at (317.1, 147.5)
- added U1: LM2596ADJ, buck converter:LM2596ADJ, F.Cu at (301.6, 98.1)
- added U12: VNH5019ATR-E, Sen Robo:VNH5019A-E, F.Cu at (360.1, 51.6)
- added U2: LM2596ADJ, buck converter:LM2596ADJ, F.Cu at (313.4, 98.1)
- added U3: XT30UPB-M, xt30:XT30UPB-M, F.Cu at (301.3, 108.6)
- added U4: XT30UPB-M, xt30:XT30UPB-M, F.Cu at (301.3, 115.0)
- added U6: VNH5019ATR-E, Sen Robo:VNH5019A-E, F.Cu at (252.4, 67.6)
- added U7: VNH5019ATR-E, Sen Robo:VNH5019A-E, F.Cu at (323.3, 51.6)
- added U8: VNH5019ATR-E, Sen Robo:VNH5019A-E, F.Cu at (341.7, 51.6)
- added U9: XT30UPB-M, xt30:XT30UPB-M, F.Cu at (289.9, 114.7)

Commit message: to be fix
Other:
- outline, holes or cut-outs redrawn

Commit message: to do
add sensor fix motor drivers and teensy
Parts:
- C1, C2, Q1, R10, R11, R12, R13, R14, R15, R16, R9, U6: moved to B.Cu
- moved R10 284.0 mm to (88.4, 58.6), turned to 180 degrees
- moved R11 284.0 mm to (88.4, 61.5), turned to 180 degrees
- moved R13 284.0 mm to (88.4, 67.3), turned to 180 degrees
- moved R14 284.0 mm to (88.4, 70.2), turned to 180 degrees
- moved R15 284.0 mm to (88.4, 73.1), turned to 180 degrees
- moved R16 284.0 mm to (88.4, 76.0), turned to 180 degrees
- moved R12 283.2 mm to (89.2, 64.2), turned to 180 degrees
- moved R9 279.6 mm to (88.3, 80.7), turned to 180 degrees
- moved C2 170.5 mm to (99.2, 55.7), turned to 90 degrees
- moved Q1 165.0 mm to (89.0, 89.7), turned to 90 degrees
- moved C1 159.9 mm to (108.8, 55.7), turned to 90 degrees
- moved R1 159.2 mm to (405.6, 139.1)
- moved R2 159.2 mm to (405.6, 142.0)
- moved R3 159.2 mm to (405.6, 144.9)
- moved R5 159.2 mm to (405.6, 150.7)
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Routing:
- net Net-(C1-Pad1): track 0.00 -> 68.5 mm
- net Net-(U6-ENA/DIAGA): track 0.00 -> 48.9 mm
- net GND: track 0.00 -> 39.5 mm
- net /Motor 2 ENA: track 0.00 -> 29.6 mm
- net +12V: track 0.00 -> 29.6 mm
- net /PWM Motor 2: track 0.00 -> 28.4 mm
- net Net-(U6-INA): track 0.00 -> 27.6 mm
- net +3V3: track 0.00 -> 23.6 mm
- net Net-(U6-INB): track 0.00 -> 21.7 mm
- net Net-(U6-PWM): track 0.00 -> 20.3 mm
- net /Motor 2 ENB: track 0.00 -> 13.5 mm
- net /Motor Driver: track 0.00 -> 2.90 mm

Commit message: 2 more motor drivers to go!
Parts:
- added H21: MountingHole, MountingHole:MountingHole_3.2mm_M3_DIN965_Pad, F.Cu at (102.0, 160.4)
- added H22: MountingHole, MountingHole:MountingHole_3.2mm_M3_DIN965_Pad, F.Cu at (109.0, 160.4)
- added J3: XT60-M, xt60-m:AMASS_XT60-M, F.Cu at (342.7, 204.9)
- C3, C4, Q2, R1, R2, R3, R4, R5, R6, R7, R8: moved to B.Cu
- U12: footprint Sen Robo:VNH5019A-E -> vhn5019:IC_VNH5019ATR-E; moved to B.Cu
- U6, U7, U8: footprint Sen Robo:VNH5019A-E -> vhn5019:IC_VNH5019ATR-E
- moved R6 309.0 mm to (113.4, 53.1), turned to 180 degrees
- moved R7 307.7 mm to (113.5, 59.7), turned to 180 degrees
- moved R8 307.4 mm to (113.7, 63.1), turned to 180 degrees
- moved R1 303.5 mm to (113.5, 56.6), turned to 180 degrees
- moved R4 299.5 mm to (119.5, 59.9)
- moved R2 299.4 mm to (119.7, 53.1)
- moved R3 299.3 mm to (119.6, 56.8)
- moved R5 299.2 mm to (119.5, 63.2)
- moved U12 263.9 mm to (96.4, 63.3), turned to 180 degrees
- moved C3 194.1 mm to (120.3, 107.9)
- moved Q2 193.9 mm to (112.8, 101.6), turned to 180 degrees
- moved C4 190.9 mm to (120.4, 98.4)
- moved U7 150.5 mm to (280.4, 195.8)
- moved R10 37.2 mm to (115.9, 83.6)
- moved R13 36.1 mm to (116.4, 90.0)
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Connections:
- U2 pad 2: /3v3 -> +3V3
- U4 pad P$1: /3v3 -> +3V3
Routing:
- net GND: track 39.5 -> 176.9 mm
- net Net-(C3-Pad1): track 0.00 -> 55.5 mm
- net +12V: track 29.6 -> 68.5 mm, vias 0 -> 3
- net Net-(U6-ENA/DIAGA): track 48.9 -> 11.3 mm
- net /Motor 1 Out A: track 0.00 -> 32.2 mm
- net /Motor 1 Out B: track 0.00 -> 30.5 mm
- net Net-(C1-Pad1): track 68.5 -> 96.9 mm
- net /Motor 2 Out B: track 0.00 -> 27.5 mm
- net Net-(U12-PWM): track 0.00 -> 24.7 mm, vias 0 -> 2
- net Net-(U12-ENA/DIAGA): track 0.00 -> 22.7 mm
- net /Motor 2 ENA: track 29.6 -> 7.39 mm
- net Net-(U6-INA): track 27.6 -> 6.13 mm
- net /PWM Motor 2: track 28.4 -> 8.49 mm, vias 0 -> 2
- net Net-(U12-INA): track 0.00 -> 18.4 mm
- net Net-(U12-ENB/DIAGB): track 0.00 -> 18.1 mm
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- added copper zone on B.Cu, net GND
- added copper zone on F.Cu, net GND
Other:
- outline, holes or cut-outs redrawn
