File: Electrical/PCB V2 ( 26 Nov)/L2/Layer_2/Layer_2.kicad_pcb (KiCad board)
At the start: 2 copper layers, 178 x 169.6 mm, 82 parts, among them J1 Conn_01x02, J2 Conn_01x02, J3 XT60-M, Q1 AON6354, Q2 AON6354, Q3 AON6354, Q4 AON6354, SW1 SW_Push, SW2 SW_Nidec_CAS-120A1, U1 LM2596ADJ, U12 VNH5019ATR-E, U2 LM2596ADJ, U3 XT30UPB-M, U4 XT30UPB-M, U6 VNH5019ATR-E, U7 VNH5019ATR-E, U8 VNH5019ATR-E, U9 XT30UPB-M

Commit message: cred tbc and switches
Parts:
- removed H11, H21: MountingHole, MountingHole:MountingHole_3.2mm_M3_DIN965_Pad
- removed U9: XT30UPB-M, xt30:XT30UPB-M
- C5, C6, C7, C8, Q3, Q4, R17, R18, R19, R20, R21, R22, R23, R24, R25, R26, R27, R28, R29, R30, R31, R32, U7, U8: moved to B.Cu
- moved J3 294.2 mm to (105.2, 31.3), turned to 90 degrees
- moved R28 265.1 mm to (114.2, 134.8), turned to 180 degrees
- moved SW2 265.0 mm to (53.8, 118.3), turned to 90 degrees
- moved SW1 264.9 mm to (47.2, 97.5), turned to 90 degrees
- moved R29 264.9 mm to (114.3, 137.4), turned to 180 degrees
- moved R30 264.9 mm to (114.3, 140.0), turned to 180 degrees
- moved R31 264.6 mm to (114.5, 142.4), turned to 180 degrees
- moved R22 263.9 mm to (109.3, 107.5), turned to 180 degrees
- moved R20 263.8 mm to (109.2, 110.2), turned to 180 degrees
- moved R24 263.7 mm to (109.4, 113.2), turned to 180 degrees
- moved R23 263.7 mm to (109.3, 119.5), turned to 180 degrees
- moved R21 263.7 mm to (109.4, 116.3), turned to 180 degrees
- moved U8 259.8 mm to (96.1, 136.5), turned to 180 degrees
- moved R19 258.6 mm to (114.5, 113.0)
- moved R32 257.3 mm to (121.7, 142.8), turned to 180 degrees
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Routing:
- net +3V3: track 36.9 -> 217.3 mm, vias 0 -> 2
- net /12v: track 0.00 -> 122.2 mm, vias 0 -> 2
- net /Motor Driver: track 10.5 -> 132.1 mm, vias 0 -> 5
- net GND: track 176.9 -> 289.4 mm
- net /5v: track 0.00 -> 110.4 mm
- net +12V: track 68.5 -> 162.2 mm, vias 3 -> 5
- net Net-(C7-Pad1): track 0.00 -> 90.4 mm
- net Net-(C5-Pad1): track 0.00 -> 66.4 mm
- net /PWM Motor 2: track 8.49 -> 41.1 mm, vias 2 -> 3
- net /Motor 4 Out B: track 0.00 -> 31.1 mm, vias 0 -> 2
- net /Motor 4 Out A: track 0.00 -> 27.5 mm
- net /Motor 3 Out A: track 0.00 -> 27.5 mm
- net /Motor 3 Out B: track 0.00 -> 27.5 mm
- net Net-(Q3-G): track 0.00 -> 22.5 mm, vias 0 -> 2
- net Net-(U8-PWM): track 0.00 -> 20.4 mm
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Other:
- board text added: "Cred Sen Robo Tks"

Commit message: to be done : solve the teensy mystyery
Parts:
- removed the J1 at (308.5, 121.2)
- removed J2: Conn_01x02, Connector_PinHeader_1.00mm:PinHeader_1x02_P1.00mm_Horizontal
- A1: footprint Sen Robo:Teensy 4.0 -> Teensy:MODULE_DEV-15583
- SW1: renamed from SW2; footprint Button_Switch_SMD:Nidec_Copal_CAS-120A -> Connector_PinHeader_1.00mm:PinHeader_1x03_P1.00mm_Vertical
- SW2: renamed from SW1; footprint flipswitch:SW_100SP1T1B4M2QE -> Connector_PinHeader_1.00mm:PinHeader_1x03_P1.00mm_Vertical
- moved R9 22.5 mm to (43.1, 108.8)
- moved SW1 10.5 mm to (49.6, 108.7), turned to -90 degrees
- moved SW2 9.15 mm to (47.5, 88.4)
- renumbered H2 to H1, H4 to H10, H3 to H11, H8 to H12, H7 to H13, H12 to H14, H17 to H15, H18 to H17, H19 to H18, H20 to H19, H1 to H2, H22 to H20, H6 to H3, H5 to H4, H10 to H5, H9 to H6, H14 to H7, H13 to H8, H15 to H9, J3 to J1, R8 to R1, R9 to R10, R10 to R11, R11 to R12, R12 to R13, R13 to R14, R14 to R15, R15 to R16, R16 to R17, R17 to R18, R18 to R19, R7 to R2, R19 to R20, R20 to R21, R21 to R22, R22 to R23, R23 to R24, R24 to R25, R25 to R26, R26 to R27, R27 to R28, R28 to R29, R6 to R3, R29 to R30, R30 to R31, R31 to R32, R32 to R33, R5 to R4, R4 to R5, R3 to R6, R1 to R7, R2 to R8, R33 to R9, U2 to U1, U1 to U2, U12 to U3, U3 to U4, U4 to U5
Connections:
- net /Motor 1 ENA renamed /Motor 1 EN A
- net /Motor 1 ENB renamed /Motor 1 EN B
- net /Motor 2 ENA renamed /Motor 2 EN A
- net /Motor 2 ENB renamed /Motor 2 EN B
- net /Motor 3 ENA renamed /Motor 3 EN A
- net /Motor 3 ENB renamed /Motor 3 EN B
- net /Motor 4 ENA renamed /Motor 4 EN A
- net /Motor 4 ENB renamed /Motor 4 EN B
- Q1 pad 1: +12V -> /12V
- Q1 pad 2: +12V -> /12V
- Q1 pad 3: +12V -> /12V
- Q2 pad 1: +12V -> /12V
- Q2 pad 2: +12V -> /12V
- Q2 pad 3: +12V -> /12V
- Q3 pad 1: +12V -> /12V
- Q3 pad 2: +12V -> /12V
- Q3 pad 3: +12V -> /12V
- Q4 pad 1: +12V -> /12V
- Q4 pad 2: +12V -> /12V
- Q4 pad 3: +12V -> /12V
- R20 pad 1: /PWM Motor 2 -> /PWM Motor 3
- R25 pad 1: /PWM Motor 2 -> /PWM Motor 3
- SW1 pad 2: Net-(J2-Pin_2) -> /Motor Driver
- U3 pad 12: +12V -> /12V
- U6 pad 12: +12V -> /12V
- U7 pad 12: +12V -> /12V
- U8 pad 12: +12V -> /12V
Routing:
- net +3V3: track 217.3 -> 386.7 mm, vias 2 -> 6
- net /12V: track 0.00 -> 162.2 mm, vias 0 -> 5
- net +12V: track 162.2 -> 0.00 mm, vias 5 -> 0
- net /Motor Driver: track 132.1 -> 228.4 mm
- net /12v: track 122.2 -> 210.8 mm, vias 2 -> 4
- net /Motor 2 Out A: track 0.00 -> 27.5 mm
- net Net-(Q2-G): track 0.00 -> 12.4 mm, vias 0 -> 2
- net Net-(SW1-A): track 0.00 -> 6.92 mm
- net /5v: track 110.4 -> 110.9 mm
Other:
- board text added: "We extend our heartfelt and profound gratitude to sentinels robotics and kessoku band for graciously granting us permission to take inspiration from their esteemed motor driver schematics and PCB layout, which have greatly guided our endeavors."
- board text added: "We extend our most profound gratitude unto sentinels robotics and kessoku band ,who hath graciously bestowed upon us leave to draw nobleinspiration from their esteemed motor driver schematics and PCB layout."
- board text added: "We wish to express our deepest gratitude to sentinels robotics and kessoku band for graciously granting us permission to derive substantialinspiration from their exemplary motor driver schematics and PCB layout."
- board text added: "We would like to extend our utmost thanks to sentinels robotics and kessoku band for granting us permission to draw significant inspiration from their motor driver schematics and PCB layout."
- board text removed: "Cred Sen Robo Tks"
