File: Electrical/PCB V2 ( 26 Nov)/L2/Layer_2/Layer_2.kicad_sch (KiCad schematic)
At the start: 50 parts, among them J1 Conn_01x02, Q1 AON6354, Q2 AON6354, SW1 SW_Push, U1 LM2596ADJ, U12 VNH5019ATR-E, U2 LM2596ADJ, U3 XT30UPB-M, U4 XT30UPB-M, U5 ESP32-S3-DEVKITM-1-N8, U6 VNH5019ATR-E

Commit message: 4 motor drivers
Parts:
- removed BT1: Battery, symbol Device:Battery
- removed U5: ESP32-S3-DEVKITM-1-N8, ESP32-S3-DEVKITM-1-N8:MODULE_ESP32-S3-DEVKITM-1-N8, symbol ESP32-S3-DEVKITM-1-N8:ESP32-S3-DEVKITM-1-N8
- added A1: TEENSY_4.0, Sen Robo:Teensy 4.0, symbol Teensy 4.0:TEENSY_4.0
- added C5, C6, C7, C8: 470u, Sen Robo:CP_Radial_D8.0mm_P3.50mm, symbol Device:C_Polarized
- added H19, H20: MountingHole, MountingHole:MountingHole_3.2mm_M3_DIN965_Pad, symbol Mechanical:MountingHole
- added J2: Conn_01x02, Connector_PinHeader_1.00mm:PinHeader_1x02_P1.00mm_Horizontal, symbol Connector_Generic:Conn_01x02
- added Q3, Q4: AON6354, Sen Robo:8-DFN (5x6), symbol vincent:AON6354
- added R17, R18, R25, R26: 3K3, Sen Robo:res0603, symbol Device:R
- added R19, R27: 10K, Sen Robo:res0603, symbol Device:R
- added R20, R21, R22, R23, R24, R28, R29, R30, R31, R32, R33: 1K, Sen Robo:res0603, symbol Device:R
- added SW2: SW_Nidec_CAS-120A1, Button_Switch_SMD:Nidec_Copal_CAS-120A, symbol Switch:SW_Nidec_CAS-120A1
- added U7, U8: VNH5019ATR-E, Sen Robo:VNH5019A-E, symbol VHN5019ATR-E:VNH5019ATR-E
- added U9: XT30UPB-M, xt30:XT30UPB-M, symbol XT30UPB-M:XT30UPB-M
- C1, C2, C3, C4: footprint 2024l2:CP_Radial_D8.0mm_P3.50mm -> Sen Robo:CP_Radial_D8.0mm_P3.50mm
- Q1, Q2: footprint 2024l2:8-DFN (5x6) -> Sen Robo:8-DFN (5x6)
- R1, R10, R11, R12, R13, R14, R15, R16, R2, R3, R4, R5, R6, R7, R8, R9: footprint 2024l2:res0603 -> Sen Robo:res0603
- U1, U2: footprint LM2596ADJ:LM2596ADJ -> buck converter:LM2596ADJ
- U12, U6: footprint VNH5019ATR-E:IC_VNH5019ATR-E -> Sen Robo:VNH5019A-E
Connections:
- net Motor 1 In B is gone; now on net Motor Driver: R1.1, R15.1
- net +12V: now also Q3.1 (S), Q3.2 (S), Q3.3 (S), Q4.1 (S), Q4.2 (S), Q4.3 (S), R33.2, U7.12 (VBAT), U8.12 (VBAT)
- net +3V3: now also R17.2, R18.2, R25.2, R26.2
- net 12v: now also U9.P$1 (+)
- net GND: now also A1.AGND/GND (GND), A1.GND, C5.2, C6.2, C7.2, C8.2, R19.2, R27.2, U7.18 (GNDB), U7.19 (GNDB), U7.20 (GNDB), U7.26 (GNDA), U7.27 (GNDA), U7.28 (GNDA), U8.18 (GNDB), U8.19 (GNDB), U8.20 (GNDB), U8.26 (GNDA), U8.27 (GNDA), U8.28 (GNDA), U9.P$2 (-)
- net Motor 1 ENA: no longer R12.1, R9.1
- net Motor 1 ENB: no longer R10.1, R13.1
- net Motor 1 Out A: no longer U6.1 (OUTA), U6.25 (OUTA), U6.30 (OUTA), U6.HS2 (OUTA)
- net Motor 1 Out B: no longer U6.15 (OUTB), U6.16 (OUTB), U6.21 (OUTB), U6.HS3 (OUTB)
- net PWM Motor 1: no longer R11.1, R16.1
- net Battery: now reaches SW1.1
- net Motor 1 In A renamed Motor Driver
- net Motor Driver: now also J2.1 (Pin_1), R22.1, R23.1, R30.1, R31.1
- new net: C7.1, C8.1, Q4.5 (D), Q4.6 (D), Q4.7 (D), Q4.8 (D), Q4.9 (D), U8.13 (VCC), U8.23 (VCC), U8.3 (VCC), U8.HS1 (VCC)
- new net: R21.2, U7.9 (ENB/DIAGB)
- new net: R24.2, U7.7 (PWM)
- new net: R30.2, U8.4 (INA)
- new net: R22.2, U7.4 (INA)
- new net: R33.1, SW2.3 (A)
- new net: R20.2, U7.5 (ENA/DIAGA)
- new net: Q4.4 (G), U8.11 (CP)
- new net: Q3.4 (G), U7.11 (CP)
- new net: C5.1, C6.1, Q3.5 (D), Q3.6 (D), Q3.7 (D), Q3.8 (D), Q3.9 (D), U7.13 (VCC), U7.23 (VCC), U7.3 (VCC), U7.HS1 (VCC)
- new net: R23.2, U7.10 (INB)
- new net: R29.2, U8.9 (ENB/DIAGB)
- new net: R31.2, U8.10 (INB)
- new net: J2.2 (Pin_2), SW2.2 (B)
- new net: R32.2, U8.7 (PWM)
- new net: R28.2, U8.5 (ENA/DIAGA)
- new net Motor 2 ENA: R12.1, R9.1
- new net Motor 2 ENB: R10.1, R13.1
- new net Motor 2 Out A: U6.1 (OUTA), U6.25 (OUTA), U6.30 (OUTA), U6.HS2 (OUTA)
- new net Motor 2 Out B: U6.15 (OUTB), U6.16 (OUTB), U6.21 (OUTB), U6.HS3 (OUTB)
- new net Motor 3 ENA: R17.1, R20.1
- new net Motor 3 ENB: R18.1, R21.1
- new net Motor 3 Out A: U7.1 (OUTA), U7.25 (OUTA), U7.30 (OUTA), U7.HS2 (OUTA)
- new net Motor 3 Out B: U7.15 (OUTB), U7.16 (OUTB), U7.21 (OUTB), U7.HS3 (OUTB)
- new net Motor 4 ENA: R25.1, R28.1
- new net Motor 4 ENB: R26.1, R29.1
- new net Motor 4 Out A: U8.1 (OUTA), U8.25 (OUTA), U8.30 (OUTA), U8.HS2 (OUTA)
- new net Motor 4 Out B: U8.15 (OUTB), U8.16 (OUTB), U8.21 (OUTB), U8.HS3 (OUTB)
- new net PWM Motor 2: R11.1, R16.1, R19.1, R24.1
- new net PWM Motor 4: R27.1, R32.1
- no-connect marks 8 -> 12
Other:
- note added: "Motor 2 Driver"
- note added: "Motor 3 Driver"
- note added: "Motor 4 Driver"
- note added: "Tensy 4.0"
- note removed: "ESP32 for motor control"
- moved on the sheet: C1, C2, C3, C4, H1, H10, H11, H12, H13, H14, H15, H16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

Commit message: to be fix
Parts:
- added H21, H22: MountingHole, MountingHole:MountingHole_3.2mm_M3_DIN965_Pad, symbol Mechanical:MountingHole
Changed lines of the file:
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@@
 	(rectangle
 		(start 15.0454 176.4851)
-		(end 142.24 195.5351)
+		(end 152.4 195.5351)
 		(stroke
 			(width 0)
@@
 	(text "Mounting Holes"
 		(exclude_from_sim no)
-		(at 151.13 179.578 0)
+		(at 159.512 179.324 0)
 		(effects
 			(font
@@
 	)
 	(symbol
+		(lib_id "Mechanical:MountingHole")
+		(at 148.59 191.77 90)
+		(unit 1)
+		(exclude_from_sim yes)
+		(in_bom no)
+		(on_board yes)
+		(dnp no)
+		(property "Reference" "H22"
+			(at 147.3199 189.23 0)
+			(effects
+				(font
+					(size 1.27 1.27)
+				)
+				(justify left)
+			)
+		)
+		(property "Value" "MountingHole"
+			(at 149.8599 189.23 0)
+			(effects
+				(font
+					(size 1.27 1.27)
+				)
+				(justify left)
+			)
+		)
+		(property "Footprint" "MountingHole:MountingHole_3.2mm_M3_DIN965_Pad"
+			(at 148.59 191.77 0)
+			(effects
+				(font
+					(size 1.27 1.27)
+				)
+				(hide yes)
+			)
+		)
+		(property "Datasheet" "~"
+			(at 148.59 191.77 0)
+			(effects
+				(font
+					(size 1.27 1.27)
+				)
+				(hide yes)
+			)
+		)
+		(property "Description" "Mounting Hole without connection"
+			(at 148.59 191.77 0)
+			(effects
+				(font
+					(size 1.27 1.27)
+				)
+				(hide yes)
+			)
+		)
+		(instances
+			(project "Layer_2"
+				(path "/164539e9-489b-4b17-b405-637c12a94360"
+					(reference "H22")
+					(unit 1)
+				)
+			)
+		)
+	)
+	(symbol
 		(lib_id "power:+3V3")
 		(at 223.52 123.19 0)
@@
 					(unit 1)
 				)
+			)
+		)
+	)
+	(symbol
+		(lib_id "Mechanical:MountingHole")
+		(at 142.24 191.77 90)
+		(unit 1)
+		(exclude_from_sim yes)
+		(in_bom no)
+		(on_board yes)
+		(dnp no)
+		(property "Reference" "H21"
+			(at 140.9699 189.23 0)
+			(effects
+				(font
+					(size 1.27 1.27)
+				)
+				(justify left)
+			)
+		)
+		(property "Value" "MountingHole"
+			(at 143.5099 189.23 0)
+			(effects
+				(font
+					(size 1.27 1.27)
+				)
+				(justify left)
+			)
+		)
+		(property "Footprint" "MountingHole:MountingHole_3.2mm_M3_DIN965_Pad"
+			(at 142.24 191.77 0)
+			(effects
+				(font
+					(size 1.27 1.27)
+				)
+				(hide yes)
+			)
+		)
+		(property "Datasheet" "~"
+			(at 142.24 191.77 0)
+			(effects
+				(font
+					(size 1.27 1.27)
+				)
+				(hide yes)
+			)
+		)
+		(property "Description" "Mounting Hole without connection"
+			(at 142.24 191.77 0)
+			(effects
+				(font
+					(size 1.27 1.27)
+				)
+				(hide yes)
+			)
+		)
+		(instances
+			(project "Layer_2"
+				(path "/164539e9-489b-4b17-b405-637c12a94360"
+					(reference "H21")
+					(unit 1)
+				)

Commit message: to do
add sensor fix motor drivers and teensy
Connections:
- net 3v3 is gone; now on net +3V3: U2.2 (OUT), U4.P$1 (+)

Commit message: 2 more motor drivers to go!
Parts:
- removed U9: XT30UPB-M, xt30:XT30UPB-M, symbol XT30UPB-M:XT30UPB-M
- added J3: XT60-M, xt60-m:AMASS_XT60-M, symbol XT60-M:XT60-M
- U12, U6, U7, U8: footprint Sen Robo:VNH5019A-E -> vhn5019:IC_VNH5019ATR-E
Connections:
- net 12v: now also J3.P (POS)
- net GND: now also J3.N (NEG)
Changed lines of the file:
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@@
 	)
 	(label "GND"
-		(at 54.61 113.03 0)
+		(at 54.61 110.49 0)
 		(fields_autoplaced yes)
 		(effects
@@
 	)
 	(label "12v"
-		(at 54.61 110.49 0)
+		(at 54.61 113.03 0)
 		(fields_autoplaced yes)
 		(effects
@@
 			)
 		)
-		(property "Footprint" "Sen Robo:VNH5019A-E"
+		(property "Footprint" "vhn5019:IC_VNH5019ATR-E"
 			(at 158.75 146.05 0)
 			(effects
@@
 	)
 	(symbol
+		(lib_id "XT60-M:XT60-M")
+		(at 49.53 110.49 180)
+		(unit 1)
+		(exclude_from_sim no)
+		(in_bom yes)
+		(on_board yes)
+		(dnp no)
+		(fields_autoplaced yes)
+		(property "Reference" "J3"
+			(at 45.72 102.87 0)
+			(effects
+				(font
+					(size 1.27 1.27)
+				)
+			)
+		)
+		(property "Value" "XT60-M"
+			(at 45.72 105.41 0)
+			(effects
+				(font
+					(size 1.27 1.27)
+				)
+			)
+		)
+		(property "Footprint" "xt60-m:AMASS_XT60-M"
+			(at 49.53 110.49 0)
+			(effects
+				(font
+					(size 1.27 1.27)
+				)
+				(justify bottom)
+				(hide yes)
+			)
+		)
+		(property "Datasheet" ""
+			(at 49.53 110.49 0)
+			(effects
+				(font
+					(size 1.27 1.27)
+				)
+				(hide yes)
+			)
+		)
+		(property "Description" ""
+			(at 49.53 110.49 0)
+			(effects
+				(font
+					(size 1.27 1.27)
+				)
+				(hide yes)
+			)
+		)
+		(property "MF" "AMASS"
+			(at 49.53 110.49 0)
+			(effects
+				(font
+					(size 1.27 1.27)
+				)
+				(justify bottom)
+				(hide yes)
+			)
+		)
+		(property "MAXIMUM_PACKAGE_HEIGHT" "16.00 mm"
+			(at 49.53 110.49 0)
+			(effects
+				(font
+					(size 1.27 1.27)
+				)
+				(justify bottom)
+				(hide yes)
+			)
+		)
+		(property "Package" "Package"
+			(at 49.53 110.49 0)
+			(effects
+				(font
+					(size 1.27 1.27)
+				)
+				(justify bottom)
+				(hide yes)
+			)
+		)
+		(property "Price" "None"
+			(at 49.53 110.49 0)
+			(effects
+				(font
+					(size 1.27 1.27)
+				)
+				(justify bottom)
+				(hide yes)
+			)
+		)
+		(property "Check_prices" "https://www.snapeda.com/parts/XT60-M/AMASS/view-part/?ref=eda"
+			(at 49.53 110.49 0)
+			(effects
+				(font
+					(size 1.27 1.27)
+				)
+				(justify bottom)
+				(hide yes)
+			)
+		)
+		(property "STANDARD" "IPC 7351B"
+			(at 49.53 110.49 0)
+			(effects
+				(font
+					(size 1.27 1.27)
+				)
+				(justify bottom)
+				(hide yes)
+			)
+		)
+		(property "PARTREV" "V1.2"
+			(at 49.53 110.49 0)
+			(effects
+				(font
+					(size 1.27 1.27)
+				)
+				(justify bottom)
+				(hide yes)
+			)
+		)
+		(property "SnapEDA_Link" "https://www.snapeda.com/parts/XT60-M/AMASS/view-part/?ref=snap"
+			(at 49.53 110.49 0)
+			(effects
+				(font
+					(size 1.27 1.27)
+				)
+				(justify bottom)
+				(hide yes)
+			)
+		)
+		(property "MP" "XT60-M"
+			(at 49.53 110.49 0)
+			(effects
+				(font
+					(size 1.27 1.27)
+				)
+				(justify bottom)
+				(hide yes)
+			)
+		)
+		(property "Description_1" "\n                        \n                            Plug; DC supply; XT60; male; PIN: 2; for cable; soldered; 30A; 500V\n                        \n"
+			(at 49.53 110.49 0)
+			(effects
+				(font
+					(size 1.27 1.27)
+				)
+				(justify bottom)
+				(hide yes)
+			)
+		)
+		(property "Availability" "Not in stock"
+			(at 49.53 110.49 0)
+			(effects
+				(font
+					(size 1.27 1.27)
+				)
+				(justify bottom)
+				(hide yes)
+			)
+		)
+		(property "MANUFACTURER" "AMASS"
+			(at 49.53 110.49 0)
+			(effects
+				(font
+					(size 1.27 1.27)
+				)
+				(justify bottom)
+				(hide yes)
+			)
+		)
+		(pin "P"
+		)
+		(pin "N"
+		)
+		(instances
+			(project ""
+				(path "/164539e9-489b-4b17-b405-637c12a94360"
+					(reference "J3")
+					(unit 1)
+				)
+			)
+		)
+	)
+	(symbol
 		(lib_id "power:+12V")
 		(at 35.56 107.95 0)
@@
 			)
 		)
-		(property "Footprint" "Sen Robo:VNH5019A-E"
+		(property "Footprint" "vhn5019:IC_VNH5019ATR-E"
 			(at 255.27 146.05 0)
 			(effects
@@
 			)
 		)
-		(property "Footprint" "Sen Robo:VNH5019A-E"
+		(property "Footprint" "vhn5019:IC_VNH5019ATR-E"
 			(at 62.23 146.05 0)
 			(effects
@@
 			)
 		)
-		(property "Footprint" "Sen Robo:VNH5019A-E"
+		(property "Footprint" "vhn5019:IC_VNH5019ATR-E"
 			(at 351.79 146.05 0)
 			(effects
@@
 					(unit 1)
 				)
-			)
-		)
-	)
-	(symbol
-		(lib_id "XT30UPB-M:XT30UPB-M")
-		(at 46.99 113.03 0)
-		(unit 1)
-		(exclude_from_sim no)
-		(in_bom yes)
-		(on_board yes)
-		(dnp no)
-		(fields_autoplaced yes)
-		(property "Reference" "U9"
-			(at 47.625 102.87 0)
-			(effects
-				(font
-					(size 1.27 1.27)
-				)
-			)
-		)
-		(property "Value" "XT30UPB-M"
-			(at 47.625 105.41 0)
-			(effects
-				(font
-					(size 1.27 1.27)
-				)
-			)
-		)
-		(property "Footprint" "xt30:XT30UPB-M"
-			(at 46.99 113.03 0)
-			(effects
-				(font
-					(size 1.27 1.27)
-				)
-				(justify bottom)
-				(hide yes)
-			)
-		)
-		(property "Datasheet" ""
-			(at 46.99 113.03 0)
-			(effects
-				(font
-					(size 1.27 1.27)
-				)
-				(hide yes)
-			)
-		)
-		(property "Description" ""
-			(at 46.99 113.03 0)
-			(effects
-				(font
-					(size 1.27 1.27)
-				)
-				(hide yes)
-			)
-		)
-		(property "MF" "amass"
-			(at 46.99 113.03 0)
-			(effects
-				(font
-					(size 1.27 1.27)
-				)
-				(justify bottom)
-				(hide yes)
-			)
-		)
-		(property "Description_1" "\n                        \n                            Socket; DC supply; XT30; male; PIN: 2; on PCBs; THT; yellow; 15A; 500V\n                        \n"
-			(at 46.99 113.03 0)
-			(effects
-				(font
-					(size 1.27 1.27)
-				)
-				(justify bottom)
-				(hide yes)
-			)
-		)
-		(property "Package" "None"
-			(at 46.99 113.03 0)
-			(effects
-				(font
-					(size 1.27 1.27)
-				)
-				(justify bottom)
-				(hide yes)
-			)
-		)
-		(property "Price" "None"
-			(at 46.99 113.03 0)
-			(effects
-				(font
-					(size 1.27 1.27)
-				)
-				(justify bottom)
-				(hide yes)
-			)
-		)
-		(property "SnapEDA_Link" "https://www.snapeda.com/parts/XT30UPB-M/AMASS/view-part/?ref=snap"
-			(at 46.99 113.03 0)
-			(effects
-				(font
-					(size 1.27 1.27)
-				)
-				(justify bottom)
-				(hide yes)
-			)
-		)
-		(property "MP" "XT30UPB-M"
-			(at 46.99 113.03 0)
-			(effects
-				(font
-					(size 1.27 1.27)
-				)
-				(justify bottom)
-				(hide yes)
-			)
-		)
-		(property "Availability" "Not in stock"
-			(at 46.99 113.03 0)
-			(effects
-				(font
-					(size 1.27 1.27)
-				)
-				(justify bottom)
-				(hide yes)
-			)
-		)
-		(property "Check_prices" "https://www.snapeda.com/parts/XT30UPB-M/AMASS/view-part/?ref=eda"
-			(at 46.99 113.03 0)
-			(effects
-				(font
-					(size 1.27 1.27)
-				)
-				(justify bottom)
-				(hide yes)
-			)
-		)
-		(pin "P$2"
-		)
-		(pin "P$1"
-		)
-		(instances
-			(project "Layer_2"
-				(path "/164539e9-489b-4b17-b405-637c12a94360"
-					(reference "U9")
-					(unit 1)
-				)

Commit message: cred tbc and switches
Parts:
- removed H11, H21: MountingHole, MountingHole:MountingHole_3.2mm_M3_DIN965_Pad, symbol Mechanical:MountingHole
Other:
- moved on the sheet: H16, H17, H18, H19, H20, H22
Changed lines of the file:
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@@
 	)
 	(symbol
-		(lib_id "Mechanical:MountingHole")
-		(at 108.1446 191.8149 90)
-		(unit 1)
-		(exclude_from_sim yes)
-		(in_bom no)
-		(on_board yes)
-		(dnp no)
-		(property "Reference" "H11"
-			(at 106.8745 189.2749 0)
-			(effects
-				(font
-					(size 1.27 1.27)
-				)
-				(justify left)
-			)
-		)
-		(property "Value" "MountingHole"
-			(at 109.4145 189.2749 0)
-			(effects
-				(font
-					(size 1.27 1.27)
-				)
-				(justify left)
-			)
-		)
-		(property "Footprint" "MountingHole:MountingHole_3.2mm_M3_DIN965_Pad"
-			(at 108.1446 191.8149 0)
-			(effects
-				(font
-					(size 1.27 1.27)
-				)
-				(hide yes)
-			)
-		)
-		(property "Datasheet" "~"
-			(at 108.1446 191.8149 0)
-			(effects
-				(font
-					(size 1.27 1.27)
-				)
-				(hide yes)
-			)
-		)
-		(property "Description" "Mounting Hole without connection"
-			(at 108.1446 191.8149 0)
-			(effects
-				(font
-					(size 1.27 1.27)
-				)
-				(hide yes)
-			)
-		)
-		(instances
-			(project "Layer_2"
-				(path "/164539e9-489b-4b17-b405-637c12a94360"
-					(reference "H11")
-					(unit 1)
-				)
-			)
-		)
-	)
-	(symbol
 		(lib_id "Device:C_Polarized")
 		(at 381 158.75 0)
@@
 	(symbol
 		(lib_id "Mechanical:MountingHole")
-		(at 122.1146 191.8149 90)
+		(at 113.2246 191.8149 90)
 		(unit 1)
 		(exclude_from_sim yes)
@@
 		(dnp no)
 		(property "Reference" "H16"
-			(at 120.8445 189.2749 0)
+			(at 111.9545 189.2749 0)
 			(effects
 				(font
@@
 		)
 		(property "Value" "MountingHole"
-			(at 123.3845 189.2749 0)
+			(at 114.4945 189.2749 0)
 			(effects
 				(font
@@
 		)
 		(property "Footprint" "MountingHole:MountingHole_3.2mm_M3_DIN965_Pad"
-			(at 122.1146 191.8149 0)
+			(at 113.2246 191.8149 0)
 			(effects
 				(font
@@
 		)
 		(property "Datasheet" "~"
-			(at 122.1146 191.8149 0)
+			(at 113.2246 191.8149 0)
 			(effects
 				(font
@@
 		)
 		(property "Description" "Mounting Hole without connection"
-			(at 122.1146 191.8149 0)
+			(at 113.2246 191.8149 0)
 			(effects
 				(font
@@
 	(symbol
 		(lib_id "Mechanical:MountingHole")
-		(at 132.08 191.77 90)
+		(at 123.19 191.77 90)
 		(unit 1)
 		(exclude_from_sim yes)
@@
 		(dnp no)
 		(property "Reference" "H19"
-			(at 130.8099 189.23 0)
+			(at 121.9199 189.23 0)
 			(effects
 				(font
@@
 		)
 		(property "Value" "MountingHole"
-			(at 133.3499 189.23 0)
+			(at 124.4599 189.23 0)
 			(effects
 				(font
@@
 		)
 		(property "Footprint" "MountingHole:MountingHole_3.2mm_M3_DIN965_Pad"
-			(at 132.08 191.77 0)
+			(at 123.19 191.77 0)
 			(effects
 				(font
@@
 		)
 		(property "Datasheet" "~"
-			(at 132.08 191.77 0)
+			(at 123.19 191.77 0)
 			(effects
 				(font
@@
 		)
 		(property "Description" "Mounting Hole without connection"
-			(at 132.08 191.77 0)
+			(at 123.19 191.77 0)
 			(effects
 				(font
@@
 	(symbol
 		(lib_id "Mechanical:MountingHole")
-		(at 115.57 191.77 90)
+		(at 106.68 191.77 90)
 		(unit 1)
 		(exclude_from_sim yes)
@@
 		(dnp no)
 		(property "Reference" "H17"
-			(at 114.2999 189.23 0)
+			(at 105.4099 189.23 0)
 			(effects
 				(font
@@
 		)
 		(property "Value" "MountingHole"
-			(at 116.8399 189.23 0)
+			(at 107.9499 189.23 0)
 			(effects
 				(font
@@
 		)
 		(property "Footprint" "MountingHole:MountingHole_3.2mm_M3_DIN965_Pad"
-			(at 115.57 191.77 0)
+			(at 106.68 191.77 0)
 			(effects
 				(font
@@
 		)
 		(property "Datasheet" "~"
-			(at 115.57 191.77 0)
+			(at 106.68 191.77 0)
 			(effects
 				(font
@@
 		)
 		(property "Description" "Mounting Hole without connection"
-			(at 115.57 191.77 0)
+			(at 106.68 191.77 0)
 			(effects
 				(font
@@
 	(symbol
 		(lib_id "Mechanical:MountingHole")
-		(at 137.16 191.77 90)
+		(at 128.27 191.77 90)
 		(unit 1)
 		(exclude_from_sim yes)
@@
 		(dnp no)
 		(property "Reference" "H20"
-			(at 135.8899 189.23 0)
+			(at 126.9999 189.23 0)
 			(effects
 				(font
@@
 		)
 		(property "Value" "MountingHole"
-			(at 138.4299 189.23 0)
+			(at 129.5399 189.23 0)
 			(effects
 				(font
@@
 		)
 		(property "Footprint" "MountingHole:MountingHole_3.2mm_M3_DIN965_Pad"
-			(at 137.16 191.77 0)
+			(at 128.27 191.77 0)
 			(effects
 				(font
@@
 		)
 		(property "Datasheet" "~"
-			(at 137.16 191.77 0)
+			(at 128.27 191.77 0)
 			(effects
 				(font
@@
 		)
 		(property "Description" "Mounting Hole without connection"
-			(at 137.16 191.77 0)
+			(at 128.27 191.77 0)
 			(effects
 				(font
@@
 	(symbol
 		(lib_id "Mechanical:MountingHole")
-		(at 148.59 191.77 90)
+		(at 133.35 191.77 90)
 		(unit 1)
 		(exclude_from_sim yes)
@@
 		(dnp no)
 		(property "Reference" "H22"
-			(at 147.3199 189.23 0)
+			(at 132.0799 189.23 0)
 			(effects
 				(font
@@
 		)
 		(property "Value" "MountingHole"
-			(at 149.8599 189.23 0)
+			(at 134.6199 189.23 0)
 			(effects
 				(font
@@
 		)
 		(property "Footprint" "MountingHole:MountingHole_3.2mm_M3_DIN965_Pad"
-			(at 148.59 191.77 0)
+			(at 133.35 191.77 0)
 			(effects
 				(font
@@
 		)
 		(property "Datasheet" "~"
-			(at 148.59 191.77 0)
+			(at 133.35 191.77 0)
 			(effects
 				(font
@@
 		)
 		(property "Description" "Mounting Hole without connection"
-			(at 148.59 191.77 0)
+			(at 133.35 191.77 0)
 			(effects
 				(font
@@
 	(symbol
 		(lib_id "Mechanical:MountingHole")
-		(at 127 191.77 90)
+		(at 118.11 191.77 90)
 		(unit 1)
 		(exclude_from_sim yes)
@@
 		(dnp no)
 		(property "Reference" "H18"
-			(at 125.7299 189.23 0)
+			(at 116.8399 189.23 0)
 			(effects
 				(font
@@
 		)
 		(property "Value" "MountingHole"
-			(at 128.2699 189.23 0)
+			(at 119.3799 189.23 0)
 			(effects
 				(font
@@
 		)
 		(property "Footprint" "MountingHole:MountingHole_3.2mm_M3_DIN965_Pad"
-			(at 127 191.77 0)
+			(at 118.11 191.77 0)
 			(effects
 				(font
@@
 		)
 		(property "Datasheet" "~"
-			(at 127 191.77 0)
+			(at 118.11 191.77 0)
 			(effects
 				(font
@@
 		)
 		(property "Description" "Mounting Hole without connection"
-			(at 127 191.77 0)
+			(at 118.11 191.77 0)
 			(effects
 				(font
@@
 					(unit 1)
 				)
-			)
-		)
-	)
-	(symbol
-		(lib_id "Mechanical:MountingHole")
-		(at 142.24 191.77 90)
-		(unit 1)
-		(exclude_from_sim yes)
-		(in_bom no)
-		(on_board yes)
-		(dnp no)
-		(property "Reference" "H21"
-			(at 140.9699 189.23 0)
-			(effects
-				(font
-					(size 1.27 1.27)
-				)
-				(justify left)
-			)
-		)
-		(property "Value" "MountingHole"
-			(at 143.5099 189.23 0)
-			(effects
-				(font
-					(size 1.27 1.27)
-				)
-				(justify left)
-			)
-		)
-		(property "Footprint" "MountingHole:MountingHole_3.2mm_M3_DIN965_Pad"
-			(at 142.24 191.77 0)
-			(effects
-				(font
-					(size 1.27 1.27)
-				)
-				(hide yes)
-			)
-		)
-		(property "Datasheet" "~"
-			(at 142.24 191.77 0)
-			(effects
-				(font
-					(size 1.27 1.27)
-				)
-				(hide yes)
-			)
-		)
-		(property "Description" "Mounting Hole without connection"
-			(at 142.24 191.77 0)
-			(effects
-				(font
-					(size 1.27 1.27)
-				)
-				(hide yes)
-			)
-		)
-		(instances
-			(project "Layer_2"
-				(path "/164539e9-489b-4b17-b405-637c12a94360"
-					(reference "H21")
-					(unit 1)
-				)
