File: Electrical/PCB V2 ( 26 Nov)/L2/Layer_2/Layer_2.kicad_sch (KiCad schematic)
At the start: 79 parts, among them J1 Conn_01x02, J2 Conn_01x02, J3 XT60-M, Q1 AON6354, Q2 AON6354, Q3 AON6354, Q4 AON6354, SW1 SW_Push, SW2 SW_Nidec_CAS-120A1, U1 LM2596ADJ, U12 VNH5019ATR-E, U2 LM2596ADJ, U3 XT30UPB-M, U4 XT30UPB-M, U6 VNH5019ATR-E, U7 VNH5019ATR-E, U8 VNH5019ATR-E

Commit message: to be done : solve the teensy mystyery
Parts:
- removed J1, J2: Conn_01x02, Connector_PinHeader_1.00mm:PinHeader_1x02_P1.00mm_Horizontal, symbol Connector_Generic:Conn_01x02
- A1: footprint Sen Robo:Teensy 4.0 -> DEV-15583:MODULE_DEV-15583; symbol Teensy 4.0:TEENSY_4.0 -> Teensy 4.0:DEV-15583; Availability Not in stock -> In Stock; Check_prices https://www.snapeda.com/parts/Teensy%204.0/PJRC/view-part/?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 -> https://www.snapeda.com/parts/DEV-15583/SparkFun/view-part/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; Description_1 (none) -> RT1062 Teensy 4.0 series ARM® Cortex®-M7 MPU Embedded Evalu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; MANUFACTURER (none) -> Sparkfun; MAXIMUM_PACKAGE_HEIGHT (none) -> 5.87mm; MF PJRC -> SparkFun Electronics; MP Teensy 4.0 -> DEV-15583; STANDARD (none) -> Manufacturer Recommendations; SnapEDA_Link https://www.snapeda.com/parts/Teensy%204.0/PJRC/view-part/?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 -> https://www.snapeda.com/parts/DEV-15583/SparkFun/view-part/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
- SW1: renamed from SW2; footprint Button_Switch_SMD:Nidec_Copal_CAS-120A -> Connector_PinHeader_1.00mm:PinHeader_1x03_P1.00mm_Vertical
- SW2: renamed from SW1; footprint flipswitch:SW_100SP1T1B4M2QE -> Connector_PinHeader_1.00mm:PinHeader_1x03_P1.00mm_Vertical
- renumbered H2 to H1, H4 to H10, H3 to H11, H8 to H12, H7 to H13, H12 to H14, H17 to H15, H18 to H17, H19 to H18, H20 to H19, H1 to H2, H22 to H20, H6 to H3, H5 to H4, H10 to H5, H9 to H6, H14 to H7, H13 to H8, H15 to H9, J3 to J1, R8 to R1, R9 to R10, R10 to R11, R11 to R12, R12 to R13, R13 to R14, R14 to R15, R15 to R16, R16 to R17, R17 to R18, R18 to R19, R7 to R2, R19 to R20, R20 to R21, R21 to R22, R22 to R23, R23 to R24, R24 to R25, R25 to R26, R26 to R27, R27 to R28, R28 to R29, R6 to R3, R29 to R30, R30 to R31, R31 to R32, R32 to R33, R5 to R4, R4 to R5, R3 to R6, R1 to R7, R2 to R8, R33 to R9, U2 to U1, U1 to U2, U12 to U3, U3 to U4, U4 to U5
Connections:
- net 5v is gone; now on net +5V: U2.2 (OUT), U4.P$1 (+)
- net +12V: now also J1.P (POS), U1.1 (VIN), U2.1 (VIN); no longer Q1.1 (S), Q1.2 (S), Q1.3 (S), Q2.1 (S), Q2.2 (S), Q2.3 (S), Q3.1 (S), Q3.2 (S), Q3.3 (S), Q4.1 (S), Q4.2 (S), Q4.3 (S), U3.12 (VBAT), U6.12 (VBAT), U7.12 (VBAT), U8.12 (VBAT)
- net +3V3: now also A1.3.3V_1, A1.3.3V_2
- net 12v: no longer J1.P (POS), U1.1 (VIN), U2.1 (VIN)
- net GND: now also A1.G1, A1.G2, A1.G3; no longer A1.AGND/GND (GND), A1.GND
- net Motor Driver: now also SW1.2 (B)
- net PWM Motor 1: now also A1.3
- net PWM Motor 2: now also A1.2; no longer R20.1, R25.1
- net PWM Motor 4: now also A1.0
- net +5V: now reaches A1.VIN
- net Motor 1 ENA renamed Motor 1 EN A
- net Motor 1 EN A: now also A1.13
- net Motor 1 ENB renamed Motor 1 EN B
- net Motor 1 EN B: now also A1.20
- net Motor 2 ENA renamed Motor 2 EN A
- net Motor 2 EN A: now also A1.19
- net Motor 2 ENB renamed Motor 2 EN B
- net Motor 2 EN B: now also A1.18
- net Motor 3 ENA renamed Motor 3 EN A
- net Motor 3 EN A: now also A1.17
- net Motor 3 ENB renamed Motor 3 EN B
- net Motor 3 EN B: now also A1.16
- net Motor 4 ENA renamed Motor 4 EN A
- net Motor 4 EN A: now also A1.15
- net Motor 4 ENB renamed Motor 4 EN B
- net Motor 4 EN B: now also A1.14
- new net 12V: Q1.1 (S), Q1.2 (S), Q1.3 (S), Q2.1 (S), Q2.2 (S), Q2.3 (S), Q3.1 (S), Q3.2 (S), Q3.3 (S), Q4.1 (S), Q4.2 (S), Q4.3 (S), U3.12 (VBAT), U6.12 (VBAT), U7.12 (VBAT), U8.12 (VBAT)
- new net PWM Motor 3: A1.1, R20.1, R25.1
- no-connect marks 12 -> 27
Other:
- note added: "Pull Up"
- moved on the sheet: R9, SW1
