File: Electrical/PCB V3 (21 Jan)/Layer 2/Layer 2/_autosave-Layer 2.kicad_pcb (KiCad board)
At the start: 2 copper layers, 180 x 172.1 mm, 74 parts, among them J1 XT60-M, Q1 AON6354, Q2 AON6354, Q3 AON6354, Q4 AON6354, SW1 SW_Nidec_CAS-120A1, U3 VNH5019ATR-E, U4 XT30UPB-M, U5 XT30UPB-M, U6 VNH5019ATR-E, U7 VNH5019ATR-E, U8 VNH5019ATR-E

Commit message: idk what this is either
Parts:
- moved H1 145.2 mm to (87.1, 78.9)
Other:
- outline, holes or cut-outs redrawn
