File: Electrical/PCB V3 (21 Jan)/Layer 2/Layer 2/_autosave-Layer 2.kicad_pcb (KiCad board)
At the start: 2 copper layers, 178 x 170 mm, 95 parts, among them J1 Conn_01x04, J2 Conn_02x04_Counter_Clockwise, J3 XT60-M, Q1 AON6354, Q2 AON6354, Q3 AON6354, Q4 AON6354, SW1 SW_Nidec_CAS-120A1, U1 XT30UPB-M, U10 XT30UPB-M, U11 XT30UPB-M, U12 TPS5430DDAG4, U2 LM2596S-3.3, U3 VNH5019ATR-E, U4 XT30UPB-M, U5 XT30UPB-M, U6 VNH5019ATR-E, U7 VNH5019ATR-E, U8 VNH5019ATR-E, U9 LM2587S-ADJ

Commit message: yes
Connections:
- A1 pad 14: /TX1 -> /TX (CAM)
- A1 pad 15: /RX1 -> /RX (CAM)
- A1 pad 16: /RX2 -> /RX (IMU)
- A1 pad 17: /TX2 -> /TX (IMU)
- A1 pad 20: /TX1 -> / TX (L3 ESP 32)
- A1 pad 21: /RX3 -> / RX (L3 ESP 32)
- A1 pad 22: unconnected-(A1-Pad22) -> /Motor 2 EN B
- A1 pad 23: unconnected-(A1-Pad23) -> /Motor 3 EN A
- A1 pad 7: /Motor 2 EN B -> /L1 RX
- A1 pad 8: /Motor 3 EN A -> /L1 TX
Routing:
- net /Motor 1 EN A: track 37.9 -> 66.6 mm
- net Net-(D1-K): track 0.00 -> 18.7 mm
- added copper zone on F.Cu, net Net-(D3-A)

Commit message: kicad crashed ufekg still have like 70  errors
Parts:
- moved C10 0.07 mm to (56.9, 119.1)
Routing:
- net /L1 RX: track 0.00 -> 135.3 mm, vias 0 -> 2
- net /L1 TX: track 0.00 -> 130.6 mm, vias 0 -> 2
- net /PWM Motor 2: track 0.00 -> 117.8 mm, vias 0 -> 4
- net /Motor 2 EN A: track 2.23 -> 116.6 mm, vias 0 -> 7
- net /Motor 4 EN B: track 2.13 -> 112.1 mm, vias 0 -> 2
- net /PWM Motor 1: track 0.00 -> 98.2 mm, vias 0 -> 4
- net /Motor 1 EN B: track 21.0 -> 109.4 mm, vias 2 -> 5
- net +3V3: track 271.7 -> 341.4 mm, vias 3 -> 10
- net /Motor 3 EN A: track 99.8 -> 44.1 mm, vias 3 -> 0
- net /Motor 2 EN B: track 2.16 -> 54.3 mm, vias 0 -> 2
- net / RX (L3 ESP 32): track 0.00 -> 27.4 mm
- net / TX (L3 ESP 32): track 0.00 -> 21.5 mm
- net /TX (IMU): track 0.00 -> 18.2 mm
- net /RX (IMU): track 0.00 -> 16.2 mm
- net /RX (CAM): track 0.00 -> 15.4 mm
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