File: Electrical/PCB V3 (21 Jan)/Layer 2/Layer 2/_autosave-Layer 2.kicad_pcb (KiCad board)
At the start: 2 copper layers, 178 x 170 mm, 91 parts, among them J1 XT60-M, J2 Conn_02x04_Odd_Even, J3 Conn_01x04, J5 Conn_01x02, Q1 AON6354, Q2 AON6354, Q3 AON6354, Q4 AON6354, SW2 SW_SPST, SW3 SW_SPST, U1 VNH5019ATR-E, U12 VNH5019ATR-E, U2 TPS5430DDAG4, U3 TPS5430DDAG4, U4 XT30UPB-M, U5 VNH5019ATR-E, U6 XT30UPB-M, U7 XT30UPB-M, U8 XT30UPB-M, U9 VNH5019ATR-E

Commit message: dshxkvfsdk half way done want to sleep
Parts:
- removed C10, C14, C7: 470u, Sen Robo:CP_Radial_D8.0mm_P3.50mm
- removed H11, H16, H3, H7: MountingHole, MountingHole:MountingHole_3.2mm_M3_DIN965_Pad
- removed Q2, Q3, Q4: AON6354, Sen Robo:8-DFN (5x6)
- removed R12, R20, R21, R29, R30: 3K3, Sen Robo:res0603
- removed R22, R31: 10K, Sen Robo:res0603
- removed R23, R24, R25, R26, R27, R32, R33, R34, R35, R36: 1K, Sen Robo:res0603
- removed U12, U9: VNH5019ATR-E, layer2v3:fixed -onenew-newer-newest
- removed U7, U8: XT30UPB-M, layer2v3:XT30UPB-M
- added C4: 470u, Sen Robo:CP_Radial_D8.0mm_P3.50mm, B.Cu at (154.7, 145.9)
- added Q1: AON6354, Sen Robo:8-DFN (5x6), B.Cu at (165.2, 138.6)
- added R1: 3K3, Sen Robo:res0603, B.Cu at (172.1, 133.3)
- moved R18 123.7 mm to (164.2, 129.6), turned to 90 degrees
- moved R19 121.6 mm to (168.1, 129.5), turned to 90 degrees
- moved R16 119.5 mm to (166.2, 129.5), turned to 90 degrees
- moved R13 119.3 mm to (164.3, 133.3), turned to -90 degrees
- moved U4 118.8 mm to (177.2, 116.4), turned to 90 degrees
- moved R14 116.8 mm to (168.2, 133.3), turned to -90 degrees
- moved R17 115.4 mm to (172.1, 129.6), turned to 90 degrees
- moved R15 114.7 mm to (170.1, 129.5), turned to 90 degrees
- moved J2 102.1 mm to (180.7, 152.9), turned to 90 degrees
- moved U5 91.9 mm to (165.8, 117.6), turned to 90 degrees
- moved Q1 7.04 mm to (135.1, 134.0)
- moved R1 7.04 mm to (142.0, 128.7)
- moved R3 7.04 mm to (138.0, 128.7)
- moved R4 7.04 mm to (140.0, 125.0)
- moved R5 7.04 mm to (136.1, 124.9)
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Connections:
- R17 pad 1: /Motor 2 EN A -> /Motor 1 EN A
Routing:
- net +3V3: track 97.5 -> 166.4 mm, vias 7 -> 9
- net /PWM Motor 2: track 40.6 -> 89.5 mm, vias 0 -> 2
- net /Motor Driver: track 63.0 -> 109.2 mm, vias 4 -> 8
- net /PWM Motor 1: track 78.6 -> 107.5 mm, vias 2 -> 8
- net /TX (IMU): track 0.00 -> 16.9 mm, vias 0 -> 1
- net / RX (L3 ESP 32): track 0.00 -> 13.8 mm
- net / TX (L3 ESP 32): track 0.00 -> 13.8 mm
- net /RX (IMU): track 0.00 -> 12.5 mm
- net Net-(C4-Pad1): track 0.00 -> 9.25 mm, vias 0 -> 1
- net /RX (CAM): track 0.00 -> 7.82 mm
- net /TX (CAM): track 0.00 -> 7.78 mm
- net /Motor 2 EN B: track 71.5 -> 77.9 mm, vias 1 -> 2
- net /Motor 1 EN B: track 24.7 -> 30.5 mm, vias 0 -> 1
- net +12V: track 193.0 -> 197.6 mm
- net Net-(U5-INA): track 0.00 -> 3.45 mm
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- added copper zone on B.Cu, net /Motor 1 Out B
- added copper zone on B.Cu, net Net-(C7-Pad1)
