File: Electrical/PCB V3 (21 Jan)/Layer 2/Layer 2/Layer 2.kicad_pcb (KiCad board)
At the start: 2 copper layers, 74 parts, among them J1 XT60-M, Q1 AON6354, Q2 AON6354, Q3 AON6354, Q4 AON6354, SW1 SW_Nidec_CAS-120A1, U3 VNH5019ATR-E, U4 XT30UPB-M, U5 XT30UPB-M, U6 VNH5019ATR-E, U7 VNH5019ATR-E, U8 VNH5019ATR-E

Commit message: idk this too
Parts:
- removed C5, C7: 470u, Sen Robo:CP_Radial_D8.0mm_P3.50mm
- removed J1: XT60-M, layer2v3:AMASS_XT60-M
- added U2: LM2596S-3.3, Package_TO_SOT_SMD:TO-263-5_TabPin3, F.Cu at (313.8, 128.1)
- added U9: XT30UPB-M, layer2v3:AMASS_XT60-M, F.Cu at (114.0, 106.2)
- moved H1 145.2 mm to (87.1, 78.9)
- moved A1 143.1 mm to (186.7, 46.7)
- moved U3 143.1 mm to (244.6, 27.8)
- moved U6 143.1 mm to (244.6, 46.5)
- moved U7 143.1 mm to (244.6, 65.3)
- moved U8 143.1 mm to (244.6, 84.0)
- moved U4 143.1 mm to (260.8, 69.1)
- moved U5 143.1 mm to (260.8, 75.4)
Connections:
- C2 pad 1: Net-(C1-Pad1) -> Net-(C2-Pad1)
- C4 pad 1: Net-(C3-Pad1) -> Net-(C4-Pad1)
- Q1 pad 5: Net-(C1-Pad1) -> Net-(C2-Pad1)
- Q1 pad 6: Net-(C1-Pad1) -> Net-(C2-Pad1)
- Q1 pad 7: Net-(C1-Pad1) -> Net-(C2-Pad1)
- Q1 pad 8: Net-(C1-Pad1) -> Net-(C2-Pad1)
- Q1 pad 9: Net-(C1-Pad1) -> Net-(C2-Pad1)
- Q2 pad 5: Net-(C3-Pad1) -> Net-(C4-Pad1)
- Q2 pad 6: Net-(C3-Pad1) -> Net-(C4-Pad1)
- Q2 pad 7: Net-(C3-Pad1) -> Net-(C4-Pad1)
- Q2 pad 8: Net-(C3-Pad1) -> Net-(C4-Pad1)
- Q2 pad 9: Net-(C3-Pad1) -> Net-(C4-Pad1)
- R13 pad 1: /Motor 2 EN A -> /Motor Driver
- R14 pad 1: /Motor 2 EN B -> /Motor Driver
- R15 pad 1: /Motor Driver -> /Motor 2 EN A
- R16 pad 1: /Motor Driver -> /Motor 2 EN B
- R21 pad 1: /Motor 3 EN A -> /Motor Driver
- R22 pad 1: /Motor 3 EN B -> /Motor Driver
- R23 pad 1: /Motor Driver -> /Motor 3 EN A
- R24 pad 1: /Motor Driver -> /Motor 3 EN B
- R26 pad 1: /Motor 4 EN A -> /Motor 4 EN B
- R29 pad 1: /Motor 4 EN A -> /Motor Driver
- R30 pad 1: /Motor 4 EN B -> /Motor Driver
- R31 pad 1: /Motor Driver -> /Motor 4 EN A
- R32 pad 1: /Motor Driver -> /Motor 4 EN B
- U3 pad 13: Net-(C1-Pad1) -> Net-(C2-Pad1)
- U3 pad 23: Net-(C1-Pad1) -> Net-(C2-Pad1)
- U3 pad 3: Net-(C1-Pad1) -> Net-(C2-Pad1)
- U3 pad HS1: Net-(C1-Pad1) -> Net-(C2-Pad1)
- U6 pad 13: Net-(C3-Pad1) -> Net-(C4-Pad1)
- U6 pad 23: Net-(C3-Pad1) -> Net-(C4-Pad1)
- U6 pad 3: Net-(C3-Pad1) -> Net-(C4-Pad1)
- U6 pad HS1: Net-(C3-Pad1) -> Net-(C4-Pad1)
Other:
- board outline added: 180 x 172.1 mm

Commit message: lmao cx
Other:
- board outline removed

Commit message: 3 frivers add
Parts:
- removed H17, H18, H19, H20: MountingHole, MountingHole:MountingHole_3.2mm_M3_DIN965_Pad
- C1, C2, C3, C4, C6, C8, Q1, Q2, Q3, Q4, R1, R10, R11, R12, R13, R14, R15, R16, R17, R18, R19, R2, R20, R21, R22, R23, R24, R25, R26, R27, R28, R29, R3, R30, R31, R32, R33, R4, R5, R6, R7, R8, R9, U3, U6, U7, U8: moved to B.Cu
- moved H7 206.6 mm to (32.2, 205.9)
- moved H8 197.7 mm to (32.2, 159.3)
- moved U6 185.6 mm to (106.4, 170.4), turned to 180 degrees
- moved U7 184.4 mm to (122.1, 203.1)
- moved R19 184.0 mm to (99.7, 206.4), turned to 180 degrees
- moved H6 180.8 mm to (83.2, 244.1)
- moved R20 176.9 mm to (98.8, 188.0), turned to 180 degrees
- moved U3 176.8 mm to (106.2, 137.8), turned to 180 degrees
- moved R22 172.5 mm to (104.3, 196.2), turned to 180 degrees
- moved R23 172.5 mm to (104.3, 199.1), turned to 180 degrees
- moved R24 172.5 mm to (104.3, 202.0), turned to 180 degrees
- moved R25 172.5 mm to (104.3, 204.9), turned to 180 degrees
- moved H14 170.5 mm to (90.7, 212.6)
- moved R21 170.2 mm to (104.6, 187.1), turned to 90 degrees
- moved R18 167.6 mm to (104.5, 209.8), turned to 180 degrees
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Connections:
- C2 pad 1: Net-(C2-Pad1) -> /12V
- Q1 pad 4: Net-(Q1-G) -> /12V
- Q1 pad 5: Net-(C2-Pad1) -> /12V
- Q1 pad 6: Net-(C2-Pad1) -> /12V
- Q1 pad 7: Net-(C2-Pad1) -> /12V
- Q1 pad 8: Net-(C2-Pad1) -> /12V
- Q1 pad 9: Net-(C2-Pad1) -> /12V
- U3 pad 13: Net-(C2-Pad1) -> /12V
- U3 pad 23: Net-(C2-Pad1) -> /12V
- U3 pad 3: Net-(C2-Pad1) -> /12V
- U3 pad HS1: Net-(C2-Pad1) -> /12V
Routing:
- net /12V: track 0.00 -> 123.9 mm, vias 0 -> 4
- net GND: track 0.00 -> 94.5 mm, vias 0 -> 1
- net +3V3: track 0.00 -> 67.0 mm, vias 0 -> 1
- net Net-(C4-Pad1): track 0.00 -> 61.6 mm
- net /Motor Driver: track 0.00 -> 43.5 mm, vias 0 -> 2
- net /Motor 2 Out A: track 0.00 -> 27.5 mm
- net /Motor 1 Out A: track 0.00 -> 27.5 mm
- net /Motor 1 Out B: track 0.00 -> 27.5 mm
- net /Motor 2 Out B: track 0.00 -> 27.5 mm
- net Net-(Q2-G): track 0.00 -> 18.9 mm, vias 0 -> 2
- net Net-(U3-ENB/DIAGB): track 0.00 -> 16.8 mm
- net Net-(U3-INB): track 0.00 -> 16.4 mm, vias 0 -> 2
- net Net-(U3-PWM): track 0.00 -> 14.3 mm, vias 0 -> 2
- net Net-(U6-PWM): track 0.00 -> 13.8 mm, vias 0 -> 2
- net Net-(U6-INA): track 0.00 -> 13.7 mm, vias 0 -> 2
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- added copper zone on B.Cu, net GND
- added copper zone on F.Cu, net GND
Other:
- board outline added: 180 x 172.1 mm

Commit message: 2 motor controller
Parts:
- moved C6 119.3 mm to (109.3, 211.3), turned to 0 degrees
- moved Q3 100.6 mm to (122.3, 205.7), turned to -90 degrees
- moved Q4 99.7 mm to (247.2, 63.8)
- moved R27 99.7 mm to (287.2, 55.7)
- moved R28 99.7 mm to (282.5, 32.5)
- moved R31 99.7 mm to (282.5, 41.2)
- moved R32 99.7 mm to (282.5, 44.1)
- moved R33 99.7 mm to (282.5, 47.0)
- moved R9 99.7 mm to (296.6, 55.7)
- moved U2 99.7 mm to (339.2, 31.7)
- moved C1 99.7 mm to (277.9, 16.7)
- moved C3 99.7 mm to (268.3, 16.7)
- moved C8 99.7 mm to (242.2, 25.8)
- moved R26 99.7 mm to (287.2, 52.8)
- moved R30 99.7 mm to (282.5, 38.3)
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Connections:
- net /Motor 4 Out A renamed /Motor 4 Motor B
- C2 pad 1: /12V -> Net-(C2-Pad1)
- C4 pad 1: Net-(C4-Pad1) -> +12V
- Q1 pad 1: /12V -> +12V
- Q1 pad 2: /12V -> +12V
- Q1 pad 3: /12V -> +12V
- Q1 pad 4: /12V -> +12V
- Q1 pad 5: /12V -> +12V
- Q1 pad 6: /12V -> +12V
- Q1 pad 7: /12V -> +12V
- Q1 pad 8: /12V -> +12V
- Q1 pad 9: /12V -> +12V
- Q2 pad 1: /12V -> +12V
- Q2 pad 2: /12V -> +12V
- Q2 pad 3: /12V -> +12V
- Q2 pad 4: Net-(Q2-G) -> +12V
- Q2 pad 5: Net-(C4-Pad1) -> +12V
- Q2 pad 6: Net-(C4-Pad1) -> +12V
- Q2 pad 7: Net-(C4-Pad1) -> +12V
- Q2 pad 8: Net-(C4-Pad1) -> +12V
- Q2 pad 9: Net-(C4-Pad1) -> +12V
- Q3 pad 1: /12V -> +12V
- Q3 pad 2: /12V -> +12V
- Q3 pad 3: /12V -> +12V
- Q4 pad 1: /12V -> +12V
- Q4 pad 2: /12V -> +12V
- Q4 pad 3: /12V -> +12V
- U3 pad 11: Net-(Q1-G) -> +12V
- U3 pad 12: /12V -> +12V
- U3 pad 13: /12V -> Net-(C2-Pad1)
- U3 pad 15: /Motor 1 Out B -> /Motor 2 Out B
- U3 pad 16: /Motor 1 Out B -> /Motor 2 Out B
- U3 pad 21: /Motor 1 Out B -> /Motor 2 Out B
- U3 pad 23: /12V -> Net-(C2-Pad1)
- U3 pad 3: /12V -> Net-(C2-Pad1)
- U3 pad HS1: /12V -> Net-(C2-Pad1)
- U3 pad HS3: /Motor 1 Out B -> /Motor 2 Out B
- U6 pad 11: Net-(Q2-G) -> +12V
- U6 pad 12: /12V -> +12V
- U6 pad 15: /Motor 2 Out B -> /Motor 2 BOut 
- U6 pad 16: /Motor 2 Out B -> /Motor 2 BOut 
- U6 pad 21: /Motor 2 Out B -> /Motor 2 BOut 
- U6 pad HS3: /Motor 2 Out B -> /Motor 2 BOut 
- U7 pad 12: /12V -> +12V
- U8 pad 12: /12V -> +12V
Routing:
- net /12V: track 123.9 -> 0.00 mm, vias 4 -> 0
- net +12V: track 0.00 -> 109.8 mm, vias 0 -> 2
- net GND: track 94.5 -> 0.09 mm, vias 1 -> 0
- net Net-(C4-Pad1): track 61.6 -> 28.4 mm
- net Net-(C2-Pad1): track 0.00 -> 28.4 mm
- net /Motor 2 BOut : track 0.00 -> 27.5 mm
- net /Motor 1 Out B: track 27.5 -> 0.00 mm
- net Net-(Q2-G): track 18.9 -> 0.00 mm, vias 2 -> 0
- net +3V3: track 67.0 -> 79.0 mm, vias 1 -> 2
- net Net-(U7-ENA/DIAGA): track 0.00 -> 12.0 mm
- net Net-(U3-ENB/DIAGB): track 16.8 -> 5.64 mm
- net Net-(U6-INA): track 13.7 -> 4.71 mm, vias 2 -> 0
- net Net-(U3-INB): track 16.4 -> 7.79 mm, vias 2 -> 0
- net Net-(U3-PWM): track 14.3 -> 6.09 mm, vias 2 -> 0
- net Net-(U3-ENA/DIAGA): track 13.6 -> 6.18 mm
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- added copper zone on B.Cu, net +12V
- added copper zone on B.Cu, net Net-(C2-Pad1)
- added copper zone on B.Cu, net Net-(C4-Pad1)

Commit message: fix fills
Parts:
- moved U8 315.5 mm to (107.6, 225.9)
- moved R28 251.0 mm to (124.0, 227.1), turned to 0 degrees
- moved C8 250.9 mm to (113.9, 241.4)
- moved R30 249.0 mm to (120.3, 227.2)
- moved R29 247.9 mm to (120.2, 222.7)
- moved R32 246.1 mm to (120.3, 229.1)
- moved R31 242.2 mm to (120.2, 220.9)
- moved R33 240.7 mm to (120.3, 224.8)
- moved R26 240.2 mm to (124.2, 229.2), turned to 0 degrees
- moved R27 235.3 mm to (124.0, 225.2), turned to 0 degrees
- moved Q4 211.8 mm to (122.7, 235.3), turned to 0 degrees
- moved Q3 3.11 mm to (119.4, 206.9), turned to 0 degrees
- turned C6 to 180 degrees
Connections:
- C4 pad 1: +12V -> Net-(C4-Pad1)
- Q1 pad 4: +12V -> Net-(Q1-G)
- Q1 pad 5: +12V -> Net-(C2-Pad1)
- Q1 pad 6: +12V -> Net-(C2-Pad1)
- Q1 pad 7: +12V -> Net-(C2-Pad1)
- Q1 pad 8: +12V -> Net-(C2-Pad1)
- Q1 pad 9: +12V -> Net-(C2-Pad1)
- Q2 pad 4: +12V -> Net-(Q2-G)
- Q2 pad 5: +12V -> Net-(C4-Pad1)
- Q2 pad 6: +12V -> Net-(C4-Pad1)
- Q2 pad 7: +12V -> Net-(C4-Pad1)
- Q2 pad 8: +12V -> Net-(C4-Pad1)
- Q2 pad 9: +12V -> Net-(C4-Pad1)
- U3 pad 11: +12V -> Net-(Q1-G)
- U6 pad 11: +12V -> Net-(Q2-G)
Routing:
- net +3V3: track 79.0 -> 150.9 mm, vias 2 -> 3
- net /Motor Driver: track 46.5 -> 117.0 mm, vias 2 -> 4
- net Net-(C8-Pad1): track 0.00 -> 43.4 mm
- net Net-(C2-Pad1): track 28.4 -> 0.00 mm
- net /Motor 4 Out B: track 0.00 -> 27.5 mm
- net /Motor 4 Motor B: track 0.00 -> 27.5 mm
- net /Motor 2 BOut : track 27.5 -> 0.00 mm
- net Net-(C4-Pad1): track 28.4 -> 1.32 mm
- net +12V: track 109.8 -> 134.9 mm, vias 2 -> 5
- net /Motor 2 Out A: track 27.5 -> 3.06 mm
- net /Motor 2 Out B: track 27.5 -> 3.06 mm
- net /Motor 1 Out A: track 27.5 -> 3.06 mm
- net Net-(Q1-G): track 0.00 -> 20.2 mm
- net Net-(Q2-G): track 0.00 -> 18.5 mm
- net Net-(Q3-G): track 0.00 -> 16.9 mm
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- added copper zone on B.Cu, net /Motor 1 Out A
- added copper zone on B.Cu, net /Motor 2 BOut 
- added copper zone on B.Cu, net /Motor 2 Out A
- added copper zone on B.Cu, net /Motor 2 Out B
- added copper zone on B.Cu, net /Motor 4 Motor B
- added copper zone on B.Cu, net /Motor 4 Out B
- added copper zone on B.Cu, net Net-(C8-Pad1)

Commit message: tried
Parts:
- moved Q3 1.66 mm to (118.6, 205.4), turned to -90 degrees
Routing:
- net Net-(C8-Pad1): track 43.4 -> 1.35 mm
- net /Motor 4 Motor B: track 27.5 -> 7.07 mm
- net /Motor 4 Out B: track 27.5 -> 8.96 mm
- net Net-(Q3-G): track 16.9 -> 21.3 mm
- net Net-(C6-Pad1): track 2.24 -> 0.65 mm
- added copper zone on B.Cu, net /Motor 3 Out A
- removed copper zone on B.Cu, net /Motor 4 Motor B
- removed copper zone on B.Cu, net /Motor 4 Out B

Commit message: ignore this will be removed eventually
Routing:
- net +12V: track 134.9 -> 114.7 mm
- net Net-(Q4-G): track 9.57 -> 0.00 mm
- removed copper zone on B.Cu, net Net-(C8-Pad1)
Changed lines of the file:
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@@
 			(unlocked yes)
 			(layer "B.Fab")
+			(hide yes)
 			(effects
 				(font
@@
 	)
 	(segment
-		(start 124.655 231.95)
-		(end 122.905 230.2)
-		(width 0.2)
-		(layer "B.Cu")
-		(net 8)
-	)
-	(segment
-		(start 124.655 232.585)
-		(end 124.655 231.95)
-		(width 0.2)
-		(layer "B.Cu")
-		(net 8)
-	)
-	(segment
-		(start 122.905 230.2)
-		(end 119.0475 230.2)
-		(width 0.2)
-		(layer "B.Cu")
-		(net 8)
-	)
-	(segment
-		(start 117.6225 228.775)
-		(end 117.04 228.775)
-		(width 0.2)
-		(layer "B.Cu")
-		(net 8)
-	)
-	(segment
-		(start 119.0475 230.2)
-		(end 117.6225 228.775)
-		(width 0.2)
-		(layer "B.Cu")
-		(net 8)
-	)
-	(segment
 		(start 130.069998 134.629996)
 		(end 130.999998 135.559996)
@@
 	)
 	(segment
-		(start 115.37 214.65)
-		(end 115.21 214.49)
-		(width 1)
-		(layer "F.Cu")
-		(net 19)
-	)
-	(segment
 		(start 131.41 183.675)
 		(end 131.41 183.585)
@@
 	(segment
 		(start 126.17 219.324214)
-		(end 123.644214 221.85)
-		(width 1)
-		(layer "F.Cu")
-		(net 19)
-	)
-	(segment
-		(start 115.21 214.49)
-		(end 114.49 215.21)
-		(width 1)
-		(layer "F.Cu")
-		(net 19)
-	)
-	(segment
-		(start 120.24 219.274214)
-		(end 120.24 217.76)
+		(end 126.17 225.82)
 		(width 1)
 		(layer "F.Cu")
@@
 	)
 	(segment
-		(start 114.49 215.21)
-		(end 114.49 225.43)
-		(width 1)
-		(layer "F.Cu")
-		(net 19)
-	)
-	(segment
-		(start 120.24 217.14)
-		(end 117.75 214.65)
-		(width 1)
-		(layer "F.Cu")
-		(net 19)
-	)
-	(segment
-		(start 122.815786 221.85)
-		(end 120.24 219.274214)
-		(width 1)
-		(layer "F.Cu")
-		(net 19)
-	)
-	(segment
 		(start 141.49 168.58)
 		(end 134.45 168.58)
@@
 	)
 	(segment
-		(start 123.644214 221.85)
-		(end 122.815786 221.85)
-		(width 1)
-		(layer "F.Cu")
-		(net 19)
-	)
-	(segment
 		(start 131.14 183.405)
 		(end 131.41 183.675)
@@
 	)
 	(segment
-		(start 117.75 214.65)
-		(end 115.37 214.65)
-		(width 1)
-		(layer "F.Cu")
-		(net 19)
-	)
-	(segment
 		(start 134.46 183.355)
 		(end 134.23 183.585)
@@
 	)
 	(segment
-		(start 120.24 217.76)
-		(end 120.24 217.14)
+		(start 126.77 226.42)
+		(end 126.77 230.92)
 		(width 1)
 		(layer "F.Cu")
@@
 	)
 	(segment
-		(start 114.49 225.43)
-		(end 114.49 225.55)
+		(start 126.17 225.82)
+		(end 126.77 226.42)
 		(width 1)
 		(layer "F.Cu")
@@
 	)
 	(via
-		(at 114.49 225.43)
+		(at 126.77 230.92)
 		(size 0.6)
 		(drill 0.3)
@@
 	)
 	(segment
-		(start 114.49 228.14363)
-		(end 115.69 229.34363)
-		(width 1)
-		(layer "B.Cu")
-		(net 19)
-	)
-	(segment
 		(start 127.73 183.675)
 		(end 131.41 183.675)
@@
 	)
 	(segment
-		(start 114.49 225.43)
-		(end 114.49 228.14363)
-		(width 1)
-		(layer "B.Cu")
-		(net 19)
-	)
-	(segment
 		(start 128.905002 152.585001)
 		(end 128.905002 152.280001)
@@
 			)
 		)
-	)
-	(zone
-		(net 19)
-		(net_name "+12V")
-		(layer "B.Cu")
-		(hatch edge 0.5)
-		(priority 7)
-		(connect_pads yes
-			(clearance 0.2)
-		)
-		(min_thickness 0.2)
-		(filled_areas_thickness no)
-		(fill yes
-			(thermal_gap 0.5)
-			(thermal_bridge_width 0.5)
-			(smoothing chamfer)
-			(radius 0.5)
-		)
-		(polygon
-			(pts
-				(xy 123.86 233.49) (xy 123.81 233.54) (xy 120.14 233.54) (xy 120.14 231.71) (xy 118.71 230.28) (xy 116.07 230.28)
-				(xy 115.99 230.2) (xy 115.99 229.41) (xy 115.97 229.39) (xy 116.04 229.32) (xy 118.16 229.32) (xy 119.35 230.51)
-				(xy 122.93 230.51) (xy 123.86 231.44)
-			)
-		)
-	)
-	(zone
-		(net 62)
-		(net_name "Net-(C8-Pad1)")
-		(layer "B.Cu")
-		(hatch edge 0.5)
-		(priority 6)
-		(connect_pads
-			(clearance 0.2)
-		)
-		(min_thickness 0.25)
-		(filled_areas_thickness no)
-		(fill yes
-			(thermal_gap 0.5)
-			(thermal_bridge_width 0.5)
-		)
-		(polygon
-			(pts
-				(xy 125.28 233.87) (xy 125.28 238.9) (xy 124.89 239.29) (xy 120.25 239.29) (xy 116.81 242.73) (xy 114.57 242.73)
-				(xy 114.34 242.5) (xy 114.34 240.5) (xy 114.72 240.12) (xy 116.5 240.12) (xy 116.91 240.53) (xy 116.91 240.71)
-				(xy 117.12 240.71) (xy 119.5 238.33) (xy 119.5 233.68) (xy 117.54 231.72) (xy 117.54 231.33) (xy 116.08 231.33)
-				(xy 116.03 231.38) (xy 108.15 231.38) (xy 107.7 230.93) (xy 107.7 226.27) (xy 97.79 226.27) (xy 97.62 226.44)
-				(xy 97.6 226.42) (xy 97.6 225.39) (xy 97.63 225.36) (xy 107.64 225.36) (xy 107.68 225.32) (xy 107.68 220.16)
-				(xy 115.28 220.16) (xy 115.47 220.35) (xy 117.62 220.35) (xy 117.62 221.28) (xy 117.52 221.38) (xy 116 221.38)
-				(xy 115.87 221.51) (xy 115.87 230.34) (xy 115.92 230.39) (xy 117.68 230.39) (xy 117.71 230.36) (xy 117.78 230.36)
-				(xy 120.06 232.64) (xy 120.06 233.73) (xy 120.05 233.74) (xy 120.06 233.75) (xy 125.16 233.75)
-			)
-		)
-	)
-	(zone
-		(net 19)
-		(net_name "+12V")
-		(layer "B.Cu")
-		(hatch edge 0.5)
-		(priority 9)
-		(connect_pads yes
-			(clearance 0.2)
-		)
-		(min_thickness 0.2)
-		(filled_areas_thickness no)
-		(fill yes
-			(thermal_gap 0.5)
-			(thermal_bridge_width 0.5)
-			(smoothing chamfer)
-			(radius 0.5)
-		)
-		(polygon
-			(pts
-				(xy 117.87 230.22) (xy 119.03 231.38) (xy 119.66 230.75) (xy 119.66 230.67) (xy 119.02 230.03) (xy 118.06 230.03)
-			)
-		)

Commit message: mounting hole some issue idk
Parts:
- removed C1, C3: 470u, Sen Robo:CP_Radial_D8.0mm_P3.50mm
- C2, C4, C6, C8, Q1, Q2, Q3, Q4, R1, R10, R11, R12, R13, R14, R15, R16, R17, R18, R19, R2, R20, R21, R22, R23, R24, R25, R26, R27, R28, R29, R3, R30, R31, R32, R33, R4, R5, R6, R7, R8, R9, U3, U6, U7, U8: moved to F.Cu
- moved H7 333.4 mm to (345.0, 90.5)
- moved H8 318.8 mm to (345.0, 97.7)
- moved R28 311.4 mm to (370.0, 36.2)
- moved R30 310.8 mm to (370.0, 42.0), turned to 0 degrees
- moved R29 310.0 mm to (370.0, 39.1), turned to 0 degrees
- moved R32 308.6 mm to (370.0, 47.8), turned to 0 degrees
- moved H6 307.1 mm to (345.0, 83.4)
- moved R31 305.6 mm to (370.0, 44.9), turned to 0 degrees
- moved R33 304.4 mm to (370.0, 50.7), turned to 0 degrees
- moved H14 298.0 mm to (359.3, 83.4)
- moved R26 296.6 mm to (365.3, 56.5)
- moved H15 293.2 mm to (359.3, 90.5)
- moved R27 292.7 mm to (365.3, 59.4)
- moved R19 292.1 mm to (365.3, 36.2)
- moved R22 289.6 mm to (365.3, 44.9), turned to 0 degrees
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Routing:
- net +3V3: track 150.9 -> 0.00 mm, vias 3 -> 0
- net /Motor Driver: track 117.0 -> 0.00 mm, vias 4 -> 0
- net +12V: track 114.7 -> 0.00 mm, vias 5 -> 0
- net Net-(Q3-G): track 21.3 -> 0.00 mm
- net Net-(Q1-G): track 20.2 -> 0.00 mm
- net Net-(Q2-G): track 18.5 -> 0.00 mm
- net Net-(U6-PWM): track 17.5 -> 0.00 mm
- net Net-(U7-ENA/DIAGA): track 11.4 -> 0.00 mm
- net /PWM Motor 3: track 11.2 -> 0.00 mm
- net Net-(U3-INA): track 10.6 -> 0.00 mm
- net /Motor 4 Out B: track 8.96 -> 0.00 mm
- net Net-(U3-INB): track 7.79 -> 0.00 mm
- net /Motor 2 EN B: track 7.42 -> 0.00 mm
- net /Motor 4 Motor B: track 7.07 -> 0.00 mm
- net /Motor 4 EN B: track 6.81 -> 0.00 mm
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- removed copper zone on B.Cu, net +12V
- removed copper zone on B.Cu, net /Motor 1 Out A
- removed copper zone on B.Cu, net /Motor 2 BOut 
- removed copper zone on B.Cu, net /Motor 2 Out A
- removed copper zone on B.Cu, net /Motor 2 Out B
- removed copper zone on B.Cu, net /Motor 3 Out A
- removed copper zone on B.Cu, net Net-(C2-Pad1)
- removed copper zone on B.Cu, net Net-(C4-Pad1)
Other:
- board size 180 x 172.1 mm -> 178 x 170 mm
