File: Electrical/PCB V3 (21 Jan)/Layer 2/Layer 2/Layer 2.kicad_pcb (KiCad board)
At the start: 2 copper layers, 178 x 170 mm, 92 parts, among them J1 XT60-M, J2 Conn_02x04_Odd_Even, J3 Conn_01x04, J5 Conn_01x02, Q1 AON6354, Q2 AON6354, Q3 AON6354, Q4 AON6354, SW1 SW_Nidec_CAS-120A1, SW2 SW_SPST, U1 VNH5019ATR-E, U12 VNH5019ATR-E, U2 TPS5430DDAG4, U3 TPS5430DDAG4, U4 XT30UPB-M, U5 VNH5019ATR-E, U6 XT30UPB-M, U7 XT30UPB-M, U8 XT30UPB-M, U9 VNH5019ATR-E

Commit message: .
Routing:
- net /Motor 1 EN A: track 51.2 -> 54.2 mm
- net /PWM Motor 1: track 103.6 -> 105.6 mm
- net Net-(C8-Pad1): track 25.2 -> 23.8 mm
- net /Motor Driver: track 236.7 -> 235.7 mm
- net /Motor 3 EN B: track 93.5 -> 92.7 mm
Changed lines of the file:
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@@
 			(layer "F.Fab")
 		)
-		(fp_text user "GND"
-			(at -12.065 -16.256 180)
-			(layer "F.SilkS")
-			(effects
-				(font
-					(size 0.64 0.64)
-					(thickness 0.15)
-				)
-			)
-		)
-		(fp_text user "GND"
-			(at -12.065 -16.256 180)
-			(layer "F.Fab")
-			(effects
-				(font
-					(size 0.64 0.64)
-					(thickness 0.15)
-				)
-			)
-		)
 		(pad "0" thru_hole circle
 			(at -7.62 -13.97 180)
@@
 			(layer "F.CrtYd")
 		)
-		(fp_text user "${REFERENCE}"
-			(at 0 0 0)
-			(layer "F.Fab")
-			(effects
-				(font
-					(size 1 1)
-					(thickness 0.15)
-				)
-			)
-		)
 		(pad "1" thru_hole circle
 			(at 0 0)
@@
 	)
 	(segment
-		(start 153.314377 133.049321)
-		(end 152.749377 132.484321)
-		(width 0.2)
-		(layer "F.Cu")
-		(net 12)
-	)
-	(segment
 		(start 143.189377 111.234321)
 		(end 144.869377 111.234321)
@@
 	)
 	(segment
-		(start 180.659377 106.804321)
-		(end 181.819377 106.804321)
+		(start 203.485058 162.980004)
+		(end 202.779378 162.274324)
 		(width 0.2)
 		(layer "F.Cu")
@@
 	)
 	(segment
-		(start 203.485058 162.980004)
-		(end 202.779378 162.274324)
+		(start 190.809377 119.774321)
+		(end 197.739377 126.704321)
 		(width 0.2)
 		(layer "F.Cu")
@@
 	)
 	(segment
-		(start 201.289377 137.554321)
-		(end 201.889377 137.554321)
+		(start 185.589377 110.574321)
+		(end 185.589377 117.964321)
 		(width 0.2)
 		(layer "F.Cu")
@@
 	)
 	(segment
-		(start 190.809377 119.774321)
-		(end 197.739377 126.704321)
+		(start 180.659377 106.804321)
+		(end 181.819377 106.804321)
 		(width 0.2)
 		(layer "F.Cu")
@@
 	)
 	(segment
-		(start 181.819377 106.804321)
-		(end 186.179377 111.164321)
+		(start 197.739377 126.704321)
+		(end 197.739377 134.004321)
 		(width 0.2)
 		(layer "F.Cu")
@@
 	)
 	(segment
-		(start 197.739377 134.004321)
-		(end 201.289377 137.554321)
+		(start 185.589377 117.964321)
+		(end 187.399377 119.774321)
 		(width 0.2)
 		(layer "F.Cu")
@@
 	)
 	(segment
-		(start 204.969377 141.434321)
-		(end 218.249377 141.434321)
+		(start 201.289377 137.554321)
+		(end 201.889377 137.554321)
 		(width 0.2)
 		(layer "F.Cu")
@@
 	)
 	(segment
-		(start 197.739377 126.704321)
-		(end 197.739377 134.004321)
+		(start 204.969377 141.434321)
+		(end 218.249377 141.434321)
 		(width 0.2)
 		(layer "F.Cu")
@@
 	)
 	(segment
-		(start 186.179377 111.184321)
-		(end 190.809377 115.814321)
+		(start 187.399377 119.774321)
+		(end 190.809377 119.774321)
 		(width 0.2)
 		(layer "F.Cu")
@@
 	)
 	(segment
-		(start 186.179377 111.164321)
-		(end 186.179377 111.184321)
+		(start 197.739377 134.004321)
+		(end 201.289377 137.554321)
 		(width 0.2)
 		(layer "F.Cu")
@@
 	)
 	(segment
-		(start 190.809377 115.814321)
-		(end 190.809377 119.774321)
+		(start 181.819377 106.804321)
+		(end 185.589377 110.574321)
 		(width 0.2)
 		(layer "F.Cu")
@@
 	)
 	(segment
+		(start 191.759377 119.374321)
+		(end 199.519377 127.134321)
+		(width 0.2)
+		(layer "F.Cu")
+		(net 26)
+	)
+	(segment
 		(start 202.779377 139.414321)
 		(end 202.85 139.484944)
@@
 	)
 	(segment
+		(start 180.249377 105.984271)
+		(end 180.369427 106.104321)
+		(width 0.2)
+		(layer "F.Cu")
+		(net 26)
+	)
+	(segment
+		(start 180.249377 102.544321)
+		(end 180.249377 105.984271)
+		(width 0.2)
+		(layer "F.Cu")
+		(net 26)
+	)
+	(segment
+		(start 199.519377 134.194371)
+		(end 202.779377 137.454371)
+		(width 0.2)
+		(layer "F.Cu")
+		(net 26)
+	)
+	(segment
 		(start 202.779377 137.454371)
 		(end 202.779377 139.414321)
@@
 	)
 	(segment
+		(start 180.369427 106.104321)
+		(end 181.685063 106.104321)
+		(width 0.2)
+		(layer "F.Cu")
+		(net 26)
+	)
+	(segment
 		(start 199.519377 127.134321)
 		(end 199.519377 134.194371)
@@
 	)
 	(segment
-		(start 180.229377 103.074321)
-		(end 192.079377 114.924321)
+		(start 181.685063 106.104321)
+		(end 185.989377 110.408635)
 		(width 0.2)
 		(layer "F.Cu")
@@
 	)
 	(segment
-		(start 199.519377 134.194371)
-		(end 202.779377 137.454371)
+		(start 187.959377 119.374321)
+		(end 191.759377 119.374321)
 		(width 0.2)
 		(layer "F.Cu")
@@
 	)
 	(segment
-		(start 192.079377 119.694321)
-		(end 199.519377 127.134321)
+		(start 185.989377 110.408635)
+		(end 185.989377 117.404321)
 		(width 0.2)
 		(layer "F.Cu")
@@
 	(segment
 		(start 180.229377 102.524321)
-		(end 180.229377 103.074321)
+		(end 180.249377 102.544321)
 		(width 0.2)
 		(layer "F.Cu")
@@
 	)
 	(segment
-		(start 192.079377 114.924321)
-		(end 192.079377 119.694321)
+		(start 185.989377 117.404321)
+		(end 187.959377 119.374321)
 		(width 0.2)
 		(layer "F.Cu")
@@
 	)
 	(segment
-		(start 149.749377 83.584321)
-		(end 152.543296 80.790402)
-		(width 2.54)
-		(layer "B.Cu")
-		(net 31)
-	)
-	(segment
 		(start 175.029377 124.154321)
 		(end 175.079377 124.104321)
@@
 	)
 	(segment
+		(start 149.749377 83.584321)
+		(end 152.543296 80.790402)
+		(width 2.54)
+		(layer "B.Cu")
+		(net 31)
+	)
+	(segment
 		(start 139.199377 90.954321)
 		(end 139.289377 91.044321)
@@
 	)
 	(segment
-		(start 100.259377 150.314321)
-		(end 99.309377 150.314321)
-		(width 0.2)
-		(layer "F.Cu")
-		(net 45)
-	)
-	(segment
 		(start 169.779377 130.304321)
 		(end 158.009377 130.304321)
@@
 		(width 1.5)
 		(layer "B.Cu")
-		(net 91)
-	)
-	(segment
-		(start 164.293296 81.284321)
-		(end 164.293296 79.830402)
-		(width 1.5)
-		(layer "B.Cu")

Commit message: next jst
Parts:
- removed SW1: SW_Nidec_CAS-120A1, Connector_JST:JST_EH_B3B-EH-A_1x03_P2.50mm_Vertical
- added SW3: SW_SPST, Connector_JST:JST_XH_B2B-XH-A_1x02_P2.50mm_Vertical, F.Cu at (91.8, 150.2)
- moved R38 2.61 mm to (95.9, 145.7), turned to -90 degrees
Connections:
- R38 pad 1: Net-(SW1-C) -> GND
- R38 pad 2: GND -> /Motor Driver
Routing:
- net Net-(SW1-C): track 4.08 -> 0.00 mm
- net /Motor 2 EN A: track 66.9 -> 63.1 mm
- net +3V3: track 240.1 -> 243.5 mm
- net /Motor Driver: track 235.7 -> 238.0 mm, vias 9 -> 10
- net Net-(SW3-B): track 4.13 -> 2.58 mm
- net /Motor 1 EN B: track 48.0 -> 49.4 mm
- net /Motor 1 EN A: track 54.2 -> 53.7 mm
- net GND: vias 194 -> 193
Other:
- outline, holes or cut-outs redrawn

Commit message: me tired
Parts:
- moved U12 0.20 mm to (118.6, 151.3)
Routing:
- net +12V: track 339.5 -> 299.6 mm, vias 31 -> 10
- net /Motor Driver: track 238.0 -> 237.3 mm, vias 10 -> 16
- net +3V3: track 243.5 -> 243.7 mm, vias 2 -> 4
- net GND: vias 193 -> 25
- removed copper zone on B.Cu, net /Motor 3 Out A
- removed copper zone on B.Cu, net /Motor 3 Out B

Commit message: am i done im tired
Parts:
- J2: footprint Connector_JST:JST_EH_B8B-EH-A_1x08_P2.50mm_Vertical -> Connector_JST:JST_EH_B10B-EH-A_1x10_P2.50mm_Vertical
- SW2, U4, U6: moved to B.Cu
- moved R9 3.80 mm to (93.3, 156.7)
- moved A1 0.50 mm to (195.7, 155.9)
Routing:
- net +12V: track 299.6 -> 275.1 mm
- net +3V3: track 243.7 -> 255.7 mm, vias 4 -> 2
- net /Motor 2 EN A: track 63.1 -> 70.8 mm, vias 2 -> 4
- net /Motor Driver: track 237.3 -> 232.2 mm, vias 16 -> 15
- net /PWM Motor 1: track 105.8 -> 102.9 mm
- net /TX (IMU): track 17.4 -> 15.4 mm
- net +5V: track 105.0 -> 106.9 mm
- net /Motor 4 EN A: track 141.0 -> 142.9 mm
- net /Motor 1 EN A: track 53.7 -> 55.6 mm
- net /PWM Motor 3: track 136.7 -> 138.5 mm
- net Net-(SW3-B): track 2.58 -> 4.21 mm
- net /RX (IMU): track 13.6 -> 12.0 mm
- net /Motor 1 EN B: track 49.4 -> 50.6 mm
- net /TX (CAM): track 7.28 -> 7.78 mm
- net /RX (CAM): track 7.27 -> 7.77 mm
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- added copper zone on B.Cu, net /Motor 3 Out A
- added copper zone on B.Cu, net /Motor 3 Out B
- added copper zone on F.Cu, net Net-(C7-Pad1)

Commit message: did some touching up made traces less cursed with gnd fills in between and made schmeatics look better with aligned boxes
Routing:
- net /Motor Driver: track 232.2 -> 229.8 mm
- net /Motor 2 EN A: track 70.8 -> 72.5 mm
- net GND: vias 19 -> 18

Commit message: erm
Routing:
- net +12V: vias 10 -> 14
- net GND: vias 18 -> 17
