File: Electrical/PCB V3 (21 Jan)/Layer 2/Layer 2/Layer 2.kicad_sch (KiCad schematic)
At the start: 92 parts, among them J1 XT60-M, J2 Conn_02x04_Odd_Even, J3 Conn_01x04, J5 Conn_01x02, Q1 AON6354, Q2 AON6354, Q3 AON6354, Q4 AON6354, SW1 SW_Nidec_CAS-120A1, SW2 SW_SPST, U1 VNH5019ATR-E, U12 VNH5019ATR-E, U2 TPS5430DDAG4, U3 TPS5430DDAG4, U4 XT30UPB-M, U5 VNH5019ATR-E, U6 XT30UPB-M, U7 XT30UPB-M, U8 XT30UPB-M, U9 VNH5019ATR-E

Commit message: next jst
Parts:
- removed R38: 1K, Sen Robo:res0603, symbol Device:R
- removed SW1: SW_Nidec_CAS-120A1, Connector_JST:JST_EH_B3B-EH-A_1x03_P2.50mm_Vertical, symbol Switch:SW_Nidec_CAS-120A1
- added SW3: SW_SPST, Connector_JST:JST_XH_B2B-XH-A_1x02_P2.50mm_Vertical, symbol Switch:SW_SPST
Connections:
- net Motor Driver: now also SW3.1 (A)
- net at R9.1: now also SW3.2 (B)
Other:
- moved on the sheet: R9
Changed lines of the file:
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@@
 	)
 	(symbol
-		(lib_id "power:GND")
-		(at 55.88 233.68 90)
-		(unit 1)
-		(exclude_from_sim no)
-		(in_bom yes)
-		(on_board yes)
-		(dnp no)
-		(fields_autoplaced yes)
-		(property "Reference" "#PWR037"
-			(at 62.23 233.68 0)
-			(effects
-				(font
-					(size 1.27 1.27)
-				)
-				(hide yes)
-			)
-		)
-		(property "Value" "GND"
-			(at 59.69 233.6799 90)
-			(effects
-				(font
-					(size 1.27 1.27)
-				)
-				(justify right)
-			)
-		)
-		(property "Footprint" ""
-			(at 55.88 233.68 0)
-			(effects
-				(font
-					(size 1.27 1.27)
-				)
-				(hide yes)
-			)
-		)
-		(property "Datasheet" ""
-			(at 55.88 233.68 0)
-			(effects
-				(font
-					(size 1.27 1.27)
-				)
-				(hide yes)
-			)
-		)
-		(property "Description" "Power symbol creates a global label with name \"GND\" , ground"
-			(at 55.88 233.68 0)
-			(effects
-				(font
-					(size 1.27 1.27)
-				)
-				(hide yes)
-			)
-		)
-		(pin "1"
-		)
-		(instances
-			(project ""
-				(path "/73bb99ca-959f-40cf-90f8-36d6928b007b"
-					(reference "#PWR037")
-					(unit 1)
-				)
-			)
-		)
-	)
-	(symbol
 		(lib_id "Device:R")
 		(at 34.29 172.72 0)
@@
 	(symbol
 		(lib_id "Device:R")
-		(at 52.07 228.6 90)
+		(at 52.07 231.14 90)
 		(unit 1)
 		(exclude_from_sim no)
@@
 		(dnp no)
 		(property "Reference" "R9"
-			(at 52.07 226.06 90)
+			(at 52.07 228.6 90)
 			(effects
 				(font
@@
 		)
 		(property "Value" "1K"
-			(at 52.07 228.6 90)
+			(at 52.07 231.14 90)
 			(effects
 				(font
@@
 		)
 		(property "Footprint" "Sen Robo:res0603"
-			(at 52.07 230.378 90)
+			(at 52.07 232.918 90)
 			(effects
 				(font
@@
 		)
 		(property "Datasheet" "~"
-			(at 52.07 228.6 0)
+			(at 52.07 231.14 0)
 			(effects
 				(font
@@
 		)
 		(property "Description" ""
-			(at 52.07 228.6 0)
+			(at 52.07 231.14 0)
 			(effects
 				(font
@@
 	)
 	(symbol
-		(lib_id "Device:R")
-		(at 52.07 233.68 90)
-		(unit 1)
-		(exclude_from_sim no)
-		(in_bom yes)
-		(on_board yes)
-		(dnp no)
-		(property "Reference" "R38"
-			(at 52.07 231.14 90)
-			(effects
-				(font
-					(size 1.27 1.27)
-				)
-			)
-		)
-		(property "Value" "1K"
-			(at 52.07 233.68 90)
-			(effects
-				(font
-					(size 1.27 1.27)
-				)
-			)
-		)
-		(property "Footprint" "Sen Robo:res0603"
-			(at 52.07 235.458 90)
-			(effects
-				(font
-					(size 1.27 1.27)
-				)
-				(hide yes)
-			)
-		)
-		(property "Datasheet" "~"
-			(at 52.07 233.68 0)
-			(effects
-				(font
-					(size 1.27 1.27)
-				)
-				(hide yes)
-			)
-		)
-		(property "Description" ""
-			(at 52.07 233.68 0)
-			(effects
-				(font
-					(size 1.27 1.27)
-				)
-				(hide yes)
-			)
-		)
-		(pin "1"
-		)
-		(pin "2"
-		)
-		(instances
-			(project "Layer 2"
-				(path "/73bb99ca-959f-40cf-90f8-36d6928b007b"
-					(reference "R38")
-					(unit 1)
-				)
-			)
-		)
-	)
-	(symbol
 		(lib_id "Connector_Generic:Conn_01x04")
 		(at 274.32 214.63 180)
@@
 	)
 	(symbol
+		(lib_id "Switch:SW_SPST")
+		(at 43.18 231.14 0)
+		(unit 1)
+		(exclude_from_sim no)
+		(in_bom yes)
+		(on_board yes)
+		(dnp no)
+		(fields_autoplaced yes)
+		(property "Reference" "SW3"
+			(at 43.18 224.79 0)
+			(effects
+				(font
+					(size 1.27 1.27)
+				)
+			)
+		)
+		(property "Value" "SW_SPST"
+			(at 43.18 227.33 0)
+			(effects
+				(font
+					(size 1.27 1.27)
+				)
+			)
+		)
+		(property "Footprint" "Connector_JST:JST_XH_B2B-XH-A_1x02_P2.50mm_Vertical"
+			(at 43.18 231.14 0)
+			(effects
+				(font
+					(size 1.27 1.27)
+				)
+				(hide yes)
+			)
+		)
+		(property "Datasheet" "~"
+			(at 43.18 231.14 0)
+			(effects
+				(font
+					(size 1.27 1.27)
+				)
+				(hide yes)
+			)
+		)
+		(property "Description" "Single Pole Single Throw (SPST) switch"
+			(at 43.18 231.14 0)
+			(effects
+				(font
+					(size 1.27 1.27)
+				)
+				(hide yes)
+			)
+		)
+		(pin "1"
+		)
+		(pin "2"
+		)
+		(instances
+			(project "Layer 2"
+				(path "/73bb99ca-959f-40cf-90f8-36d6928b007b"
+					(reference "SW3")
+					(unit 1)
+				)
+			)
+		)
+	)
+	(symbol
 		(lib_id "Device:R")
 		(at 119.38 138.43 180)
@@
 	)
 	(symbol
-		(lib_id "Switch:SW_Nidec_CAS-120A1")
-		(at 43.18 231.14 0)
-		(unit 1)
-		(exclude_from_sim no)
-		(in_bom yes)
-		(on_board yes)
-		(dnp no)
-		(fields_autoplaced yes)
-		(property "Reference" "SW1"
-			(at 43.18 222.25 0)
-			(effects
-				(font
-					(size 1.27 1.27)
-				)
-			)
-		)
-		(property "Value" "SW_Nidec_CAS-120A1"
-			(at 43.18 224.79 0)
-			(effects
-				(font
-					(size 1.27 1.27)
-				)
-			)
-		)
-		(property "Footprint" "Connector_JST:JST_EH_B3B-EH-A_1x03_P2.50mm_Vertical"
-			(at 43.18 241.3 0)
-			(effects
-				(font
-					(size 1.27 1.27)
-				)
-				(hide yes)
-			)
-		)
-		(property "Datasheet" "https://www.nidec-components.com/e/catalog/switch/cas.pdf"
-			(at 43.18 238.76 0)
-			(effects
-				(font
-					(size 1.27 1.27)
-				)
-				(hide yes)
-			)
-		)
-		(property "Description" "Switch, single pole double throw"
-			(at 43.18 231.14 0)
-			(effects
-				(font
-					(size 1.27 1.27)
-				)
-				(hide yes)
-			)
-		)
-		(pin "2"
-		)
-		(pin "3"
-		)
-		(pin "1"
-		)
-		(instances
-			(project "Layer 2"
-				(path "/73bb99ca-959f-40cf-90f8-36d6928b007b"
-					(reference "SW1")
-					(unit 1)
-				)
-			)
-		)
-	)
-	(symbol
 		(lib_id "Mechanical:MountingHole")
 		(at 90.17 201.93 90)
@@
 	(symbol
 		(lib_id "power:+5V")
-		(at 55.88 228.6 270)
+		(at 55.88 231.14 270)
 		(unit 1)
 		(exclude_from_sim no)
@@
 		(fields_autoplaced yes)
 		(property "Reference" "#PWR05"
-			(at 52.07 228.6 0)
+			(at 52.07 231.14 0)
 			(effects
 				(font
@@
 		)
 		(property "Value" "+5V"
-			(at 59.69 228.5999 90)
+			(at 59.69 231.1399 90)
 			(effects
 				(font
@@
 		)
 		(property "Footprint" ""
-			(at 55.88 228.6 0)
+			(at 55.88 231.14 0)
 			(effects
 				(font
@@
 		)
 		(property "Datasheet" ""
-			(at 55.88 228.6 0)
+			(at 55.88 231.14 0)
 			(effects
 				(font
@@
 		)
 		(property "Description" "Power symbol creates a global label with name \"+5V\""
-			(at 55.88 228.6 0)
+			(at 55.88 231.14 0)
 			(effects
 				(font

Commit message: DHMN V D
Parts:
- added R38: 1K, Sen Robo:res0603, symbol Device:R
Connections:
- net GND: now also R38.1
- net Motor Driver: now also R38.2
Changed lines of the file:
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@@
 	)
 	(junction
+		(at 35.56 231.14)
+		(diameter 0)
+		(color 0 0 0 0)
+	)
+	(junction
 		(at 194.31 151.13)
 		(diameter 0)
@@
 	(wire
 		(pts
+			(xy 35.56 231.14) (xy 38.1 231.14)
+		)
+		(stroke
+			(width 0)
+			(type default)
+		)
+	)
+	(wire
+		(pts
 			(xy 97.79 173.99) (xy 97.79 172.72)
 		)
@@
 	(wire
 		(pts
-			(xy 31.75 231.14) (xy 38.1 231.14)
+			(xy 31.75 231.14) (xy 35.56 231.14)
 		)
 		(stroke
@@
 	)
 	(symbol
+		(lib_id "Device:R")
+		(at 35.56 234.95 180)
+		(unit 1)
+		(exclude_from_sim no)
+		(in_bom yes)
+		(on_board yes)
+		(dnp no)
+		(property "Reference" "R38"
+			(at 33.02 234.95 90)
+			(effects
+				(font
+					(size 1.27 1.27)
+				)
+			)
+		)
+		(property "Value" "1K"
+			(at 35.56 234.95 90)
+			(effects
+				(font
+					(size 1.27 1.27)
+				)
+			)
+		)
+		(property "Footprint" "Sen Robo:res0603"
+			(at 37.338 234.95 90)
+			(effects
+				(font
+					(size 1.27 1.27)
+				)
+				(hide yes)
+			)
+		)
+		(property "Datasheet" "~"
+			(at 35.56 234.95 0)
+			(effects
+				(font
+					(size 1.27 1.27)
+				)
+				(hide yes)
+			)
+		)
+		(property "Description" ""
+			(at 35.56 234.95 0)
+			(effects
+				(font
+					(size 1.27 1.27)
+				)
+				(hide yes)
+			)
+		)
+		(pin "1"
+		)
+		(pin "2"
+		)
+		(instances
+			(project "Layer 2"
+				(path "/73bb99ca-959f-40cf-90f8-36d6928b007b"
+					(reference "R38")
+					(unit 1)
+				)
+			)
+		)
+	)
+	(symbol
 		(lib_id "Device:C_Polarized")
 		(at 290.83 168.91 0)
@@
 					(unit 1)
 				)
+			)
+		)
+	)
+	(symbol
+		(lib_id "power:GND")
+		(at 35.56 238.76 0)
+		(unit 1)
+		(exclude_from_sim no)
+		(in_bom yes)
+		(on_board yes)
+		(dnp no)
+		(fields_autoplaced yes)
+		(property "Reference" "#PWR024"
+			(at 35.56 245.11 0)
+			(effects
+				(font
+					(size 1.27 1.27)
+				)
+				(hide yes)
+			)
+		)
+		(property "Value" "GND"
+			(at 35.56 243.84 0)
+			(effects
+				(font
+					(size 1.27 1.27)
+				)
+			)
+		)
+		(property "Footprint" ""
+			(at 35.56 238.76 0)
+			(effects
+				(font
+					(size 1.27 1.27)
+				)
+				(hide yes)
+			)
+		)
+		(property "Datasheet" ""
+			(at 35.56 238.76 0)
+			(effects
+				(font
+					(size 1.27 1.27)
+				)
+				(hide yes)
+			)
+		)
+		(property "Description" "Power symbol creates a global label with name \"GND\" , ground"
+			(at 35.56 238.76 0)
+			(effects
+				(font
+					(size 1.27 1.27)
+				)
+				(hide yes)
+			)
+		)
+		(pin "1"
+		)
+		(instances
+			(project ""
+				(path "/73bb99ca-959f-40cf-90f8-36d6928b007b"
+					(reference "#PWR024")
+					(unit 1)
+				)

Commit message: am i done im tired
Parts:
- J2: footprint Connector_JST:JST_EH_B8B-EH-A_1x08_P2.50mm_Vertical -> Connector_JST:JST_EH_B10B-EH-A_1x10_P2.50mm_Vertical
Changed lines of the file:
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@@
 			)
 		)
-		(property "Footprint" "Connector_JST:JST_EH_B8B-EH-A_1x08_P2.50mm_Vertical"
+		(property "Footprint" "Connector_JST:JST_EH_B10B-EH-A_1x10_P2.50mm_Vertical"
 			(at 110.49 238.76 0)
 			(effects

Commit message: did some touching up made traces less cursed with gnd fills in between and made schmeatics look better with aligned boxes
Other:
- note added: "2-Chairs."
- note added: "27 Febuary 2025"
- note added: "L1 Connections"
- note added: "L3 connection"
- note added: "Layer 2"
- note added: "Pull Up/ Down for Motor Drivers"
- note added: "V3"
- note removed: "L1 JST"
- note removed: "L3 JST"
- note removed: "Pull Up"
- moved on the sheet: A1, C1, C10, C14, C2, C3, C4, C5, C6, C7, C8, D1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

Commit message: m
Parts:
- TP1, TP2, TP3: footprint Custom Testpointverycool:testpoint_2pad_2-chairs. -> Custom Testpointverycool:14 AWG Testpoint
Connections:
- net +3V3: now also C8.1, L2.2, R28.1, TP3.1; no longer TP3.2
- net +5V: now also C5.1, L1.2, R10.1, TP2.1; no longer TP2.2
- net GND: now also TP2.2, TP3.2
Other:
- note added: "Test Points"
- moved on the sheet: TP2, TP3

Commit message: ok testpoints
Parts:
- TP1, TP3: footprint Custom Testpointverycool:14 AWG Testpoint -> Custom Testpointverycool:14 AWG Testpoint (Vertical)
Other:
- note removed: "Test Point 12V :(From XT60)"
- moved on the sheet: TP1, U4, U6, U7, U8

Commit message: erm moved 2 drivers flip
Parts:
- TP2: footprint Custom Testpointverycool:14 AWG Testpoint -> Custom Testpointverycool:14 AWG Testpoint (Vertical)
Changed lines of the file:
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@@
 			)
 		)
-		(property "Footprint" "Custom Testpointverycool:14 AWG Testpoint"
+		(property "Footprint" "Custom Testpointverycool:14 AWG Testpoint (Vertical)"
 			(at 260.35 189.23 0)
 			(effects

Commit message: fixed l2
Connections:
- net GND: no longer U3.6 (GND), U3.9 (POWER_PAD)
- net  RX (L3 ESP 32) renamed RX (L3 ESP 32)
- net  TX (L3 ESP 32) renamed TX (L3 ESP 32)
Other:
- moved on the sheet: C1, C10, C14, C2, C3, C4, C5, C6, C7, C8, D1, D2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
