File: Electrical/PCB V3 (21 Jan)/Layer 2/Layer 2/Layer 2.kicad_sch (KiCad schematic)
At the start: 86 parts, among them J1 XT60-M, J2 Conn_02x04_Odd_Even, J3 Conn_01x04, J5 Conn_01x02, Q1 AON6354, Q2 AON6354, Q3 AON6354, Q4 AON6354, SW2 SW_SPST, SW3 SW_SPST, U1 VNH5019ATR-E, U12 VNH5019ATR-E, U2 TPS5430DDAG4, U3 TPS5430DDAG4, U4 XT30UPB-M, U5 VNH5019ATR-E, U6 XT30UPB-M, U7 XT30UPB-M, U8 XT30UPB-M, U9 VNH5019ATR-E

Commit message: fixed l2
Parts:
- C10, C14, C4, C7: footprint Sen Robo:CP_Radial_D8.0mm_P3.50mm -> Capacitor_THT:CP_Radial_D8.0mm_P3.50mm
Changed lines of the file:
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@@
 	(label "Motor Driver"
 		(at 317.5 123.19 0)
-		(fields_autoplaced yes)
 		(effects
 			(font
@@
 	(label "Motor 1 EN B"
 		(at 171.45 52.07 0)
-		(fields_autoplaced yes)
 		(effects
 			(font
@@
 	(label "Motor 3 Out B"
 		(at 152.4 199.39 180)
-		(fields_autoplaced yes)
 		(effects
 			(font
@@
 	(label "Motor 2 EN B"
 		(at 171.45 57.15 0)
-		(fields_autoplaced yes)
 		(effects
 			(font
@@
 	(label "Motor 4 EN A"
 		(at 171.45 64.77 0)
-		(fields_autoplaced yes)
 		(effects
 			(font
@@
 	(label "Motor 1 EN A"
 		(at 26.67 128.27 0)
-		(fields_autoplaced yes)
 		(effects
 			(font
@@
 	(label "PWM Motor 4"
 		(at 171.45 80.01 0)
-		(fields_autoplaced yes)
 		(effects
 			(font
@@
 	(label "PWM Motor 2"
 		(at 120.65 140.97 0)
-		(fields_autoplaced yes)
 		(effects
 			(font
@@
 	(label "Motor 2 EN B"
 		(at 123.19 133.35 0)
-		(fields_autoplaced yes)
 		(effects
 			(font
@@
 	(label "Motor Driver"
 		(at 123.19 121.92 0)
-		(fields_autoplaced yes)
 		(effects
 			(font
@@
 	(label "Motor 2 Out A"
 		(at 177.8 179.07 180)
-		(fields_autoplaced yes)
 		(effects
 			(font
@@
 	(label "Motor 2 EN A"
 		(at 123.19 128.27 0)
-		(fields_autoplaced yes)
 		(effects
 			(font
@@
 	(label "Motor 1 Out B"
 		(at 96.52 133.35 180)
-		(fields_autoplaced yes)
 		(effects
 			(font
@@
 	(label "GND"
 		(at 171.45 82.55 0)
-		(fields_autoplaced yes)
 		(effects
 			(font
@@
 	(label "L1 RX"
 		(at 171.45 62.23 0)
-		(fields_autoplaced yes)
 		(effects
 			(font
@@
 	(label "RX (IMU)"
 		(at 135.89 57.15 180)
-		(fields_autoplaced yes)
 		(effects
 			(font
@@
 	(label "Motor 2 Out A"
 		(at 193.04 128.27 180)
-		(fields_autoplaced yes)
 		(effects
 			(font
@@
 	(label "PWM Motor 2"
 		(at 171.45 74.93 0)
-		(fields_autoplaced yes)
 		(effects
 			(font
@@
 	(label "Motor 4 Out A"
 		(at 387.35 129.54 180)
-		(fields_autoplaced yes)
 		(effects
 			(font
@@
 	(label "Motor 1 Out A"
 		(at 96.52 128.27 180)
-		(fields_autoplaced yes)
 		(effects
 			(font
@@
 	(label "TX (L3 ESP 32)"
 		(at 135.89 67.31 180)
-		(fields_autoplaced yes)
 		(effects
 			(font
@@
 	(label "Motor 2 Out B"
 		(at 193.04 133.35 180)
-		(fields_autoplaced yes)
 		(effects
 			(font
@@
 	(label "Motor 1 Out B"
 		(at 152.4 182.88 180)
-		(fields_autoplaced yes)
 		(effects
 			(font
@@
 	(label "TX (IMU)"
 		(at 135.89 59.69 180)
-		(fields_autoplaced yes)
 		(effects
 			(font
@@
 	(label "Motor 4 Out B"
 		(at 179.07 198.12 180)
-		(fields_autoplaced yes)
 		(effects
 			(font
@@
 	(label "Motor Driver"
 		(at 218.44 119.38 0)
-		(fields_autoplaced yes)
 		(effects
 			(font
@@
 	(label "RX (CAM)"
 		(at 135.89 54.61 180)
-		(fields_autoplaced yes)
 		(effects
 			(font
@@
 	(label "TX (L3 ESP 32)"
 		(at 72.39 185.42 0)
-		(fields_autoplaced yes)
 		(effects
 			(font
@@
 	(label "Motor 1 EN A"
 		(at 171.45 49.53 0)
-		(fields_autoplaced yes)
 		(effects
 			(font
@@
 	(label "Motor 3 EN B"
 		(at 135.89 74.93 180)
-		(fields_autoplaced yes)
 		(effects
 			(font
@@
 	(label "PWM Motor 3"
 		(at 171.45 77.47 0)
-		(fields_autoplaced yes)
 		(effects
 			(font
@@
 	(label "Motor 2 EN A"
 		(at 171.45 54.61 0)
-		(fields_autoplaced yes)
 		(effects
 			(font
@@
 	(label "RX (L3 ESP 32)"
 		(at 135.89 69.85 180)
-		(fields_autoplaced yes)
 		(effects
 			(font
@@
 	(label "Motor 4 EN B"
 		(at 171.45 67.31 0)
-		(fields_autoplaced yes)
 		(effects
 			(font
@@
 	(label "Motor Driver"
 		(at 16.51 173.99 0)
-		(fields_autoplaced yes)
 		(effects
 			(font
@@
 	(label "PWM Motor 3"
 		(at 217.17 138.43 0)
-		(fields_autoplaced yes)
 		(effects
 			(font
@@
 	(label "Motor 3 EN B"
 		(at 218.44 130.81 0)
-		(fields_autoplaced yes)
 		(effects
 			(font
@@
 	(label "Motor 1 Out A"
 		(at 152.4 180.34 180)
-		(fields_autoplaced yes)
 		(effects
 			(font
@@
 	(label "Motor 3 Out A"
 		(at 289.56 125.73 180)
-		(fields_autoplaced yes)
 		(effects
 			(font
@@
 	(label "Motor 4 EN B"
 		(at 317.5 134.62 0)
-		(fields_autoplaced yes)
 		(effects
 			(font
@@
 	(label "Motor 4 Out B"
 		(at 387.35 134.62 180)
-		(fields_autoplaced yes)
 		(effects
 			(font
@@
 	(label "RX (IMU)"
 		(at 72.39 193.04 0)
-		(fields_autoplaced yes)
 		(effects
 			(font
@@
 	(label "Motor 3 EN A"
 		(at 135.89 72.39 180)
-		(fields_autoplaced yes)
 		(effects
 			(font
@@
 	(label "RX (L3 ESP 32)"
 		(at 72.39 182.88 0)
-		(fields_autoplaced yes)
 		(effects
 			(font
@@
 	(label "Motor 2 Out B"
 		(at 177.8 181.61 180)
-		(fields_autoplaced yes)
 		(effects
 			(font
@@
 	(label "Motor Driver"
 		(at 26.67 121.92 0)
-		(fields_autoplaced yes)
 		(effects
 			(font
@@
 	(label "TX (CAM)"
 		(at 135.89 52.07 180)
-		(fields_autoplaced yes)
 		(effects
 			(font
@@
 	(label "L1 TX"
 		(at 207.01 181.61 180)
-		(fields_autoplaced yes)
 		(effects
 			(font
@@
 	(label "Motor 3 EN A"
 		(at 218.44 125.73 0)
-		(fields_autoplaced yes)
 		(effects
 			(font
@@
 	(label "L1 RX"
 		(at 207.01 179.07 180)
-		(fields_autoplaced yes)
 		(effects
 			(font
@@
 	(label "PWM Motor 4"
 		(at 314.96 142.24 0)
-		(fields_autoplaced yes)
 		(effects
 			(font
@@
 	(label "L1 TX"
 		(at 171.45 59.69 0)
-		(fields_autoplaced yes)
 		(effects
 			(font
@@
 	(label "Motor 3 Out B"
 		(at 289.56 130.81 180)
-		(fields_autoplaced yes)
 		(effects
 			(font
@@
 	(label "TX (CAM)"
 		(at 72.39 190.5 0)
-		(fields_autoplaced yes)
 		(effects
 			(font
@@
 	(label "Motor 4 EN A"
 		(at 317.5 129.54 0)
-		(fields_autoplaced yes)
 		(effects
 			(font
@@
 	(label "TX (IMU)"
 		(at 72.39 195.58 0)
-		(fields_autoplaced yes)
 		(effects
 			(font
@@
 	(label "Motor 1 EN B"
 		(at 26.67 133.35 0)
-		(fields_autoplaced yes)
 		(effects
 			(font
@@
 	(label "Motor 4 Out A"
 		(at 179.07 195.58 180)
-		(fields_autoplaced yes)
 		(effects
 			(font
@@
 	(label "RX (CAM)"
 		(at 72.39 187.96 0)
-		(fields_autoplaced yes)
 		(effects
 			(font
@@
 	(label "PWM Motor 1"
 		(at 24.13 140.97 0)
-		(fields_autoplaced yes)
 		(effects
 			(font
@@
 	(label "PWM Motor 1"
 		(at 171.45 72.39 0)
-		(fields_autoplaced yes)
 		(effects
 			(font
@@
 	(label "Motor 3 Out A"
 		(at 152.4 196.85 180)
-		(fields_autoplaced yes)
 		(effects
 			(font
@@
 			)
 		)
-		(property "Footprint" "Sen Robo:CP_Radial_D8.0mm_P3.50mm"
+		(property "Footprint" "Capacitor_THT:CP_Radial_D8.0mm_P3.50mm"
 			(at 100.0252 147.32 0)
 			(effects
@@
 			)
 		)
-		(property "Footprint" "Sen Robo:CP_Radial_D8.0mm_P3.50mm"
+		(property "Footprint" "Capacitor_THT:CP_Radial_D8.0mm_P3.50mm"
 			(at 293.0652 144.78 0)
 			(effects
@@
 		(dnp no)
 		(property "Reference" "R20"
-			(at 224.79 110.744 0)
+			(at 218.948 110.744 0)
 			(effects
 				(font
@@
 		)
 		(property "Value" "3K3"
-			(at 224.028 113.03 0)
+			(at 218.948 112.776 0)
 			(effects
 				(font
@@
 			)
 		)
-		(property "Footprint" "Sen Robo:CP_Radial_D8.0mm_P3.50mm"
+		(property "Footprint" "Capacitor_THT:CP_Radial_D8.0mm_P3.50mm"
 			(at 196.5452 147.32 0)
 			(effects
@@
 			)
 		)
-		(property "Footprint" "Sen Robo:CP_Radial_D8.0mm_P3.50mm"
+		(property "Footprint" "Capacitor_THT:CP_Radial_D8.0mm_P3.50mm"
 			(at 390.8552 149.86 0)
 			(effects

Commit message: ugly buck
Parts:
- L1, L2: footprint Inductor_SMD:L_0603_1608Metric_Pad1.05x0.95mm_HandSolder -> layer2v3:0630 One Piece Inductor
Changed lines of the file:
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@@
 	(label "Motor Driver"
 		(at 317.5 123.19 0)
+		(fields_autoplaced yes)
 		(effects
 			(font
@@
 	(label "Motor 1 EN B"
 		(at 171.45 52.07 0)
+		(fields_autoplaced yes)
 		(effects
 			(font
@@
 	(label "Motor 3 Out B"
 		(at 152.4 199.39 180)
+		(fields_autoplaced yes)
 		(effects
 			(font
@@
 	(label "Motor 2 EN B"
 		(at 171.45 57.15 0)
+		(fields_autoplaced yes)
 		(effects
 			(font
@@
 	(label "Motor 4 EN A"
 		(at 171.45 64.77 0)
+		(fields_autoplaced yes)
 		(effects
 			(font
@@
 	(label "Motor 1 EN A"
 		(at 26.67 128.27 0)
+		(fields_autoplaced yes)
 		(effects
 			(font
@@
 	(label "PWM Motor 4"
 		(at 171.45 80.01 0)
+		(fields_autoplaced yes)
 		(effects
 			(font
@@
 	(label "PWM Motor 2"
 		(at 120.65 140.97 0)
+		(fields_autoplaced yes)
 		(effects
 			(font
@@
 	(label "Motor 2 EN B"
 		(at 123.19 133.35 0)
+		(fields_autoplaced yes)
 		(effects
 			(font
@@
 	(label "Motor Driver"
 		(at 123.19 121.92 0)
+		(fields_autoplaced yes)
 		(effects
 			(font
@@
 	(label "Motor 2 Out A"
 		(at 177.8 179.07 180)
+		(fields_autoplaced yes)
 		(effects
 			(font
@@
 	(label "Motor 2 EN A"
 		(at 123.19 128.27 0)
+		(fields_autoplaced yes)
 		(effects
 			(font
@@
 	(label "Motor 1 Out B"
 		(at 96.52 133.35 180)
+		(fields_autoplaced yes)
 		(effects
 			(font
@@
 	(label "GND"
 		(at 171.45 82.55 0)
+		(fields_autoplaced yes)
 		(effects
 			(font
@@
 	(label "L1 RX"
 		(at 171.45 62.23 0)
+		(fields_autoplaced yes)
 		(effects
 			(font
@@
 	(label "RX (IMU)"
 		(at 135.89 57.15 180)
+		(fields_autoplaced yes)
 		(effects
 			(font
@@
 	(label "Motor 2 Out A"
 		(at 193.04 128.27 180)
+		(fields_autoplaced yes)
 		(effects
 			(font
@@
 	(label "PWM Motor 2"
 		(at 171.45 74.93 0)
+		(fields_autoplaced yes)
 		(effects
 			(font
@@
 	(label "Motor 4 Out A"
 		(at 387.35 129.54 180)
+		(fields_autoplaced yes)
 		(effects
 			(font
@@
 	(label "Motor 1 Out A"
 		(at 96.52 128.27 180)
+		(fields_autoplaced yes)
 		(effects
 			(font
@@
 	(label "TX (L3 ESP 32)"
 		(at 135.89 67.31 180)
+		(fields_autoplaced yes)
 		(effects
 			(font
@@
 	(label "Motor 2 Out B"
 		(at 193.04 133.35 180)
+		(fields_autoplaced yes)
 		(effects
 			(font
@@
 	(label "Motor 1 Out B"
 		(at 152.4 182.88 180)
+		(fields_autoplaced yes)
 		(effects
 			(font
@@
 	(label "TX (IMU)"
 		(at 135.89 59.69 180)
+		(fields_autoplaced yes)
 		(effects
 			(font
@@
 	(label "Motor 4 Out B"
 		(at 179.07 198.12 180)
+		(fields_autoplaced yes)
 		(effects
 			(font
@@
 	(label "Motor Driver"
 		(at 218.44 119.38 0)
+		(fields_autoplaced yes)
 		(effects
 			(font
@@
 	(label "RX (CAM)"
 		(at 135.89 54.61 180)
+		(fields_autoplaced yes)
 		(effects
 			(font
@@
 	(label "TX (L3 ESP 32)"
 		(at 72.39 185.42 0)
+		(fields_autoplaced yes)
 		(effects
 			(font
@@
 	(label "Motor 1 EN A"
 		(at 171.45 49.53 0)
+		(fields_autoplaced yes)
 		(effects
 			(font
@@
 	(label "Motor 3 EN B"
 		(at 135.89 74.93 180)
+		(fields_autoplaced yes)
 		(effects
 			(font
@@
 	(label "PWM Motor 3"
 		(at 171.45 77.47 0)
+		(fields_autoplaced yes)
 		(effects
 			(font
@@
 	(label "Motor 2 EN A"
 		(at 171.45 54.61 0)
+		(fields_autoplaced yes)
 		(effects
 			(font
@@
 	(label "RX (L3 ESP 32)"
 		(at 135.89 69.85 180)
+		(fields_autoplaced yes)
 		(effects
 			(font
@@
 	(label "Motor 4 EN B"
 		(at 171.45 67.31 0)
+		(fields_autoplaced yes)
 		(effects
 			(font
@@
 	(label "Motor Driver"
 		(at 16.51 173.99 0)
+		(fields_autoplaced yes)
 		(effects
 			(font
@@
 	(label "PWM Motor 3"
 		(at 217.17 138.43 0)
+		(fields_autoplaced yes)
 		(effects
 			(font
@@
 	(label "Motor 3 EN B"
 		(at 218.44 130.81 0)
+		(fields_autoplaced yes)
 		(effects
 			(font
@@
 	(label "Motor 1 Out A"
 		(at 152.4 180.34 180)
+		(fields_autoplaced yes)
 		(effects
 			(font
@@
 	(label "Motor 3 Out A"
 		(at 289.56 125.73 180)
+		(fields_autoplaced yes)
 		(effects
 			(font
@@
 	(label "Motor 4 EN B"
 		(at 317.5 134.62 0)
+		(fields_autoplaced yes)
 		(effects
 			(font
@@
 	(label "Motor 4 Out B"
 		(at 387.35 134.62 180)
+		(fields_autoplaced yes)
 		(effects
 			(font
@@
 	(label "RX (IMU)"
 		(at 72.39 193.04 0)
+		(fields_autoplaced yes)
 		(effects
 			(font
@@
 	(label "Motor 3 EN A"
 		(at 135.89 72.39 180)
+		(fields_autoplaced yes)
 		(effects
 			(font
@@
 	(label "RX (L3 ESP 32)"
 		(at 72.39 182.88 0)
+		(fields_autoplaced yes)
 		(effects
 			(font
@@
 	(label "Motor 2 Out B"
 		(at 177.8 181.61 180)
+		(fields_autoplaced yes)
 		(effects
 			(font
@@
 	(label "Motor Driver"
 		(at 26.67 121.92 0)
+		(fields_autoplaced yes)
 		(effects
 			(font
@@
 	(label "TX (CAM)"
 		(at 135.89 52.07 180)
+		(fields_autoplaced yes)
 		(effects
 			(font
@@
 	(label "L1 TX"
 		(at 207.01 181.61 180)
+		(fields_autoplaced yes)
 		(effects
 			(font
@@
 	(label "Motor 3 EN A"
 		(at 218.44 125.73 0)
+		(fields_autoplaced yes)
 		(effects
 			(font
@@
 	(label "L1 RX"
 		(at 207.01 179.07 180)
+		(fields_autoplaced yes)
 		(effects
 			(font
@@
 	(label "PWM Motor 4"
 		(at 314.96 142.24 0)
+		(fields_autoplaced yes)
 		(effects
 			(font
@@
 	(label "L1 TX"
 		(at 171.45 59.69 0)
+		(fields_autoplaced yes)
 		(effects
 			(font
@@
 	(label "Motor 3 Out B"
 		(at 289.56 130.81 180)
+		(fields_autoplaced yes)
 		(effects
 			(font
@@
 	(label "TX (CAM)"
 		(at 72.39 190.5 0)
+		(fields_autoplaced yes)
 		(effects
 			(font
@@
 	(label "Motor 4 EN A"
 		(at 317.5 129.54 0)
+		(fields_autoplaced yes)
 		(effects
 			(font
@@
 	(label "TX (IMU)"
 		(at 72.39 195.58 0)
+		(fields_autoplaced yes)
 		(effects
 			(font
@@
 	(label "Motor 1 EN B"
 		(at 26.67 133.35 0)
+		(fields_autoplaced yes)
 		(effects
 			(font
@@
 	(label "Motor 4 Out A"
 		(at 179.07 195.58 180)
+		(fields_autoplaced yes)
 		(effects
 			(font
@@
 	(label "RX (CAM)"
 		(at 72.39 187.96 0)
+		(fields_autoplaced yes)
 		(effects
 			(font
@@
 	(label "PWM Motor 1"
 		(at 24.13 140.97 0)
+		(fields_autoplaced yes)
 		(effects
 			(font
@@
 	(label "PWM Motor 1"
 		(at 171.45 72.39 0)
+		(fields_autoplaced yes)
 		(effects
 			(font
@@
 	(label "Motor 3 Out A"
 		(at 152.4 196.85 180)
+		(fields_autoplaced yes)
 		(effects
 			(font
@@
 			)
 		)
-		(property "Footprint" "Inductor_SMD:L_0603_1608Metric_Pad1.05x0.95mm_HandSolder"
+		(property "Footprint" "layer2v3:0630 One Piece Inductor"
 			(at 83.82 69.85 0)
 			(effects
@@
 			)
 		)
-		(property "Footprint" "Inductor_SMD:L_0603_1608Metric_Pad1.05x0.95mm_HandSolder"
+		(property "Footprint" "layer2v3:0630 One Piece Inductor"
 			(at 83.82 31.75 0)
 			(effects

Commit message: tidied up 3v3 buck
Parts:
- C2, C6: footprint Capacitor_SMD:C_0603_1608Metric_Pad1.08x0.95mm_HandSolder -> Capacitor_SMD:C_0603_1608Metric
- R28, R37: footprint Sen Robo:res0603 -> Resistor_SMD:R_0603_1608Metric
Changed lines of the file:
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@@
 	(label "Motor Driver"
 		(at 317.5 123.19 0)
-		(fields_autoplaced yes)
 		(effects
 			(font
@@
 	(label "Motor 1 EN B"
 		(at 171.45 52.07 0)
-		(fields_autoplaced yes)
 		(effects
 			(font
@@
 	(label "Motor 3 Out B"
 		(at 152.4 199.39 180)
-		(fields_autoplaced yes)
 		(effects
 			(font
@@
 	(label "Motor 2 EN B"
 		(at 171.45 57.15 0)
-		(fields_autoplaced yes)
 		(effects
 			(font
@@
 	(label "Motor 4 EN A"
 		(at 171.45 64.77 0)
-		(fields_autoplaced yes)
 		(effects
 			(font
@@
 	(label "Motor 1 EN A"
 		(at 26.67 128.27 0)
-		(fields_autoplaced yes)
 		(effects
 			(font
@@
 	(label "PWM Motor 4"
 		(at 171.45 80.01 0)
-		(fields_autoplaced yes)
 		(effects
 			(font
@@
 	(label "PWM Motor 2"
 		(at 120.65 140.97 0)
-		(fields_autoplaced yes)
 		(effects
 			(font
@@
 	(label "Motor 2 EN B"
 		(at 123.19 133.35 0)
-		(fields_autoplaced yes)
 		(effects
 			(font
@@
 	(label "Motor Driver"
 		(at 123.19 121.92 0)
-		(fields_autoplaced yes)
 		(effects
 			(font
@@
 	(label "Motor 2 Out A"
 		(at 177.8 179.07 180)
-		(fields_autoplaced yes)
 		(effects
 			(font
@@
 	(label "Motor 2 EN A"
 		(at 123.19 128.27 0)
-		(fields_autoplaced yes)
 		(effects
 			(font
@@
 	(label "Motor 1 Out B"
 		(at 96.52 133.35 180)
-		(fields_autoplaced yes)
 		(effects
 			(font
@@
 	(label "GND"
 		(at 171.45 82.55 0)
-		(fields_autoplaced yes)
 		(effects
 			(font
@@
 	(label "L1 RX"
 		(at 171.45 62.23 0)
-		(fields_autoplaced yes)
 		(effects
 			(font
@@
 	(label "RX (IMU)"
 		(at 135.89 57.15 180)
-		(fields_autoplaced yes)
 		(effects
 			(font
@@
 	(label "Motor 2 Out A"
 		(at 193.04 128.27 180)
-		(fields_autoplaced yes)
 		(effects
 			(font
@@
 	(label "PWM Motor 2"
 		(at 171.45 74.93 0)
-		(fields_autoplaced yes)
 		(effects
 			(font
@@
 	(label "Motor 4 Out A"
 		(at 387.35 129.54 180)
-		(fields_autoplaced yes)
 		(effects
 			(font
@@
 	(label "Motor 1 Out A"
 		(at 96.52 128.27 180)
-		(fields_autoplaced yes)
 		(effects
 			(font
@@
 	(label "TX (L3 ESP 32)"
 		(at 135.89 67.31 180)
-		(fields_autoplaced yes)
 		(effects
 			(font
@@
 	(label "Motor 2 Out B"
 		(at 193.04 133.35 180)
-		(fields_autoplaced yes)
 		(effects
 			(font
@@
 	(label "Motor 1 Out B"
 		(at 152.4 182.88 180)
-		(fields_autoplaced yes)
 		(effects
 			(font
@@
 	(label "TX (IMU)"
 		(at 135.89 59.69 180)
-		(fields_autoplaced yes)
 		(effects
 			(font
@@
 	(label "Motor 4 Out B"
 		(at 179.07 198.12 180)
-		(fields_autoplaced yes)
 		(effects
 			(font
@@
 	(label "Motor Driver"
 		(at 218.44 119.38 0)
-		(fields_autoplaced yes)
 		(effects
 			(font
@@
 	(label "RX (CAM)"
 		(at 135.89 54.61 180)
-		(fields_autoplaced yes)
 		(effects
 			(font
@@
 	(label "TX (L3 ESP 32)"
 		(at 72.39 185.42 0)
-		(fields_autoplaced yes)
 		(effects
 			(font
@@
 	(label "Motor 1 EN A"
 		(at 171.45 49.53 0)
-		(fields_autoplaced yes)
 		(effects
 			(font
@@
 	(label "Motor 3 EN B"
 		(at 135.89 74.93 180)
-		(fields_autoplaced yes)
 		(effects
 			(font
@@
 	(label "PWM Motor 3"
 		(at 171.45 77.47 0)
-		(fields_autoplaced yes)
 		(effects
 			(font
@@
 	(label "Motor 2 EN A"
 		(at 171.45 54.61 0)
-		(fields_autoplaced yes)
 		(effects
 			(font
@@
 	(label "RX (L3 ESP 32)"
 		(at 135.89 69.85 180)
-		(fields_autoplaced yes)
 		(effects
 			(font
@@
 	(label "Motor 4 EN B"
 		(at 171.45 67.31 0)
-		(fields_autoplaced yes)
 		(effects
 			(font
@@
 	(label "Motor Driver"
 		(at 16.51 173.99 0)
-		(fields_autoplaced yes)
 		(effects
 			(font
@@
 	(label "PWM Motor 3"
 		(at 217.17 138.43 0)
-		(fields_autoplaced yes)
 		(effects
 			(font
@@
 	(label "Motor 3 EN B"
 		(at 218.44 130.81 0)
-		(fields_autoplaced yes)
 		(effects
 			(font
@@
 	(label "Motor 1 Out A"
 		(at 152.4 180.34 180)
-		(fields_autoplaced yes)
 		(effects
 			(font
@@
 	(label "Motor 3 Out A"
 		(at 289.56 125.73 180)
-		(fields_autoplaced yes)
 		(effects
 			(font
@@
 	(label "Motor 4 EN B"
 		(at 317.5 134.62 0)
-		(fields_autoplaced yes)
 		(effects
 			(font
@@
 	(label "Motor 4 Out B"
 		(at 387.35 134.62 180)
-		(fields_autoplaced yes)
 		(effects
 			(font
@@
 	(label "RX (IMU)"
 		(at 72.39 193.04 0)
-		(fields_autoplaced yes)
 		(effects
 			(font
@@
 	(label "Motor 3 EN A"
 		(at 135.89 72.39 180)
-		(fields_autoplaced yes)
 		(effects
 			(font
@@
 	(label "RX (L3 ESP 32)"
 		(at 72.39 182.88 0)
-		(fields_autoplaced yes)
 		(effects
 			(font
@@
 	(label "Motor 2 Out B"
 		(at 177.8 181.61 180)
-		(fields_autoplaced yes)
 		(effects
 			(font
@@
 	(label "Motor Driver"
 		(at 26.67 121.92 0)
-		(fields_autoplaced yes)
 		(effects
 			(font
@@
 	(label "TX (CAM)"
 		(at 135.89 52.07 180)
-		(fields_autoplaced yes)
 		(effects
 			(font
@@
 	(label "L1 TX"
 		(at 207.01 181.61 180)
-		(fields_autoplaced yes)
 		(effects
 			(font
@@
 	(label "Motor 3 EN A"
 		(at 218.44 125.73 0)
-		(fields_autoplaced yes)
 		(effects
 			(font
@@
 	(label "L1 RX"
 		(at 207.01 179.07 180)
-		(fields_autoplaced yes)
 		(effects
 			(font
@@
 	(label "PWM Motor 4"
 		(at 314.96 142.24 0)
-		(fields_autoplaced yes)
 		(effects
 			(font
@@
 	(label "L1 TX"
 		(at 171.45 59.69 0)
-		(fields_autoplaced yes)
 		(effects
 			(font
@@
 	(label "Motor 3 Out B"
 		(at 289.56 130.81 180)
-		(fields_autoplaced yes)
 		(effects
 			(font
@@
 	(label "TX (CAM)"
 		(at 72.39 190.5 0)
-		(fields_autoplaced yes)
 		(effects
 			(font
@@
 	(label "Motor 4 EN A"
 		(at 317.5 129.54 0)
-		(fields_autoplaced yes)
 		(effects
 			(font
@@
 	(label "TX (IMU)"
 		(at 72.39 195.58 0)
-		(fields_autoplaced yes)
 		(effects
 			(font
@@
 	(label "Motor 1 EN B"
 		(at 26.67 133.35 0)
-		(fields_autoplaced yes)
 		(effects
 			(font
@@
 	(label "Motor 4 Out A"
 		(at 179.07 195.58 180)
-		(fields_autoplaced yes)
 		(effects
 			(font
@@
 	(label "RX (CAM)"
 		(at 72.39 187.96 0)
-		(fields_autoplaced yes)
 		(effects
 			(font
@@
 	(label "PWM Motor 1"
 		(at 24.13 140.97 0)
-		(fields_autoplaced yes)
 		(effects
 			(font
@@
 	(label "PWM Motor 1"
 		(at 171.45 72.39 0)
-		(fields_autoplaced yes)
 		(effects
 			(font
@@
 	(label "Motor 3 Out A"
 		(at 152.4 196.85 180)
-		(fields_autoplaced yes)
 		(effects
 			(font
@@
 			)
 		)
-		(property "Footprint" "Sen Robo:res0603"
+		(property "Footprint" "Resistor_SMD:R_0603_1608Metric"
 			(at 101.092 74.93 90)
 			(effects
@@
 			)
 		)
-		(property "Footprint" "Capacitor_SMD:C_0603_1608Metric_Pad1.08x0.95mm_HandSolder"
+		(property "Footprint" "Capacitor_SMD:C_0603_1608Metric"
 			(at 28.9052 80.01 0)
 			(effects
@@
 			)
 		)
-		(property "Footprint" "Capacitor_SMD:C_0603_1608Metric_Pad1.08x0.95mm_HandSolder"
+		(property "Footprint" "Capacitor_SMD:C_0603_1608Metric"
 			(at 72.39 63.8048 0)
 			(effects
@@
 			)
 		)
-		(property "Footprint" "Sen Robo:res0603"
+		(property "Footprint" "Resistor_SMD:R_0603_1608Metric"
 			(at 101.092 86.36 90)
 			(effects
