File: Electrical/PCB V3 (21 Jan)/Layer 2/Layer 2/_autosave-Layer 2.kicad_sch (KiCad schematic)
At the start: 86 parts, among them J1 XT60-M, J2 Conn_02x04_Odd_Even, J3 Conn_01x04, J5 Conn_01x02, Q1 AON6354, Q2 AON6354, Q3 AON6354, Q4 AON6354, SW2 SW_SPST, SW3 SW_SPST, U1 VNH5019ATR-E, U12 VNH5019ATR-E, U2 TPS5430DDAG4, U3 TPS5430DDAG4, U4 XT30UPB-M, U5 VNH5019ATR-E, U6 XT30UPB-M, U7 XT30UPB-M, U8 XT30UPB-M, U9 VNH5019ATR-E

Commit message: did alot of uncursing
Parts:
- added H11, H12: MountingHole, MountingHole:MountingHole_3.2mm_M3_DIN965_Pad, symbol Mechanical:MountingHole
Other:
- moved on the sheet: H10, H6, H7, H8, H9
Changed lines of the file:
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@@
 	(symbol
 		(lib_id "Mechanical:MountingHole")
-		(at 224.79 44.45 180)
+		(at 224.79 39.37 180)
 		(unit 1)
 		(exclude_from_sim yes)
@@
 		(fields_autoplaced yes)
 		(property "Reference" "H7"
-			(at 227.5246 43.1799 0)
+			(at 227.5246 38.0999 0)
 			(effects
 				(font
@@
 		)
 		(property "Value" "MountingHole"
-			(at 227.5246 45.7199 0)
+			(at 227.5246 40.6399 0)
 			(effects
 				(font
@@
 		)
 		(property "Footprint" "MountingHole:MountingHole_3.2mm_M3_DIN965_Pad"
-			(at 224.79 44.45 0)
+			(at 224.79 39.37 0)
 			(effects
 				(font
@@
 		)
 		(property "Datasheet" "~"
-			(at 224.79 44.45 0)
+			(at 224.79 39.37 0)
 			(effects
 				(font
@@
 		)
 		(property "Description" "Mounting Hole without connection"
-			(at 224.79 44.45 0)
+			(at 224.79 39.37 0)
 			(effects
 				(font
@@
 	(symbol
 		(lib_id "Mechanical:MountingHole")
-		(at 224.79 49.53 180)
+		(at 224.79 44.45 180)
 		(unit 1)
 		(exclude_from_sim yes)
@@
 		(fields_autoplaced yes)
 		(property "Reference" "H8"
-			(at 227.33 48.2599 0)
+			(at 227.33 43.1799 0)
 			(effects
 				(font
@@
 		)
 		(property "Value" "MountingHole"
-			(at 227.33 50.7999 0)
+			(at 227.33 45.7199 0)
 			(effects
 				(font
@@
 		)
 		(property "Footprint" "MountingHole:MountingHole_3.2mm_M3_DIN965_Pad"
-			(at 224.79 49.53 0)
+			(at 224.79 44.45 0)
 			(effects
 				(font
@@
 		)
 		(property "Datasheet" "~"
-			(at 224.79 49.53 0)
+			(at 224.79 44.45 0)
 			(effects
 				(font
@@
 		)
 		(property "Description" "Mounting Hole without connection"
-			(at 224.79 49.53 0)
+			(at 224.79 44.45 0)
 			(effects
 				(font
@@
 	(symbol
 		(lib_id "Mechanical:MountingHole")
-		(at 224.79 39.37 180)
+		(at 204.47 64.77 180)
 		(unit 1)
 		(exclude_from_sim yes)
@@
 		(fields_autoplaced yes)
 		(property "Reference" "H6"
-			(at 227.33 38.0999 0)
+			(at 207.01 63.4999 0)
 			(effects
 				(font
@@
 		)
 		(property "Value" "MountingHole"
-			(at 227.33 40.6399 0)
+			(at 207.01 66.0399 0)
 			(effects
 				(font
@@
 		)
 		(property "Footprint" "MountingHole:MountingHole_3.2mm_M3_DIN965_Pad"
-			(at 224.79 39.37 0)
+			(at 204.47 64.77 0)
 			(effects
 				(font
@@
 		)
 		(property "Datasheet" "~"
-			(at 224.79 39.37 0)
+			(at 204.47 64.77 0)
 			(effects
 				(font
@@
 		)
 		(property "Description" "Mounting Hole without connection"
-			(at 224.79 39.37 0)
+			(at 204.47 64.77 0)
 			(effects
 				(font
@@
 	(symbol
 		(lib_id "Mechanical:MountingHole")
-		(at 224.79 59.69 180)
+		(at 224.79 54.61 180)
 		(unit 1)
 		(exclude_from_sim yes)
@@
 		(fields_autoplaced yes)
 		(property "Reference" "H10"
-			(at 227.33 58.4199 0)
+			(at 227.33 53.3399 0)
 			(effects
 				(font
@@
 		)
 		(property "Value" "MountingHole"
-			(at 227.33 60.9599 0)
+			(at 227.33 55.8799 0)
 			(effects
 				(font
@@
 		)
 		(property "Footprint" "MountingHole:MountingHole_3.2mm_M3_DIN965_Pad"
-			(at 224.79 59.69 0)
+			(at 224.79 54.61 0)
 			(effects
 				(font
@@
 		)
 		(property "Datasheet" "~"
-			(at 224.79 59.69 0)
+			(at 224.79 54.61 0)
 			(effects
 				(font
@@
 		)
 		(property "Description" "Mounting Hole without connection"
-			(at 224.79 59.69 0)
+			(at 224.79 54.61 0)
 			(effects
 				(font
@@
 	(symbol
 		(lib_id "Mechanical:MountingHole")
-		(at 224.79 54.61 180)
+		(at 224.79 49.53 180)
 		(unit 1)
 		(exclude_from_sim yes)
@@
 		(fields_autoplaced yes)
 		(property "Reference" "H9"
-			(at 227.5246 53.3399 0)
+			(at 227.5246 48.2599 0)
 			(effects
 				(font
@@
 		)
 		(property "Value" "MountingHole"
-			(at 227.5246 55.8799 0)
+			(at 227.5246 50.7999 0)
 			(effects
 				(font
@@
 		)
 		(property "Footprint" "MountingHole:MountingHole_3.2mm_M3_DIN965_Pad"
-			(at 224.79 54.61 0)
+			(at 224.79 49.53 0)
 			(effects
 				(font
@@
 		)
 		(property "Datasheet" "~"
-			(at 224.79 54.61 0)
+			(at 224.79 49.53 0)
 			(effects
 				(font
@@
 		)
 		(property "Description" "Mounting Hole without connection"
-			(at 224.79 54.61 0)
+			(at 224.79 49.53 0)
 			(effects
 				(font
@@
 					(unit 1)
 				)
+			)
+		)
+	)
+	(symbol
+		(lib_id "Mechanical:MountingHole")
+		(at 224.79 64.77 180)
+		(unit 1)
+		(exclude_from_sim yes)
+		(in_bom no)
+		(on_board yes)
+		(dnp no)
+		(property "Reference" "H12"
+			(at 227.33 63.4999 0)
+			(effects
+				(font
+					(size 1.27 1.27)
+				)
+				(justify right)
+			)
+		)
+		(property "Value" "MountingHole"
+			(at 227.33 66.0399 0)
+			(effects
+				(font
+					(size 1.27 1.27)
+				)
+				(justify right)
+			)
+		)
+		(property "Footprint" "MountingHole:MountingHole_3.2mm_M3_DIN965_Pad"
+			(at 224.79 64.77 0)
+			(effects
+				(font
+					(size 1.27 1.27)
+				)
+				(hide yes)
+			)
+		)
+		(property "Datasheet" "~"
+			(at 224.79 64.77 0)
+			(effects
+				(font
+					(size 1.27 1.27)
+				)
+				(hide yes)
+			)
+		)
+		(property "Description" "Mounting Hole without connection"
+			(at 224.79 64.77 0)
+			(effects
+				(font
+					(size 1.27 1.27)
+				)
+				(hide yes)
+			)
+		)
+		(instances
+			(project "Layer 2"
+				(path "/73bb99ca-959f-40cf-90f8-36d6928b007b"
+					(reference "H12")
+					(unit 1)
+				)
+			)
+		)
+	)
+	(symbol
+		(lib_id "Mechanical:MountingHole")
+		(at 224.79 59.69 180)
+		(unit 1)
+		(exclude_from_sim yes)
+		(in_bom no)
+		(on_board yes)
+		(dnp no)
+		(property "Reference" "H11"
+			(at 227.33 58.42 0)
+			(effects
+				(font
+					(size 1.27 1.27)
+				)
+				(justify right)
+			)
+		)
+		(property "Value" "MountingHole"
+			(at 227.076 60.96 0)
+			(effects
+				(font
+					(size 1.27 1.27)
+				)
+				(justify right)
+			)
+		)
+		(property "Footprint" "MountingHole:MountingHole_3.2mm_M3_DIN965_Pad"
+			(at 224.79 59.69 0)
+			(effects
+				(font
+					(size 1.27 1.27)
+				)
+				(hide yes)
+			)
+		)
+		(property "Datasheet" "~"
+			(at 224.79 59.69 0)
+			(effects
+				(font
+					(size 1.27 1.27)
+				)
+				(hide yes)
+			)
+		)
+		(property "Description" "Mounting Hole without connection"
+			(at 224.79 59.69 0)
+			(effects
+				(font
+					(size 1.27 1.27)
+				)
+				(hide yes)
+			)
+		)
+		(instances
+			(project "Layer 2"
+				(path "/73bb99ca-959f-40cf-90f8-36d6928b007b"
+					(reference "H11")
+					(unit 1)
+				)
