File: Electrical/PCB V2 (26 Nov)/L3/Layer 3 schematics 24 jan/_autosave-layer 3 schematics 15 jan.kicad_sch (KiCad schematic)
At the start: 3 parts, among them J1 Conn_01x06, U2 XT30UPB-M

Commit message: 24 JAN UPDATE
LLOL
Parts:
- removed U1: ~, symbol openmv m7:Openmv_M7
- removed U2: XT30UPB-M, XT30UPB-M:XT30UPB-M, symbol XT30UPB-M:XT30UPB-M
- added J2: Conn_01x02_Pin, Connector_PinHeader_1.00mm:PinHeader_1x02_P1.00mm_Vertical, symbol Connector:Conn_01x02_Pin
- added U1: XT30UPB-M, XT30UPB-M:XT30UPB-M, symbol XT30UPB-M:XT30UPB-M
- added U2: ~, symbol openmv m7:Openmv_M7
- J1: footprint (none) -> Connector_PinHeader_1.00mm:PinHeader_1x06_P1.00mm_Vertical
Connections:
- net GND: now also U1.P$2 (-), U2. (VIN)
- net SCL: now reaches J1.3 (Pin_3)
- net SDA: now reaches J1.4 (Pin_4)
- net 5V renamed 3V3
- net 3V3: now also U1.P$1 (+), U2. (VIN)
- new net RX: J2.1 (Pin_1), U2. (VIN)
- new net TX: J2.2 (Pin_2), U2. (VIN)
Other:
- note added: "CONNECTORS"
- note added: "OPENMV M7"
- note added: "POWER SUPPLY"
- moved on the sheet: J1
