File: Electrical/PCB V3 (21 Jan)/Layer 3/layer 3 schematics 24 jan.kicad_pcb (KiCad board)
At the start: 2 copper layers, 76.1 x 110 mm, 22 parts, among them J1 Conn_01x06, J2 Conn_01x02, J3 Conn_01x06, J4 Conn_01x06, J5 Conn_01x06, J7 Conn_01x08, J8 Conn_01x02, U2 XT30UPB-M, U3 4754

Commit message: Updated L3
chen xuan wants to do when i gone
Parts:
- moved J4 146.4 mm to (248.0, 93.9), turned to 180 degrees
- moved J1 135.3 mm to (232.6, 36.3), turned to -90 degrees
- moved J3 124.4 mm to (194.9, 138.7), turned to 90 degrees
- moved H1 122.4 mm to (71.9, 147.6)
- moved H10 122.4 mm to (91.9, 182.1)
- moved H12 122.4 mm to (116.9, 98.1)
- moved H2 122.4 mm to (76.9, 182.1)
- moved H3 122.4 mm to (122.0, 147.6)
- moved H4 122.4 mm to (71.9, 132.6)
- moved H6 122.4 mm to (122.0, 132.6)
- moved H8 122.4 mm to (101.9, 98.1)
- moved H11 122.4 mm to (73.9, 110.1)
- moved H5 122.4 mm to (73.9, 170.1)
- moved H7 122.4 mm to (120.0, 170.1)
- moved H9 122.4 mm to (120.0, 111.8)
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Other:
- board size 76.1 x 110 mm -> 181.6 x 151.3 mm

Commit message: 7 feb update!!! stop at pull up res
Parts:
- removed J2, J8: Conn_01x02, Connector_PinHeader_2.54mm:PinHeader_1x02_P2.54mm_Vertical
- removed J7: Conn_01x08, Connector_PinHeader_2.54mm:PinHeader_1x08_P2.54mm_Vertical
- removed U2: XT30UPB-M, XT30UPB-M:XT30UPB-M
- added J6: Conn_01x06, Connector_JST:JST_EH_B6B-EH-A_1x06_P2.50mm_Vertical, F.Cu at (217.9, 138.9)
- H1, H10, H11, H12, H2, H3, H4, H5, H6, H7, H8, H9: footprint MountingHole:MountingHole_3.2mm_M3 -> MountingHole:MountingHole_3.2mm_M3_Pad_Via
- moved H2 183.8 mm to (238.8, 95.0)
- moved H11 171.2 mm to (236.8, 57.5)
- moved H3 135.0 mm to (238.8, 80.0)
- moved H1 128.1 mm to (188.7, 95.0)
- moved H10 128.1 mm to (208.7, 129.5)
- moved H12 128.1 mm to (233.7, 45.5)
- moved H4 128.1 mm to (188.7, 80.0)
- moved H8 128.1 mm to (218.7, 45.5)
- moved H5 126.6 mm to (193.7, 129.5)
- moved H6 115.8 mm to (236.8, 117.5)
- moved H9 89.1 mm to (190.7, 57.5)
- moved H7 88.1 mm to (190.7, 117.5)
Connections:
- net /3V3 renamed +3V3
- net /GND renamed GND
- U1 pad 1: /RX -> /L3 RX
- U1 pad 2: /TX -> /L3 TX
Other:
- board size 181.6 x 151.3 mm -> 129.9 x 119.9 mm

Commit message: last motor driver to be done and jst
Parts:
- removed J6: Conn_01x06, Connector_JST:JST_EH_B6B-EH-A_1x06_P2.50mm_Vertical
- added J2: Conn_02x04_Counter_Clockwise, Connector_JST:JST_PHD_B8B-PHDSS_2x04_P2.00mm_Vertical, F.Cu at (250.4, 68.8)
