File: Electrical/PCB V3 (21 Jan)/Layer 1/L1.kicad_sch (KiCad schematic)
At the start: 219 parts, among them J1 Conn_01x05, Q1 NMOS, U1 LM2587S-ADJ, U2 CD74HC4067SM, U3 CD74HC4067SM, U4 XT30UPB-M, U5 113991054

Commit message: somewhat finished l1, need to improve and un uglify
Parts:
- removed TP2: TestPoint_2Pole, customTps-2-Chairs:testpoint_2pad_2-chairs., symbol Connector:TestPoint_2Pole
- U4: footprint layer2v3:XT30UPB-M -> Connector_AMASS:AMASS_XT30U-M_1x02_P5.0mm_Vertical
Other:
- note removed: "12V/24V TP"
Changed lines of the file:
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@@
 		)
 	)
-	(text "12V/24V TP"
-		(exclude_from_sim no)
-		(at 362.204 190.754 0)
-		(effects
-			(font
-				(size 1.778 1.778)
-			)
-		)
-	)
 	(text "Boost & Capactiors"
 		(exclude_from_sim no)
@@
 	)
 	(symbol
-		(lib_id "power:+12V")
-		(at 356.87 200.66 90)
-		(unit 1)
-		(exclude_from_sim no)
-		(in_bom yes)
-		(on_board yes)
-		(dnp no)
-		(fields_autoplaced yes)
-		(property "Reference" "#PWR024"
-			(at 360.68 200.66 0)
-			(effects
-				(font
-					(size 1.27 1.27)
-				)
-				(hide yes)
-			)
-		)
-		(property "Value" "+12V"
-			(at 353.06 200.6599 90)
-			(effects
-				(font
-					(size 1.27 1.27)
-				)
-				(justify left)
-			)
-		)
-		(property "Footprint" ""
-			(at 356.87 200.66 0)
-			(effects
-				(font
-					(size 1.27 1.27)
-				)
-				(hide yes)
-			)
-		)
-		(property "Datasheet" ""
-			(at 356.87 200.66 0)
-			(effects
-				(font
-					(size 1.27 1.27)
-				)
-				(hide yes)
-			)
-		)
-		(property "Description" "Power symbol creates a global label with name \"+12V\""
-			(at 356.87 200.66 0)
-			(effects
-				(font
-					(size 1.27 1.27)
-				)
-				(hide yes)
-			)
-		)
-		(pin "1"
-		)
-		(instances
-			(project ""
-				(path "/9e8a7821-ee65-4356-a785-1f444d794ef4"
-					(reference "#PWR024")
-					(unit 1)
-				)
-			)
-		)
-	)
-	(symbol
 		(lib_id "Device:R_Photo")
 		(at 283.21 146.05 0)
@@
 			)
 		)
-		(property "Footprint" "layer2v3:XT30UPB-M"
+		(property "Footprint" "Connector_AMASS:AMASS_XT30U-M_1x02_P5.0mm_Vertical"
 			(at 501.65 190.5 0)
 			(effects
@@
 	)
 	(symbol
-		(lib_id "Connector:TestPoint_2Pole")
-		(at 361.95 200.66 0)
-		(unit 1)
-		(exclude_from_sim no)
-		(in_bom yes)
-		(on_board yes)
-		(dnp no)
-		(property "Reference" "TP2"
-			(at 361.95 194.818 0)
-			(effects
-				(font
-					(size 1.27 1.27)
-				)
-			)
-		)
-		(property "Value" "TestPoint_2Pole"
-			(at 361.95 197.358 0)
-			(effects
-				(font
-					(size 1.27 1.27)
-				)
-			)
-		)
-		(property "Footprint" "customTps-2-Chairs:testpoint_2pad_2-chairs."
-			(at 361.95 200.66 0)
-			(effects
-				(font
-					(size 1.27 1.27)
-				)
-				(hide yes)
-			)
-		)
-		(property "Datasheet" "~"
-			(at 361.95 200.66 0)
-			(effects
-				(font
-					(size 1.27 1.27)
-				)
-				(hide yes)
-			)
-		)
-		(property "Description" "2-polar test point"
-			(at 361.95 200.66 0)
-			(effects
-				(font
-					(size 1.27 1.27)
-				)
-				(hide yes)
-			)
-		)
-		(pin "1"
-		)
-		(pin "2"
-		)
-		(instances
-			(project "L1"
-				(path "/9e8a7821-ee65-4356-a785-1f444d794ef4"
-					(reference "TP2")
-					(unit 1)
-				)
-			)
-		)
-	)
-	(symbol
 		(lib_id "pspice:INDUCTOR")
 		(at 160.02 81.28 90)
@@
 	)
 	(symbol
-		(lib_id "power:+24V")
-		(at 367.03 200.66 270)
-		(unit 1)
-		(exclude_from_sim no)
-		(in_bom yes)
-		(on_board yes)
-		(dnp no)
-		(fields_autoplaced yes)
-		(property "Reference" "#PWR025"
-			(at 363.22 200.66 0)
-			(effects
-				(font
-					(size 1.27 1.27)
-				)
-				(hide yes)
-			)
-		)
-		(property "Value" "+24V"
-			(at 370.84 200.6599 90)
-			(effects
-				(font
-					(size 1.27 1.27)
-				)
-				(justify left)
-			)
-		)
-		(property "Footprint" ""
-			(at 367.03 200.66 0)
-			(effects
-				(font
-					(size 1.27 1.27)
-				)
-				(hide yes)
-			)
-		)
-		(property "Datasheet" ""
-			(at 367.03 200.66 0)
-			(effects
-				(font
-					(size 1.27 1.27)
-				)
-				(hide yes)
-			)
-		)
-		(property "Description" "Power symbol creates a global label with name \"+24V\""
-			(at 367.03 200.66 0)
-			(effects
-				(font
-					(size 1.27 1.27)
-				)
-				(hide yes)
-			)
-		)
-		(pin "1"
-		)
-		(instances
-			(project ""
-				(path "/9e8a7821-ee65-4356-a785-1f444d794ef4"
-					(reference "#PWR025")
-					(unit 1)
-				)
-			)
-		)
-	)
-	(symbol
 		(lib_id "Device:LED")
 		(at 238.76 91.44 90)
@@
 					(size 1.27 1.27)
 				)
-				(hide yes)
 			)
 		)
